Commit message: added logo and applied aluminum textures
git-svn-id: https://roboticssrv.wtb.tue.nl/svn/ros/code/tue-ros-pkg/trunk/tue_robot_models/amigo_robot_model@6886 3a3c2cfb-d3b9-409e-9e75-db8fcdbcaac6

File: body/body.urdf.xacro (robot description, xacro)
@@ -9,10 +9,10 @@
    <box size="0.25 0.25 0.5"/>
 </xacro:my_link_texturedmesh_diff_coll>
-<xacro:my_link name="torso_slider" mass="0.1" color="Grey">
-   <cylinder radius="0.024" length="0.6" />
+<xacro:my_link_texturedmesh name="torso_slider" mass="0.1" texture="aluminum">
    <origin xyz="0 0 0" rpy="0 0 0"/>
-   <origin xyz="0.0 0.0 0.0" rpy="0 1.5708 0"/>
+   <origin xyz="-0.35 0.0 0.0" rpy="0 1.5708 0"/>
    <inertia ixx="0.01"  ixy="0"  ixz="0" iyy="0.01" iyz="0" izz="0.01" />
-</xacro:my_link>
+   <mesh filename="package://amigo_robot_model/body/torsoslidertextured.dae" scale="0.01 0.01 0.01"/>
+</xacro:my_link_texturedmesh>
 <xacro:my_link name="base_link" mass="0" color="Red">
    <cylinder radius="0.0" length="0.00" />

File: body_extra_visuals/body_extra.urdf.xacro (robot description, xacro)
@@ -2,22 +2,22 @@
 <robot xmlns:xacro="http://ros.org/wiki/xacro">
 <!--torso sliders-->
-<xacro:my_link name="torso_assist_slider_right" mass="0.01" color="Grey">
-   <box size="0.6 0.01 0.03"/>
+<xacro:my_link_texturedmesh name="torso_assist_slider_right" mass="0.01" texture="aluminum">
    <origin xyz="0 0 0" rpy="0 0 0"/>
-   <origin xyz="0.0 0.0 0.0" rpy="0 0 0"/>
+   <origin xyz="-0.3  0.0 0.0" rpy="0 1.5708 0"/>
    <inertia ixx="0.01"  ixy="0"  ixz="0" iyy="0.01" iyz="0" izz="0.01" />
-</xacro:my_link>
-<xacro:my_link name="torso_assist_slider_left" mass="0.01" color="Grey">
-   <box size="0.6 0.01 0.03"/>
+   <mesh filename="package://amigo_robot_model/body_extra_visuals/torsoassistslidertextured.dae" scale="0.01 0.01 0.01"/>
+</xacro:my_link_texturedmesh>
+<xacro:my_link_texturedmesh name="torso_assist_slider_left" mass="0.01" texture="aluminum">
    <origin xyz="0 0 0" rpy="0 0 0"/>
-   <origin xyz="0.0 0.0 0.0" rpy="0 0 0"/>
+   <origin xyz="-0.3  0.0 0.0" rpy="0 1.5708 0"/>
    <inertia ixx="0.01"  ixy="0"  ixz="0" iyy="0.01" iyz="0" izz="0.01" />
-</xacro:my_link>
-<xacro:my_link name="torso_assist_slider_back" mass="0.01" color="Grey">
-   <box size="0.6 0.01 0.03"/>
+   <mesh filename="package://amigo_robot_model/body_extra_visuals/torsoassistslidertextured.dae" scale="0.01 0.01 0.01"/>
+</xacro:my_link_texturedmesh>
+<xacro:my_link_texturedmesh name="torso_assist_slider_back" mass="0.01" texture="aluminum">
    <origin xyz="0 0 0" rpy="0 0 0"/>
-   <origin xyz="0.0 0.0 0.0" rpy="0 0 0"/>
+   <origin xyz="-0.3 0.0 0.0" rpy="0 1.5708 0"/>
    <inertia ixx="0.01"  ixy="0"  ixz="0" iyy="0.01" iyz="0" izz="0.01" />
-</xacro:my_link>
+   <mesh filename="package://amigo_robot_model/body_extra_visuals/torsoassistslidertextured.dae" scale="0.01 0.01 0.01"/>
+</xacro:my_link_texturedmesh>
 <joint name="torso_slider_assist_joint_right" type="fixed">
     <parent link="torso"/>

File: head/head.urdf.xacro (robot description, xacro)
@@ -9,5 +9,5 @@
 </xacro:my_link>
 <xacro:my_link name="neck_pan" mass="0.05" color="Black">
-   <cylinder radius="0.015" length="0.08" /> <!--*--> <!--checked-->
+   <cylinder radius="0.015" length="0.0525" /> <!--*--> <!--checked-->
    <origin xyz="0.0 0.0 0.0335" rpy="0 0 0"/>
    <origin xyz="0.0 0.0 0.0335" rpy="0 0 0" />
@@ -15,10 +15,10 @@
    <color rgba="0.25 0.25 0.25 1.0"/>
 </xacro:my_link>
-<xacro:my_link name="neck_tilt" mass="0.05" color="Black">
-   <cylinder radius="0.015" length="0.057"  /> <!--*-->
+<xacro:my_link_texturedmesh name="neck_tilt" mass="0.05" texture="aluminum">
    <origin xyz="0.0 -0.0 0.0285" rpy="0 0 0"/>
-   <origin xyz="0.0 -0.0 0.0285" rpy="0 0 0" />
+   <origin xyz="0.0 -0.0 0.015" rpy="0 0 0" />
    <inertia ixx="0.001"  ixy="0"  ixz="0" iyy="0.001" iyz="0" izz="0.001" /> <!--*-->
-</xacro:my_link>
+   <mesh filename="package://amigo_robot_model/head/necktilttextured.dae" scale="0.01 0.01 0.01"/>
+</xacro:my_link_texturedmesh>
  <my_link_texturedmesh name="head" mass="0" texture="white">
    <origin xyz="0 0 0" rpy="0 0 0"/>

File: laser/laser.urdf.xacro (robot description, xacro)
@@ -13,3 +13,13 @@
    <limit effort="13.4" velocity="1.0" lower="-0.7809" upper="1.5708" />
 </xacro:my_joint>
+<xacro:my_link_texturedmesh name="logo" mass="0.01" texture="logo">
+   <origin xyz="0.0 0.0 0.0" rpy="0 0 0"/>
+   <origin xyz="0.025 0.0 0.006" rpy="0 0 3.1415" />
+   <inertia ixx="0.0001"  ixy="0"  ixz="0" iyy="0.0001" iyz="0" izz="0.0001" /> <!--*-->
+   <mesh filename="package://amigo_robot_model/laser/logo.dae" scale="0.004 0.004 0.004"/>
+</xacro:my_link_texturedmesh>
+  <joint name="logo_joint" type="fixed">
+    <parent link="base_laser"/>
+    <child link="logo"/>
+  </joint>
 </robot>

File: materials.urdf.xacro (robot description, xacro)
@@ -31,3 +31,9 @@
     <texture filename="package://amigo_robot_model/Media/materials/textures/white/white.jpg" />
   </material>
+  <material name="logo">
+    <texture filename="package://amigo_robot_model/Media/materials/textures/logo/tue.jpg" />
+  </material>
+  <material name="aluminum">
+    <texture filename="package://amigo_robot_model/Media/materials/textures/aluminum/aluminium_0001_c.jpg" />
+  </material>
 </robot>

Commit message: Updated offsets
git-svn-id: https://roboticssrv.wtb.tue.nl/svn/ros/code/tue-ros-pkg/trunk/tue_robot_models/amigo_robot_model@6890 3a3c2cfb-d3b9-409e-9e75-db8fcdbcaac6

File: body/body.urdf.xacro (robot description, xacro)
@@ -4,5 +4,5 @@
 <xacro:my_link_texturedmesh_diff_coll name="base" mass="20" texture="bottomcovers">
    <origin xyz="0.0 0.0 0.3275" rpy="0 0 0"/>
-   <origin xyz="0.0 0.0 0.3275" rpy="0 0 -1.5708" />
+   <origin xyz="0.0 0.0 0.23" rpy="0 0 -1.5708" />
    <inertia ixx="2.63"  ixy="0"  ixz="0" iyy="2.63" iyz="0" izz="2.4" /> <!--*-->
    <mesh filename="package://amigo_robot_model/body/bottomcovers.dae" scale="0.001 0.001 0.001"/>

File: laser/laser.urdf.xacro (robot description, xacro)
@@ -2,11 +2,11 @@
 <robot xmlns:xacro="http://ros.org/wiki/xacro">
 <xacro:my_link name="base_laser" mass="0.5" color="Black">
-   <box size="0.05 0.06 0.12" /> <!--*-->
+   <box size="0.05 0.065 0.12" /> <!--*-->
    <origin xyz="0.0 0.0 0.0" rpy="0 0 0"/>
-   <origin xyz="-0.005 0.0 0.0525" rpy="0 0 0" />
+   <origin xyz="-0.005 0.0 -0.0525" rpy="0 0 0" />
    <inertia ixx="0.0001"  ixy="0"  ixz="0" iyy="0.0001" iyz="0" izz="0.0001" /> <!--*-->
 </xacro:my_link>
 <xacro:my_joint name="base_laser_joint" type="fixed" parent="base" child="base_laser">
-   <origin xyz="0.31 0.0 0.1475" rpy="0 0 0"/>
+   <origin xyz="0.31 0.0 0.185" rpy="0 0 0"/>
    <dynamics damping="0.1" friction="0"/>
    <axis xyz="0 1 0"/>
@@ -15,5 +15,5 @@
 <xacro:my_link_texturedmesh name="logo" mass="0.01" texture="logo">
    <origin xyz="0.0 0.0 0.0" rpy="0 0 0"/>
-   <origin xyz="0.025 0.0 0.006" rpy="0 0 3.1415" />
+   <origin xyz="0.025 0.0 -0.165" rpy="0 0 3.1415" />
    <inertia ixx="0.0001"  ixy="0"  ixz="0" iyy="0.0001" iyz="0" izz="0.0001" /> <!--*-->
    <mesh filename="package://amigo_robot_model/laser/logo.dae" scale="0.004 0.004 0.004"/>

File: wheels/wheels.urdf.xacro (robot description, xacro)
@@ -7,5 +7,5 @@
     <child link="wheel_${side_LR}_${side_FR}"/>
     <axis xyz="1 0 0"/>
-    <origin xyz="${sign_LR}0.2 ${sign_FR}0.2 0.08" rpy="0 0 ${wheel_angle}"/>
+    <origin xyz="${sign_LR}0.205 ${sign_FR}0.205 0.005" rpy="0 0 ${wheel_angle}"/>
     <dynamics damping="1" friction="0.0"/>
     <limit effort="5.0" velocity="5.0"/>

Commit message: base plate, orange laser top, extended assist sliders and bounding boxes for batteries
git-svn-id: https://roboticssrv.wtb.tue.nl/svn/ros/code/tue-ros-pkg/trunk/tue_robot_models/amigo_robot_model@6923 3a3c2cfb-d3b9-409e-9e75-db8fcdbcaac6

File: body/body.urdf.xacro (robot description, xacro)
@@ -5,7 +5,8 @@
    <origin xyz="0.0 0.0 0.3275" rpy="0 0 0"/>
    <origin xyz="0.0 0.0 0.23" rpy="0 0 -1.5708" />
+   <origin xyz="0.0 0.0 0.33" rpy="0 0 -1.5708" />
    <inertia ixx="2.63"  ixy="0"  ixz="0" iyy="2.63" iyz="0" izz="2.4" /> <!--*-->
    <mesh filename="package://amigo_robot_model/body/bottomcovers.dae" scale="0.001 0.001 0.001"/>
-   <box size="0.25 0.25 0.5"/>
+   <box size="0.275 0.275 0.6"/>
 </xacro:my_link_texturedmesh_diff_coll>
 <xacro:my_link_texturedmesh name="torso_slider" mass="0.1" texture="aluminum">
@@ -21,4 +22,79 @@
    <inertia ixx="0"  ixy="0"  ixz="0" iyy="0" iyz="0" izz="0" />
 </xacro:my_link>
+<link name="batterycovercollision_left">
+   <inertial>
+     <origin xyz="0.0 0.0 0.0" />
+     <mass value="0.001"/>
+     <inertia ixx="0.01"  ixy="0"  ixz="0" iyy="0.01" iyz="0" izz="0.01" />
+   </inertial>
+    <visual>
+		<origin xyz="0.0 0.0 0.0" />
+		<geometry>
+			<box size="0.0 0.0 0.0"/>
+		</geometry>
+    </visual>
+    <collision>
+		<origin xyz="0.0 0.0 0.0" />
+		<geometry>
+			<box size="0.25 0.15 0.125"/>
+		</geometry>
+    </collision>
+</link>
+<joint name="batterycovercollision_left_joint" type="fixed">
+    <parent link="base"/>
+    <child link="batterycovercollision_left"/>
+    <axis xyz="1 0 0"/>
+    <origin xyz="0.0 0.25 0.1" rpy="0 0 0"/>
+</joint>
+<link name="batterycovercollision_right">
+   <inertial>
+     <origin xyz="0.0 0.0 0.0" />
+     <mass value="0.001"/>
+     <inertia ixx="0.01"  ixy="0"  ixz="0" iyy="0.01" iyz="0" izz="0.01" />
+   </inertial>
+    <visual>
+		<origin xyz="0.0 0.0 0.0" />
+		<geometry>
+			<box size="0.0 0.0 0.0"/>
+		</geometry>
+    </visual>
+    <collision>
+		<origin xyz="0.0 0.0 0.0" />
+		<geometry>
+			<box size="0.25 0.15 0.125"/>
+		</geometry>
+    </collision>
+</link>
+<joint name="batterycovercollision_right_joint" type="fixed">
+    <parent link="base"/>
+    <child link="batterycovercollision_right"/>
+    <axis xyz="1 0 0"/>
+    <origin xyz="0.0 -0.25 0.1" rpy="0 0 0"/>
+</joint>
+<link name="batterycovercollision_back">
+   <inertial>
+     <origin xyz="0.0 0.0 0.0" />
+     <mass value="0.001"/>
+     <inertia ixx="0.01"  ixy="0"  ixz="0" iyy="0.01" iyz="0" izz="0.01" />
+   </inertial>
+    <visual>
+		<origin xyz="0.0 0.0 0.0" />
+		<geometry>
+			<box size="0.0 0.0 0.0"/>
+		</geometry>
+    </visual>
+    <collision>
+		<origin xyz="0.0 0.0 0.0" />
+		<geometry>
+			<box size="0.25 0.15 0.175"/>
+		</geometry>
+    </collision>
+</link>
+<joint name="batterycovercollision_back_joint" type="fixed">
+    <parent link="base"/>
+    <child link="batterycovercollision_back"/>
+    <axis xyz="1 0 0"/>
+    <origin xyz="-0.25 0.0 0.125" rpy="0 0 1.5708"/>
+</joint>
 <xacro:my_link_texturedmesh name="torso" mass="16" texture="white">
    <origin xyz="0.0 0.0 0.0" rpy="0 0 0"/>

File: body_extra_visuals/body_extra.urdf.xacro (robot description, xacro)
@@ -1,22 +1,35 @@
 <?xml version="1.0"?>
 <robot xmlns:xacro="http://ros.org/wiki/xacro">
+<!--base plate-->
+<xacro:my_link_textured name="base_plate" mass="0" texture="aluminum">
+   <cylinder radius="0.333" length="0.02" />
+   <origin xyz="0.0 0.0 0.0" rpy="0 0 0"/>
+   <origin xyz="0.0 0.0 0.0" rpy="0 0 0" />
+   <inertia ixx="0"  ixy="0"  ixz="0" iyy="0" iyz="0" izz="0" />
+</xacro:my_link_textured>
+  <joint name="base_plate_joint" type="fixed">
+    <parent link="base_link"/>
+    <child link="base_plate"/>
+    <axis xyz="1 0 0"/>
+    <origin xyz="0.0 0.0 0.05" rpy="0 0 0"/>
+  </joint>
 <!--torso sliders-->
 <xacro:my_link_texturedmesh name="torso_assist_slider_right" mass="0.01" texture="aluminum">
    <origin xyz="0 0 0" rpy="0 0 0"/>
-   <origin xyz="-0.3  0.0 0.0" rpy="0 1.5708 0"/>
+   <origin xyz="-0.4  0.0 0.0" rpy="0 1.5708 0"/>
    <inertia ixx="0.01"  ixy="0"  ixz="0" iyy="0.01" iyz="0" izz="0.01" />
-   <mesh filename="package://amigo_robot_model/body_extra_visuals/torsoassistslidertextured.dae" scale="0.01 0.01 0.01"/>
+   <mesh filename="package://amigo_robot_model/body_extra_visuals/torsoassistslidertextured.dae" scale="0.01 0.01 0.0125"/>
 </xacro:my_link_texturedmesh>
 <xacro:my_link_texturedmesh name="torso_assist_slider_left" mass="0.01" texture="aluminum">
    <origin xyz="0 0 0" rpy="0 0 0"/>
-   <origin xyz="-0.3  0.0 0.0" rpy="0 1.5708 0"/>
+   <origin xyz="-0.4  0.0 0.0" rpy="0 1.5708 0"/>
    <inertia ixx="0.01"  ixy="0"  ixz="0" iyy="0.01" iyz="0" izz="0.01" />
-   <mesh filename="package://amigo_robot_model/body_extra_visuals/torsoassistslidertextured.dae" scale="0.01 0.01 0.01"/>
+   <mesh filename="package://amigo_robot_model/body_extra_visuals/torsoassistslidertextured.dae" scale="0.01 0.01 0.0125"/>
 </xacro:my_link_texturedmesh>
 <xacro:my_link_texturedmesh name="torso_assist_slider_back" mass="0.01" texture="aluminum">
    <origin xyz="0 0 0" rpy="0 0 0"/>
-   <origin xyz="-0.3 0.0 0.0" rpy="0 1.5708 0"/>
+   <origin xyz="-0.4 0.0 0.0" rpy="0 1.5708 0"/>
    <inertia ixx="0.01"  ixy="0"  ixz="0" iyy="0.01" iyz="0" izz="0.01" />
-   <mesh filename="package://amigo_robot_model/body_extra_visuals/torsoassistslidertextured.dae" scale="0.01 0.01 0.01"/>
+   <mesh filename="package://amigo_robot_model/body_extra_visuals/torsoassistslidertextured.dae" scale="0.01 0.01 0.0125"/>
 </xacro:my_link_texturedmesh>
 <joint name="torso_slider_assist_joint_right" type="fixed">

File: definitions.xacro (robot description, xacro)
@@ -26,4 +26,31 @@
 <gazebo reference="${name}">
       <material>Gazebo/${color}</material>
+      <turnGravityOff>false</turnGravityOff>
+    </gazebo>
+</xacro:macro>
+<xacro:macro name="my_link_textured" params="name mass texture *type *origin *visualorigin *inertia">
+  <link name="${name}">
+   <inertial>
+     <xacro:insert_block name="origin" />
+     <mass value="${mass}"/>
+     <xacro:insert_block name="inertia" />
+   </inertial>
+   <visual>
+     <xacro:insert_block name="visualorigin" />
+     <geometry>
+     <xacro:insert_block name="type" />
+     </geometry>
+     <material name="${texture}">
+     </material>
+    </visual>
+    <collision>
+     <xacro:insert_block name="visualorigin" />
+     <geometry>
+     <xacro:insert_block name="type" />
+     </geometry>
+    </collision>
+  </link>
+<gazebo reference="${name}">
+      <material>amigo_robot_model/${texture}</material>
       <turnGravityOff>false</turnGravityOff>
     </gazebo>
@@ -103,5 +130,5 @@
     </gazebo>
 </xacro:macro>
-<xacro:macro name="my_link_texturedmesh_diff_coll" params="name mass texture *origin *visualorigin *inertia *mesh *type">
+<xacro:macro name="my_link_texturedmesh_diff_coll" params="name mass texture *origin *visualorigin *collorigin *inertia *mesh *type">
   <link name="${name}">
    <inertial>
@@ -118,5 +145,5 @@
     </visual>
     <collision>
-     <xacro:insert_block name="visualorigin" />
+     <xacro:insert_block name="collorigin" />
      <geometry>
      <xacro:insert_block name="type" />

File: laser/laser.urdf.xacro (robot description, xacro)
@@ -4,5 +4,5 @@
    <box size="0.05 0.065 0.12" /> <!--*-->
    <origin xyz="0.0 0.0 0.0" rpy="0 0 0"/>
-   <origin xyz="-0.005 0.0 -0.0525" rpy="0 0 0" />
+   <origin xyz="-0.005 0.0 -0.065" rpy="0 0 0" />
    <inertia ixx="0.0001"  ixy="0"  ixz="0" iyy="0.0001" iyz="0" izz="0.0001" /> <!--*-->
 </xacro:my_link>
@@ -13,4 +13,14 @@
    <limit effort="13.4" velocity="1.0" lower="-0.7809" upper="1.5708" />
 </xacro:my_joint>
+<xacro:my_link_textured name="lasertop" mass="0.01" texture="Orange">
+   <box size="0.05 0.065 0.01" /> <!--*-->
+   <origin xyz="0.0 0.0 0.0" rpy="0 0 0"/>
+   <origin xyz="-0.005 0.0 0.0" rpy="0 0 0" />
+   <inertia ixx="0.0001"  ixy="0"  ixz="0" iyy="0.0001" iyz="0" izz="0.0001" /> <!--*-->
+</xacro:my_link_textured>
+<joint name="lasertop_joint" type="fixed">
+    <parent link="base_laser"/>
+    <child link="lasertop"/>
+</joint>
 <xacro:my_link_texturedmesh name="logo" mass="0.01" texture="logo">
    <origin xyz="0.0 0.0 0.0" rpy="0 0 0"/>

File: materials.urdf.xacro (robot description, xacro)
@@ -1,4 +1,7 @@
 <?xml version="1.0"?>
 <robot>
+  <material name="Orange">
+    <color rgba="1.0 0.45 0.0 1.0"/>
+  </material>
   <material name="Blue">
     <color rgba="0.0 0.0 0.8 1.0"/>
