Commit message: Updated urdf
git-svn-id: https://roboticssrv.wtb.tue.nl/svn/ros/code/tue-ros-pkg/trunk/tue_robot_models/amigo_robot_model@6924 3a3c2cfb-d3b9-409e-9e75-db8fcdbcaac6

File: body_extra_visuals/body_extra.urdf.xacro (robot description, xacro)
@@ -2,9 +2,9 @@
 <robot xmlns:xacro="http://ros.org/wiki/xacro">
 <!--base plate-->
-<xacro:my_link_textured name="base_plate" mass="0" texture="aluminum">
+<xacro:my_link_textured name="base_plate" mass="0.1" texture="aluminum">
    <cylinder radius="0.333" length="0.02" />
    <origin xyz="0.0 0.0 0.0" rpy="0 0 0"/>
    <origin xyz="0.0 0.0 0.0" rpy="0 0 0" />
-   <inertia ixx="0"  ixy="0"  ixz="0" iyy="0" iyz="0" izz="0" />
+   <inertia ixx="0.01"  ixy="0"  ixz="0" iyy="0.01" iyz="0" izz="0.01" />
 </xacro:my_link_textured>
   <joint name="base_plate_joint" type="fixed">
