Commit message: lasertop is now orange in gazebo aswell
git-svn-id: https://roboticssrv.wtb.tue.nl/svn/ros/code/tue-ros-pkg/trunk/tue_robot_models/amigo_robot_model@7013 3a3c2cfb-d3b9-409e-9e75-db8fcdbcaac6

File: laser/laser.urdf.xacro (robot description, xacro)
@@ -13,5 +13,5 @@
    <limit effort="13.4" velocity="1.0" lower="-0.7809" upper="1.5708" />
 </xacro:my_joint>
-<xacro:my_link_textured name="lasertop" mass="0.01" texture="Orange">
+<xacro:my_link_textured name="lasertop" mass="0.01" texture="orange">
    <box size="0.05 0.065 0.01" /> <!--*-->
    <origin xyz="0.0 0.0 0.0" rpy="0 0 0"/>

File: materials.urdf.xacro (robot description, xacro)
@@ -1,7 +1,4 @@
 <?xml version="1.0"?>
 <robot>
-  <material name="Orange">
-    <color rgba="1.0 0.45 0.0 1.0"/>
-  </material>
   <material name="Blue">
     <color rgba="0.0 0.0 0.8 1.0"/>
@@ -40,3 +37,6 @@
     <texture filename="package://amigo_robot_model/Media/materials/textures/aluminum/aluminium_0001_c.jpg" />
   </material>
+  <material name="orange">
+    <texture filename="package://amigo_robot_model/Media/materials/textures/orange/orange.jpg" />
+  </material>
 </robot>
