Commit message: Reverted wheel diameter
git-svn-id: https://roboticssrv.wtb.tue.nl/svn/ros/code/tue-ros-pkg/trunk/tue_robot_models/amigo_robot_model@6905 3a3c2cfb-d3b9-409e-9e75-db8fcdbcaac6

File: wheels/wheels.urdf.xacro (robot description, xacro)
@@ -7,5 +7,5 @@
     <child link="wheel_${side_LR}_${side_FR}"/>
     <axis xyz="1 0 0"/>
-    <origin xyz="${sign_LR}0.205 ${sign_FR}0.205 0.005" rpy="0 0 ${wheel_angle}"/>
+    <origin xyz="${sign_LR}0.2 ${sign_FR}0.2 0.005" rpy="0 0 ${wheel_angle}"/>
     <dynamics damping="1" friction="0.0"/>
     <limit effort="5.0" velocity="5.0"/>

Commit message: Different wheels
git-svn-id: https://roboticssrv.wtb.tue.nl/svn/ros/code/tue-ros-pkg/trunk/tue_robot_models/amigo_robot_model@7024 3a3c2cfb-d3b9-409e-9e75-db8fcdbcaac6

File: wheels/wheels.urdf.xacro (robot description, xacro)
@@ -12,5 +12,5 @@
   </joint>
   <xacro:my_link name="wheel_${side_LR}_${side_FR}" mass="0.5" color="Grey">
-    <cylinder radius="0.05" length="0.05"/>
+    <cylinder radius="0.05" length="0.03"/>
     <origin xyz="0.0 0.0 0.0" rpy="0 0 0"/>
     <origin xyz="0.0 0.0 0.0" rpy="0 1.5708 0" />
@@ -28,5 +28,5 @@
 	</joint>
 	<xacro:my_link name="omni_sphere${number}_${side_LR}_${side_FR}" mass="0.05" color="Grey">
-		<sphere radius="0.03" />
+		<sphere radius="0.04" />
 		<origin xyz="0.0 0.0 0.0" rpy="0 0 0"/>
 		<origin xyz="0.0 0.0 0.0" rpy="0 0 0" />

Commit message: Revert to previous wheels
git-svn-id: https://roboticssrv.wtb.tue.nl/svn/ros/code/tue-ros-pkg/trunk/tue_robot_models/amigo_robot_model@7033 3a3c2cfb-d3b9-409e-9e75-db8fcdbcaac6

File: wheels/wheels.urdf.xacro (robot description, xacro)
@@ -12,5 +12,5 @@
   </joint>
   <xacro:my_link name="wheel_${side_LR}_${side_FR}" mass="0.5" color="Grey">
-    <cylinder radius="0.05" length="0.03"/>
+    <cylinder radius="0.05" length="0.05"/>
     <origin xyz="0.0 0.0 0.0" rpy="0 0 0"/>
     <origin xyz="0.0 0.0 0.0" rpy="0 1.5708 0" />
@@ -28,5 +28,5 @@
 	</joint>
 	<xacro:my_link name="omni_sphere${number}_${side_LR}_${side_FR}" mass="0.05" color="Grey">
-		<sphere radius="0.04" />
+		<sphere radius="0.03" />
 		<origin xyz="0.0 0.0 0.0" rpy="0 0 0"/>
 		<origin xyz="0.0 0.0 0.0" rpy="0 0 0" />
