Commit message: Commented Kinect collision box
git-svn-id: https://roboticssrv.wtb.tue.nl/svn/ros/code/tue-ros-pkg/trunk/tue_robot_models/amigo_robot_model@6662 3a3c2cfb-d3b9-409e-9e75-db8fcdbcaac6

File: kinect/kinect.urdf.xacro (robot description, xacro)
@@ -25,10 +25,10 @@
       </geometry>
     </visual>
-    <collision>
+    <!--<collision>
       <origin xyz="-0.0365 0.0 0.0" rpy="0 0 0" />
       <geometry>
         <box size="0.0730 .2760 0.0720"/>
       </geometry>
-    </collision>
+    </collision>-->
   </link>
   <joint name="kinect_depth_joint" type="fixed">

Commit message: Kinect box out of collision
git-svn-id: https://roboticssrv.wtb.tue.nl/svn/ros/code/tue-ros-pkg/trunk/tue_robot_models/amigo_robot_model@6909 3a3c2cfb-d3b9-409e-9e75-db8fcdbcaac6

File: kinect/kinect.urdf.xacro (robot description, xacro)
@@ -26,10 +26,10 @@
       </geometry>
     </visual>
-    <collision>
+    <!--<collision>
       <origin xyz="-0.0365 0.0 0.0" rpy="0 0 0" />
       <geometry>
         <box size="0.0730 .2760 0.0720"/>
       </geometry>
-    </collision>
+    </collision>-->
   </link>
   <joint name="kinect_depth_joint" type="fixed">

Commit message: new kinect distance
git-svn-id: https://roboticssrv.wtb.tue.nl/svn/ros/code/tue-ros-pkg/trunk/tue_robot_models/amigo_robot_model@7165 3a3c2cfb-d3b9-409e-9e75-db8fcdbcaac6

File: kinect/kinect.urdf.xacro (robot description, xacro)
@@ -6,5 +6,5 @@
   <property name="M_PI" value="3.14159"/>
   <joint name="base_kinect_joint" type="fixed">
-    <origin xyz="0.025 0 0.05" rpy="0 0 0" /> <!-- THESE VALUES ARE ROUGH ESTIMATES!! -->
+    <origin xyz="0.07 0 0.05" rpy="0 0 0" /> <!-- THESE VALUES ARE ROUGH ESTIMATES!! -->
     <parent link="head" />
     <child link="openni_camera" />

Commit message: dsfsd
git-svn-id: https://roboticssrv.wtb.tue.nl/svn/ros/code/tue-ros-pkg/trunk/tue_robot_models/amigo_robot_model@7167 3a3c2cfb-d3b9-409e-9e75-db8fcdbcaac6

File: kinect/kinect.urdf.xacro (robot description, xacro)
@@ -6,5 +6,5 @@
   <property name="M_PI" value="3.14159"/>
   <joint name="base_kinect_joint" type="fixed">
-    <origin xyz="0.07 0 0.05" rpy="0 0 0" /> <!-- THESE VALUES ARE ROUGH ESTIMATES!! -->
+    <origin xyz="0.1 0 0.1" rpy="0 0 0" /> <!-- THESE VALUES ARE ROUGH ESTIMATES!! -->
     <parent link="head" />
     <child link="openni_camera" />

Commit message: dsfds
git-svn-id: https://roboticssrv.wtb.tue.nl/svn/ros/code/tue-ros-pkg/trunk/tue_robot_models/amigo_robot_model@7168 3a3c2cfb-d3b9-409e-9e75-db8fcdbcaac6

File: kinect/kinect.urdf.xacro (robot description, xacro)
@@ -6,5 +6,5 @@
   <property name="M_PI" value="3.14159"/>
   <joint name="base_kinect_joint" type="fixed">
-    <origin xyz="0.1 0 0.1" rpy="0 0 0" /> <!-- THESE VALUES ARE ROUGH ESTIMATES!! -->
+    <origin xyz="0.07 0 0.07" rpy="0 0 0" /> <!-- THESE VALUES ARE ROUGH ESTIMATES!! -->
     <parent link="head" />
     <child link="openni_camera" />
