Commit message: Updated kinect urdf
git-svn-id: https://roboticssrv.wtb.tue.nl/svn/ros/code/tue-ros-pkg/trunk/tue_robot_models/amigo_robot_model@8291 3a3c2cfb-d3b9-409e-9e75-db8fcdbcaac6

File: kinect/base_kinect.urdf.xacro (robot description, xacro)
@@ -6,6 +6,6 @@
   <property name="M_PI" value="3.14159"/>
   <joint name="base_kinect_base_kinect_joint" type="fixed">
-    <origin xyz="0.1 0 0.1" rpy="0 0 0" /> <!-- THESE VALUES ARE ROUGH ESTIMATES!! -->
-    <parent link="base_laser" />
+    <origin xyz="0.29 0 0.31" rpy="0 -0.7854 0" /> <!-- THESE VALUES ARE ROUGH ESTIMATES!! -->
+    <parent link="base_link" />
     <child link="base_kinect_openni_camera" />
   </joint>

Commit message: Updated base_kinect position in URDF
git-svn-id: https://roboticssrv.wtb.tue.nl/svn/ros/code/tue-ros-pkg/trunk/tue_robot_models/amigo_robot_model@8307 3a3c2cfb-d3b9-409e-9e75-db8fcdbcaac6

File: kinect/base_kinect.urdf.xacro (robot description, xacro)
@@ -6,5 +6,5 @@
   <property name="M_PI" value="3.14159"/>
   <joint name="base_kinect_base_kinect_joint" type="fixed">
-    <origin xyz="0.29 0 0.31" rpy="0 -0.7854 0" /> <!-- THESE VALUES ARE ROUGH ESTIMATES!! -->
+    <origin xyz="0.29 0 0.31" rpy="0 0.1 0" /> <!-- THESE VALUES ARE ROUGH ESTIMATES!! -->
     <parent link="base_link" />
     <child link="base_kinect_openni_camera" />

Commit message: updated base kinect urdf
git-svn-id: https://roboticssrv.wtb.tue.nl/svn/ros/code/tue-ros-pkg/trunk/tue_robot_models/amigo_robot_model@8356 3a3c2cfb-d3b9-409e-9e75-db8fcdbcaac6

File: kinect/base_kinect.urdf.xacro (robot description, xacro)
@@ -6,5 +6,5 @@
   <property name="M_PI" value="3.14159"/>
   <joint name="base_kinect_base_kinect_joint" type="fixed">
-    <origin xyz="0.29 0 0.31" rpy="0 0.1 0" /> <!-- THESE VALUES ARE ROUGH ESTIMATES!! -->
+    <origin xyz="0.29 0 0.31" rpy="0 0 0" /> <!-- THESE VALUES ARE ROUGH ESTIMATES!! -->
     <parent link="base_link" />
     <child link="base_kinect_openni_camera" />

Commit message: calibrated base kinect
git-svn-id: https://roboticssrv.wtb.tue.nl/svn/ros/code/tue-ros-pkg/trunk/tue_robot_models/amigo_robot_model@8401 3a3c2cfb-d3b9-409e-9e75-db8fcdbcaac6

File: kinect/base_kinect.urdf.xacro (robot description, xacro)
@@ -6,5 +6,5 @@
   <property name="M_PI" value="3.14159"/>
   <joint name="base_kinect_base_kinect_joint" type="fixed">
-    <origin xyz="0.29 0 0.31" rpy="0 0 0" /> <!-- THESE VALUES ARE ROUGH ESTIMATES!! -->
+    <origin xyz="0.29 0 0.31" rpy="0 -0.03 0" /> <!-- THESE VALUES ARE ROUGH ESTIMATES!! -->
     <parent link="base_link" />
     <child link="base_kinect_openni_camera" />

Commit message: base kinect update
git-svn-id: https://roboticssrv.wtb.tue.nl/svn/ros/code/tue-ros-pkg/trunk/tue_robot_models/amigo_robot_model@8406 3a3c2cfb-d3b9-409e-9e75-db8fcdbcaac6

File: kinect/base_kinect.urdf.xacro (robot description, xacro)
@@ -6,5 +6,5 @@
   <property name="M_PI" value="3.14159"/>
   <joint name="base_kinect_base_kinect_joint" type="fixed">
-    <origin xyz="0.29 0 0.31" rpy="0 -0.03 0" /> <!-- THESE VALUES ARE ROUGH ESTIMATES!! -->
+    <origin xyz="0.29 0 0.31" rpy="0 -0.07 0" /> <!-- THESE VALUES ARE ROUGH ESTIMATES!! -->
     <parent link="base_link" />
     <child link="base_kinect_openni_camera" />
