Commit message: Violation constriaint temporily resolved
git-svn-id: https://roboticssrv.wtb.tue.nl/svn/ros/code/tue-ros-pkg/trunk/tue_robot_models/amigo_robot_model@6658 3a3c2cfb-d3b9-409e-9e75-db8fcdbcaac6

File: arms_DH/armDH.urdf.xacro (robot description, xacro)
@@ -85,5 +85,6 @@
    <dynamics damping="6.0" friction="4.87"/>
    <axis xyz="0 -1 0"/>
-   <limit effort="13.4" velocity="1.0" lower="-1.5708" upper="0.0" />
+   <!--<limit effort="13.4" velocity="1.0" lower="-1.5708" upper="0.0" /> -->
+   <limit effort="13.4" velocity="1.0" lower="-1.5708" upper="0.01" />
 </xacro:my_joint>
 <xacro:my_joint name="shoulder_pitch_joint_${whichside}" type="revolute" parent="shoulder_link1_${whichside}" child="shoulder_link2_${whichside}">

Commit message: Cleanup code
git-svn-id: https://roboticssrv.wtb.tue.nl/svn/ros/code/tue-ros-pkg/trunk/tue_robot_models/amigo_robot_model@6697 3a3c2cfb-d3b9-409e-9e75-db8fcdbcaac6

File: arms_DH/armDH.urdf.xacro (robot description, xacro)
@@ -32,13 +32,6 @@
 <xacro:my_link name="fore_arm_${whichside}" mass="0.8" color="Grey">
    <box size="0.065 0.065 0.28"/>
-<!--
-   <cylinder radius="0.0325" length="0.28"/>
--->
-      <origin xyz="0.0 -0.14 0.0" rpy="0.0 0 0"/>
+   <origin xyz="0.0 -0.14 0.0" rpy="0.0 0 0"/>
    <origin xyz="0.0 -0.14 0.0" rpy="1.5708 0 0" />
-<!--
-   <origin xyz="0.0 -0.14 0.0" rpy="0 0 0"/>
-   <origin xyz="0.0 -0.14 0.0" rpy="1.5708 0 0" />
--->
    <inertia ixx="0.0054"  ixy="0"  ixz="0" iyy="0.0054" iyz="0" izz="0.0004" />
    <color rgba="0.65 0.65 0.65 1.0"/>
@@ -72,5 +65,4 @@
    <color rgba="0.15 0.15 0.15 1.0"/>
 </xacro:my_link>
-<!--<link name="grippoint_${whichside}" />-->
 <xacro:my_link name="grippoint_${whichside}" mass="0.01" color="Blue">
    <box size="0.01 0.01 0.01"/>
@@ -85,6 +77,5 @@
    <dynamics damping="6.0" friction="4.87"/>
    <axis xyz="0 -1 0"/>
-   <!--<limit effort="13.4" velocity="1.0" lower="-1.5708" upper="0.0" /> -->
-   <limit effort="13.4" velocity="1.0" lower="-1.5708" upper="0.01" />
+   <limit effort="13.4" velocity="1.0" lower="-1.5708" upper="0.001" />
 </xacro:my_joint>
 <xacro:my_joint name="shoulder_pitch_joint_${whichside}" type="revolute" parent="shoulder_link1_${whichside}" child="shoulder_link2_${whichside}">

Commit message: NEW ROBOT MODEL!!!
git-svn-id: https://roboticssrv.wtb.tue.nl/svn/ros/code/tue-ros-pkg/trunk/tue_robot_models/amigo_robot_model@6876 3a3c2cfb-d3b9-409e-9e75-db8fcdbcaac6

File: arms_DH/armDH.urdf.xacro (robot description, xacro)
@@ -1,67 +1,68 @@
-<robot xmlns:xacro="http://ros.org/wiki/xacro">
+<?xml version="1.0"?>
+<robot 	xmlns:xacro="http://ros.org/wiki/xacro"
+	xmlns:sensor="http://playerstage.sourceforge.net/gazebo/xmlschema/#sensor"
+	xmlns:controller="http://playerstage.sourceforge.net/gazebo/xmlschema/#controller"
+	xmlns:interface="http://playerstage.sourceforge.net/gazebo/xmlschema/#interface">
 <!--Fill out Link macros-->
-<xacro:macro name="arm" params="whichside sidesign orientationsign rolloffset">
-<xacro:my_link name="shoulder_link1_${whichside}" mass="0.1" color="Blue">
-   <cylinder radius="0.04" length="0.105" />
+<xacro:macro name="arm" params="whichside sidesign rollsign">
+<xacro:my_link name="shoulder_mount_${whichside}" mass="0.1" color="Black">
+   <cylinder radius="0.05" length="0.11" />
    <origin xyz="0.0 0.0 0.0" rpy="0 0 0"/>
    <origin xyz="0.0 0.0 0.0" rpy="0 0 0 " />
    <inertia ixx="0.01"  ixy="0"  ixz="0" iyy="0.01" iyz="0" izz="0.01" />
-   <color rgba="0.25 0.25 0.25 1.0"/>
 </xacro:my_link>
-<xacro:my_link name="shoulder_link2_${whichside}" mass="0.1" color="Red">
-   <cylinder radius="0.01" length="0.01" />
+<xacro:my_link name="shoulder_link1_${whichside}" mass="0.1" color="Black">
+   <cylinder radius="0.045" length="0.015" />
    <origin xyz="0.0 0.0 0.0" rpy="0 0 0"/>
-   <origin xyz="0.0 0.0 0.0" rpy="0 0 0" />
+   <origin xyz="0.0 0.0 ${sidesign *0.0525}" rpy="0 0 0 " />
+   <inertia ixx="0.01"  ixy="0"  ixz="0" iyy="0.01" iyz="0" izz="0.01" />
+</xacro:my_link>
+<xacro:my_link name="shoulder_link2_${whichside}" mass="0.1" color="Black">
+   <box size="0.035 0.01 0.1" />
+   <origin xyz="0.0 0.0 0.0" rpy="0 0 0"/>
+   <origin xyz="0.0 ${-sidesign*0.06} -0.05" rpy="0 0 0" />
    <inertia ixx="0.001"  ixy="0"  ixz="0" iyy="0.001" iyz="0" izz="0.001" />
-   <color rgba="0 0 1 1.0"/>
 </xacro:my_link>
-<xacro:my_link name="upper_arm_${whichside}" mass="2.9" color="Grey">
-   <cylinder radius="0.0525" length="0.32"/>
-   <origin xyz="0.0 -0.16 0.0" rpy="0 0 0"/>
-   <origin xyz="0.0 -0.16 0.0" rpy="1.5708 0 0" />
+<xacro:my_link_texturedmesh name="upper_arm_${whichside}" mass="2.9" texture="torsocovers">
+   <origin xyz="0.0 -0.2 0.0" rpy="0 0 0"/>
+   <origin xyz="0.0 -0.2 0.0" rpy="0 0 3.1415" />
    <inertia ixx="0.027"  ixy="0"  ixz="0" iyy="0.027" iyz="0" izz="0.004" />
-   <color rgba="0.65 0.65 0.65 1.0"/>
+   <mesh filename="package://amigo_robot_model/arms_DH/upperarmtextured.dae" scale="0.001 0.001 0.001"/>
+</xacro:my_link_texturedmesh>
+<xacro:my_link name="elbow_link4_${whichside}" mass="0.1" color="Grey">
+   <cylinder radius="0.025" length="0.08"/>
+   <origin xyz="0.0 0.0 0.0" rpy="0 0 0"/>
+   <origin xyz="-0.017 0.0 0.015" rpy="1.5708 0 0" />
+   <inertia ixx="0.001"  ixy="0"  ixz="0" iyy="0.001" iyz="0" izz="0.001" />
 </xacro:my_link>
-<xacro:my_link name="elbow_link4_${whichside}" mass="0.1" color="Blue">
-   <cylinder radius="0.03" length="0.10"/>
+<xacro:my_link_texturedmesh name="fore_arm_${whichside}" mass="0.1" texture="torsocovers">
+   <origin xyz="0.0 -0.14 0.0" rpy="0.0 0 0"/>
+   <origin xyz="0.0 -0.14 0.0" rpy="0 -1.5708 0" />
+   <inertia ixx="0.0054"  ixy="0"  ixz="0" iyy="0.0054" iyz="0" izz="0.0004" />
+   <mesh filename="package://amigo_robot_model/arms_DH/forearmtextured.dae" scale="0.001 0.001 0.001"/>
+</xacro:my_link_texturedmesh>
+<xacro:my_link name="wrist_link6_${whichside}" mass="0.01" color="Black">
+   <cylinder radius="0.018" length="0.06"/>
    <origin xyz="0.0 0.0 0.0" rpy="0 0 0"/>
-   <origin xyz="0.0 0.0 0.0" rpy="1.5708 0 0" />
+   <origin xyz="0.0 0.0 -0.034" rpy="1.5708 0 0" />
    <inertia ixx="0.001"  ixy="0"  ixz="0" iyy="0.001" iyz="0" izz="0.001" />
-   <color rgba="0.25 0.25 0.25 1.0"/>
 </xacro:my_link>
-<xacro:my_link name="fore_arm_${whichside}" mass="0.8" color="Grey">
-   <box size="0.065 0.065 0.28"/>
-   <origin xyz="0.0 -0.14 0.0" rpy="0.0 0 0"/>
-   <origin xyz="0.0 -0.14 0.0" rpy="1.5708 0 0" />
-   <inertia ixx="0.0054"  ixy="0"  ixz="0" iyy="0.0054" iyz="0" izz="0.0004" />
-   <color rgba="0.65 0.65 0.65 1.0"/>
-</xacro:my_link>
-<xacro:my_link name="wrist_link6_${whichside}" mass="0.01" color="Blue">
-   <cylinder radius="0.02" length="0.09"/>
-   <origin xyz="0.0 0.0 0.0" rpy="0 0 0"/>
-   <origin xyz="0.0 0.0 0.0" rpy="1.5708 0 0" />
-   <inertia ixx="0.001"  ixy="0"  ixz="0" iyy="0.001" iyz="0" izz="0.001" />
-   <color rgba="0.25 0.25 0.25 1.0"/>
-</xacro:my_link>
-<xacro:my_link name="hand_${whichside}" mass="0.2" color="Red">
+<xacro:my_link name="hand_${whichside}" mass="0.2" color="Grey">
    <box size="0.080 0.085 0.038"/>
-   <origin xyz="0.0425 0.0 0.0" rpy="0 0 0"/>
-   <origin xyz="0.0425 0.0 0.0" rpy="0 0 0" />
+   <origin xyz="0.048 0.0 0.0" rpy="0 0 0"/>
+   <origin xyz="0.048 0.0 -0.034" rpy="0 0 0" />
    <inertia ixx="0.01"  ixy="0"  ixz="0" iyy="0.01" iyz="0" izz="0.01" />
-   <color rgba="0 0 1 1.0"/>
 </xacro:my_link>
 <xacro:my_link name="finger1_${whichside}" mass="0.05" color="Black">
    <box size="0.02 0.022 0.11"/>
    <origin xyz="0.0 0.0 -0.055" rpy="0 0 0"/>
-   <origin xyz="0.0 0.0 -0.055" rpy="0 0 0" />
+   <origin xyz="-0.034 0.0 -0.055" rpy="0 0 0" />
    <inertia ixx="0.00037"  ixy="0"  ixz="0" iyy="0.00052" iyz="0" izz="0.00052" />
-   <color rgba="0.15 0.15 0.15 1.0"/>
 </xacro:my_link>
 <xacro:my_link name="finger2_${whichside}" mass="0.05" color="Black">
    <box size="0.02 0.022 0.11"/>
    <origin xyz="0.0 0.0 -0.055" rpy="0 0 0"/>
-   <origin xyz="0.0 0.0 -0.055" rpy="0 0 0" />
+   <origin xyz="-0.034 0.0 -0.055" rpy="0 0 0" />
    <inertia ixx="0.00037"  ixy="0"  ixz="0" iyy="0.00052" iyz="0" izz="0.00052" />
-   <color rgba="0.15 0.15 0.15 1.0"/>
 </xacro:my_link>
 <xacro:my_link name="grippoint_${whichside}" mass="0.01" color="Blue">
@@ -70,12 +71,16 @@
    <origin xyz="-0.1 0.0 0.0" rpy="0 0 0 " />
    <inertia ixx="0.0001"  ixy="0"  ixz="0" iyy="0.0001" iyz="0" izz="0.0001" />
-   <color rgba="0.25 0.25 0.25 1.0"/>
 </xacro:my_link>
 <!--Fill out Joint macros-->
-<xacro:my_joint name="shoulder_yaw_joint_${whichside}" type="revolute" parent="torso" child="shoulder_link1_${whichside}">
-   <origin xyz="0.05 ${sidesign}0.202  0.0" rpy="${orientationsign} 0 0"/>
+  <joint name="shoulder_mount_joint_${whichside}" type="fixed">
+    <parent link="torso"/>
+    <child link="shoulder_mount_${whichside}"/>
+    <origin xyz="0.05 ${sidesign*0.22} 0.0" rpy="0 0 0.0"/>
+  </joint>
+<xacro:my_joint name="shoulder_yaw_joint_${whichside}" type="revolute" parent="shoulder_mount_${whichside}" child="shoulder_link1_${whichside}">
+   <origin xyz="0 0 0" rpy="-1.5708 -1.5708 0"/>
    <dynamics damping="6.0" friction="4.87"/>
-   <axis xyz="0 -1 0"/>
-   <limit effort="13.4" velocity="1.0" lower="-1.5708" upper="0.001" />
+   <axis xyz="${rollsign}1 0 0"/>
+   <limit effort="13.4" velocity="1.0" lower="-1.5708" upper="1e-3" />
 </xacro:my_joint>
 <xacro:my_joint name="shoulder_pitch_joint_${whichside}" type="revolute" parent="shoulder_link1_${whichside}" child="shoulder_link2_${whichside}">
@@ -83,10 +88,10 @@
    <dynamics damping="6.0" friction="6.06"/>
    <axis xyz="0 -1 0"/>
-   <limit effort="13.4" velocity="1.0" lower="-3.1415" upper="0" />
+   <limit effort="13.4" velocity="1.0" lower="-1.5708" upper="1.5708" />
 </xacro:my_joint>
 <xacro:my_joint name="shoulder_roll_joint_${whichside}" type="revolute" parent="shoulder_link2_${whichside}" child="upper_arm_${whichside}">
-   <origin xyz="0.0 0.0 0.0" rpy="1.5708 0 ${rolloffset}"/>
+   <origin xyz="0.0 0.0 0.0" rpy="1.5708 0 0.0"/>
    <dynamics damping="6.0" friction="2.16"/>
-   <axis xyz="0 1 0"/>
+   <axis xyz="0 ${sidesign} 0"/>
    <limit effort="9.8" velocity="1.0" lower="-1.5708" upper="1.5708"/>
 </xacro:my_joint>
@@ -95,23 +100,23 @@
    <dynamics damping="2.5" friction="1.18"/>
    <axis xyz="0 -1 0"/>
-   <limit effort="4.5" velocity="1.0" lower="0.0" upper="1.98" />
+   <limit effort="4.5" velocity="1.0" lower="0.0" upper="2.5307" />
 </xacro:my_joint>
 <xacro:my_joint name="elbow_roll_joint_${whichside}" type="revolute" parent="elbow_link4_${whichside}" child="fore_arm_${whichside}">
    <origin xyz="0.0 0.0 0.0" rpy="1.5708 0 0"/>
    <dynamics damping="2.5" friction="1.35"/>
-   <axis xyz="0 1 0"/>
-   <limit effort="4.5" velocity="1.0" lower="-1.83" upper="1.83"/>
+   <axis xyz="0 ${sidesign} 0"/>
+   <limit effort="4.5" velocity="1.0" lower="-1.8326" upper="1.8326"/>
 </xacro:my_joint>
 <xacro:my_joint name="wrist_pitch_joint_${whichside}" type="revolute" parent="fore_arm_${whichside}" child="wrist_link6_${whichside}">
-   <origin xyz="0.01 -0.28 0.0" rpy="-1.5708 0 0"/>
+   <origin xyz="0.01 -0.28 0.0" rpy="-1.5708 0 -1.5708"/>
    <dynamics damping="0.5" friction="0.63"/>
    <axis xyz="0 -1 0"/>
-   <limit effort="1" velocity="1.0" lower="-2.52" upper="-0.62"/>
+   <limit effort="1" velocity="1.0" lower="-0.9940" upper="0.9940"/>
 </xacro:my_joint>
 <xacro:my_joint name="wrist_yaw_joint_${whichside}" type="revolute" parent="wrist_link6_${whichside}" child="hand_${whichside}">
    <origin xyz="0.0 0.0 0.0" rpy="0 0 0"/>
    <dynamics damping="0.5" friction="0.68"/>
-   <axis xyz="0 0 1"/>
-   <limit effort="1" velocity="1.0" lower="-0.70" upper="0.70"/>
+   <axis xyz="0 0 ${sidesign}1"/>
+   <limit effort="1" velocity="1.0" lower="-0.7854" upper="0.7854"/>
 </xacro:my_joint>
 <xacro:my_joint name="finger1_joint_${whichside}" type="revolute" parent="hand_${whichside}" child="finger1_${whichside}">
@@ -130,6 +135,5 @@
     <parent link="hand_${whichside}"/>
     <child link="grippoint_${whichside}"/>
-    <axis xyz="0  0 1"/>
-    <origin xyz="0.14 0.0 0.0" rpy="  0.0 0.0 0.0"/>
+    <origin xyz="0.14 0.0 0.0" rpy="0 0 0"/>
   </joint>
 </xacro:macro>

File: body/body.urdf.xacro (robot description, xacro)
@@ -2,39 +2,34 @@
 <robot xmlns:xacro="http://ros.org/wiki/xacro">
 <!--body-->
-<xacro:my_link name="base" mass="20" color="Red">
-   <box size="0.2 0.2 0.655" /> <!--*-->
+<xacro:my_link_texturedmesh_diff_coll name="base" mass="20" texture="bottomcovers">
+   <origin xyz="0.0 0.0 0.3275" rpy="0 0 0"/>
+   <origin xyz="0.0 0.0 0.3275" rpy="0 0 -1.5708" />
+   <inertia ixx="2.63"  ixy="0"  ixz="0" iyy="2.63" iyz="0" izz="2.4" /> <!--*-->
+   <mesh filename="package://amigo_robot_model/body/onderkantversiekrisreducedtextured.dae" scale="0.001 0.001 0.001"/>
+   <box size="0.25 0.25 0.5"/>
+</xacro:my_link_texturedmesh_diff_coll>
+<xacro:my_link name="torso_slider" mass="0.1" color="Grey">
+   <cylinder radius="0.024" length="0.6" />
+   <origin xyz="0 0 0" rpy="0 0 0"/>
+   <origin xyz="0.0 0.0 0.0" rpy="0 1.5708 0"/>
+   <inertia ixx="0.01"  ixy="0"  ixz="0" iyy="0.01" iyz="0" izz="0.01" />
+</xacro:my_link>
+<xacro:my_link name="base_link" mass="0" color="Red">
+   <cylinder radius="0.0" length="0.00" />
    <origin xyz="0.0 0.0 0.0" rpy="0 0 0"/>
    <origin xyz="0.0 0.0 0.0" rpy="0 0 0" />
-   <inertia ixx="2.63"  ixy="0"  ixz="0" iyy="2.63" iyz="0" izz="2.4" /> <!--*-->
-   <color rgba="0.5 0.5 0.5  1.0"/>
+   <inertia ixx="0"  ixy="0"  ixz="0" iyy="0" iyz="0" izz="0" />
 </xacro:my_link>
-<xacro:my_link name="torso_slider" mass="0.1" color="Red">
-   <box size="0.2 0.2 0.655" /> <!--*-->
+<xacro:my_link_texturedmesh name="torso" mass="16" texture="torsocovers">
    <origin xyz="0.0 0.0 0.0" rpy="0 0 0"/>
-   <origin xyz="0.0 0.0 0.0" rpy="0 0 0" />
-   <inertia ixx="0.1"  ixy="0"  ixz="0" iyy="0.1" iyz="0" izz="0.1" /> <!--*-->
-   <color rgba="0.5 0.5 0.5  1.0"/>
-</xacro:my_link>
-<xacro:my_link name="base_link" mass="20" color="Red">
-   <cylinder radius="0.35" length="0.05" />
-   <!--<box size="0.45 0.45 0.05" /> -->
-   <origin xyz="0.0 0.0 0.0" rpy="0 0 0"/>
-   <origin xyz="0.0 0.0 0.0" rpy="0 0 0" />
-   <inertia ixx="0.001"  ixy="0"  ixz="0" iyy="0.001" iyz="0" izz="0.001" /> <!--*-->
-   <color rgba="0.5 0.5 0.5  1.0"/>
-</xacro:my_link>
-<!---->
-<xacro:my_link name="torso" mass="16" color="Green"> <!--*-->
-   <box size="0.2  0.387 0.097   "/> <!--*-->
-   <origin xyz="0.0475 0.0 0.0" rpy="0 0 0"/>
-   <origin xyz="0.0475 0.0 0.0" rpy="1.5708 1.5708 1.5708" />
+   <origin xyz="0.045 0.0 0.06" rpy="-1.5708 0 -1.5708" />
    <inertia ixx="0.01"  ixy="0"  ixz="0" iyy="0.01" iyz="0" izz="0.01" /> <!--*-->
-   <color rgba="0.4 0.4 0.4 1.0"/>
-</xacro:my_link>
+   <mesh filename="package://amigo_robot_model/body/torsocovers.dae" scale="0.001 0.001 0.001"/>
+</xacro:my_link_texturedmesh>
   <joint name="spindle_joint" type="prismatic">
     <parent link="base"/>
-    <child link="torso"/>
+    <child link="torso_slider"/>
     <axis xyz="1 0 0"/>
-    <origin xyz="0.0 0.0 0.3325" rpy="3.14159265 -1.5708 0"/>
+    <origin xyz="0.0 0.0 0.58" rpy="3.14159265 -1.5708 0"/>
     <dynamics damping="3" friction="0.0"/> <!--*-->
     <limit effort="30" velocity="1.0" lower="0.0" upper="0.41" /> <!--*-->
@@ -44,11 +39,11 @@
     <child link="base"/>
     <axis xyz="1 0 0"/>
-    <origin xyz="0.0 0.0 0.3475" rpy="0 0 0"/>
+    <origin xyz="0.0 0.0 0.055" rpy="0 0 0"/>
   </joint>
     <joint name="torso_slider_joint" type="fixed">
-    <parent link="torso"/>
-    <child link="torso_slider"/>
+    <parent link="torso_slider"/>
+    <child link="torso"/>
     <axis xyz="1 0 0"/>
-    <origin xyz="  -0.33 0.0 0.0" rpy="0 1.57 0"/>
+    <origin xyz="0.135 0.0 0.0" rpy="0 0 0"/>
   </joint>
 </robot>

File: definitions.xacro (robot description, xacro)
@@ -2,5 +2,5 @@
 <robot xmlns:xacro="http://ros.org/wiki/xacro">
 <!-- *************** LINK Definition *****************-->
-<xacro:macro name="my_link" params="name mass color *type *origin *visualorigin *inertia *color">
+<xacro:macro name="my_link" params="name mass color *type *origin *visualorigin *inertia">
   <link name="${name}">
    <inertial>
@@ -15,5 +15,4 @@
      </geometry>
      <material name="${color}">
-     <xacro:insert_block name="color" />
      </material>
     </visual>
@@ -30,5 +29,5 @@
     </gazebo>
 </xacro:macro>
-<xacro:macro name="my_link_coll_free" params="name mass color *type *origin *visualorigin *inertia *color">
+<xacro:macro name="my_link_coll_free" params="name mass color *type *origin *visualorigin *inertia">
   <link name="${name}">
    <inertial>
@@ -43,5 +42,4 @@
      </geometry>
      <material name="${color}">
-     <xacro:insert_block name="color" />
      </material>
     </visual>
@@ -49,4 +47,83 @@
 <gazebo reference="${name}">
       <material>Gazebo/${color}</material>
+      <turnGravityOff>false</turnGravityOff>
+    </gazebo>
+</xacro:macro>
+<xacro:macro name="my_link_mesh" params="name mass color *origin *visualorigin *inertia *mesh">
+  <link name="${name}">
+   <inertial>
+     <xacro:insert_block name="origin" />
+     <mass value="${mass}"/>
+     <xacro:insert_block name="inertia" />
+   </inertial>
+   <visual>
+     <xacro:insert_block name="visualorigin" />
+     <geometry>
+     <xacro:insert_block name="mesh" />
+     </geometry>
+     <material name="${color}">
+     </material>
+    </visual>
+    <collision>
+     <xacro:insert_block name="visualorigin" />
+     <geometry>
+     <xacro:insert_block name="mesh" />
+     </geometry>
+    </collision>
+  </link>
+<gazebo reference="${name}">
+      <material>Gazebo/${color}</material>
+      <turnGravityOff>false</turnGravityOff>
+    </gazebo>
+</xacro:macro>
+<xacro:macro name="my_link_texturedmesh" params="name mass texture *origin *visualorigin *inertia *mesh">
+  <link name="${name}">
+   <inertial>
+     <xacro:insert_block name="origin" />
+     <mass value="${mass}"/>
+     <xacro:insert_block name="inertia" />
+   </inertial>
+   <visual>
+     <xacro:insert_block name="visualorigin" />
+     <geometry>
+     <xacro:insert_block name="mesh" />
+     </geometry>
+     <material name="${texture}"/>
+    </visual>
+    <collision>
+     <xacro:insert_block name="visualorigin" />
+     <geometry>
+     <xacro:insert_block name="mesh" />
+     </geometry>
+    </collision>
+  </link>
+<gazebo reference="${name}">
+	  <material>amigo_robot_model/${texture}</material>
+      <turnGravityOff>false</turnGravityOff>
+    </gazebo>
+</xacro:macro>
+<xacro:macro name="my_link_texturedmesh_diff_coll" params="name mass texture *origin *visualorigin *inertia *mesh *type">
+  <link name="${name}">
+   <inertial>
+     <xacro:insert_block name="origin" />
+     <mass value="${mass}"/>
+     <xacro:insert_block name="inertia" />
+   </inertial>
+   <visual>
+     <xacro:insert_block name="visualorigin" />
+     <geometry>
+     <xacro:insert_block name="mesh" />
+     </geometry>
+     <material name="${texture}"/>
+    </visual>
+    <collision>
+     <xacro:insert_block name="visualorigin" />
+     <geometry>
+     <xacro:insert_block name="type" />
+     </geometry>
+    </collision>
+  </link>
+<gazebo reference="${name}">
+	  <material>amigo_robot_model/${texture}</material>
       <turnGravityOff>false</turnGravityOff>
     </gazebo>

File: gazebo/gazebo.urdf.xacro (robot description, xacro)
@@ -128,7 +128,7 @@
         <alwaysOn>true</alwaysOn>
         <updateRate>20</updateRate>
-        <imageTopicName>/camera/image_raw</imageTopicName>
-        <pointCloudTopicName>/camera/depth/points</pointCloudTopicName>
-        <cameraInfoTopicName>/camera/camera_info</cameraInfoTopicName>
+        <imageTopicName>/camera/rgb/image_raw</imageTopicName>
+        <pointCloudTopicName>/camera/rgb/points</pointCloudTopicName>
+        <cameraInfoTopicName>/camera/rgb/camera_info</cameraInfoTopicName>
         <frameName>/openni_depth_optical_frame</frameName>
         <!--<distortion_k1>0.00000001</distortion_k1>

File: head/head.urdf.xacro (robot description, xacro)
@@ -7,7 +7,6 @@
    <origin xyz="0.0 0.0 0.0" rpy="0 0 0" />
    <inertia ixx="0.0001"  ixy="0"  ixz="0" iyy="0.0001" iyz="0" izz="0.0001" /> <!--*-->
-   <color rgba="0.25 0.25 0.25 1.0"/>
 </xacro:my_link>
-<xacro:my_link name="neck_pan" mass="0.05" color="Blue">
+<xacro:my_link name="neck_pan" mass="0.05" color="Black">
    <cylinder radius="0.015" length="0.08" /> <!--*--> <!--checked-->
    <origin xyz="0.0 0.0 0.0335" rpy="0 0 0"/>
@@ -16,23 +15,21 @@
    <color rgba="0.25 0.25 0.25 1.0"/>
 </xacro:my_link>
-<xacro:my_link name="neck_tilt" mass="0.05" color="Blue">
+<xacro:my_link name="neck_tilt" mass="0.05" color="Black">
    <cylinder radius="0.015" length="0.057"  /> <!--*-->
    <origin xyz="0.0 -0.0 0.0285" rpy="0 0 0"/>
    <origin xyz="0.0 -0.0 0.0285" rpy="0 0 0" />
    <inertia ixx="0.001"  ixy="0"  ixz="0" iyy="0.001" iyz="0" izz="0.001" /> <!--*-->
-   <color rgba="0.25 0.25 0.25 1.0"/>
 </xacro:my_link>
- <link name="head">
-   <inertial>
-      <mass value="0" />
-      <origin xyz="0 0 0" />
-      <inertia ixx="0" ixy="0" ixz="0" iyy="0" iyz="0" izz="0"/>
-      </inertial>
-  </link>
+ <my_link_texturedmesh name="head" mass="0" texture="torsocovers">
+   <origin xyz="0 0 0" rpy="0 0 0"/>
+   <origin xyz="0.0 0.0 0.1" rpy="0 0 -1.5708"/>
+   <inertia ixx="0"  ixy="0"  ixz="0" iyy="0" iyz="0" izz="0" />
+   <mesh filename="package://amigo_robot_model/head/headtextured.dae" scale="0.001 0.001 0.001"/>
+  </my_link_texturedmesh>
   <joint name="head_mount_joint" type="fixed">
     <parent link="torso"/>
     <child link="head_mount"/>
     <axis xyz="0 0 1"/>
-    <origin xyz="0.097 0.0 0.046" rpy="  0.0 0.0 0.0"/>
+    <origin xyz="0.097 0.0 0.0" rpy="  0.0 0.0 0.0"/>
   </joint>
   <joint name="head_joint" type="fixed">

File: kinect/kinect.urdf.xacro (robot description, xacro)
@@ -21,14 +21,15 @@
       <origin xyz=" 0 0 0 " rpy="0 0 0" />
       <geometry>
+		<box size="0 0 0"/>
         <!--mesh filename="package://amigo_robot_model/kinect/meshes/kinect.dae" scale="0.001 0.001 0.001"/-->
-        <mesh filename="package://amigo_robot_model/kinect/meshes/kinect_without_base.dae"/>
+        <!--<mesh filename="package://amigo_robot_model/kinect/meshes/kinect_without_base.dae"/>-->
       </geometry>
     </visual>
-    <!--<collision>
+    <collision>
       <origin xyz="-0.0365 0.0 0.0" rpy="0 0 0" />
       <geometry>
         <box size="0.0730 .2760 0.0720"/>
       </geometry>
-    </collision>-->
+    </collision>
   </link>
   <joint name="kinect_depth_joint" type="fixed">

File: laser/laser.urdf.xacro (robot description, xacro)
@@ -9,5 +9,5 @@
 </xacro:my_link>
 <xacro:my_joint name="base_laser_joint" type="fixed" parent="base" child="base_laser">
-   <origin xyz="0.31 0.0 -0.2" rpy="0 0 0"/>
+   <origin xyz="0.31 0.0 0.1475" rpy="0 0 0"/>
    <dynamics damping="0.1" friction="0"/>
    <axis xyz="0 1 0"/>
