Commit message: NEW ROBOT MODEL!!!
git-svn-id: https://roboticssrv.wtb.tue.nl/svn/ros/code/tue-ros-pkg/trunk/tue_robot_models/amigo_robot_model@6876 3a3c2cfb-d3b9-409e-9e75-db8fcdbcaac6

File: robot.urdf.xacro (robot description, xacro)
@@ -8,6 +8,10 @@
 <!--get link & joint definitions -->
 <include filename="$(find amigo_robot_model)/definitions.xacro" />
+<!--get custom materials -->
+<include filename="$(find amigo_robot_model)/materials.urdf.xacro" />
 <!--========BUILD BODY======-->
 <include filename="$(find amigo_robot_model)/body/body.urdf.xacro" />
+<!--extra body visuals-->
+<include filename="$(find amigo_robot_model)/body_extra_visuals/body_extra.urdf.xacro" />
 <!--========BUILD LASER======-->
 <include filename="$(find amigo_robot_model)/laser/laser.urdf.xacro" />
@@ -16,20 +20,13 @@
 <!--========BUILD KINECT======-->
 <include filename="$(find amigo_robot_model)/kinect/kinect.urdf.xacro" />
-<!--========BUILD BASE KINECT======-->
-<!--<include filename="$(find amigo_robot_model)/base_kinect/base_kinect.urdf.xacro" />-->
-<!--========BUILD WHEELS======-->
-<include filename="$(find amigo_robot_model)/wheels/wheels.urdf.xacro" />
-<xacro:wheel side_LR="left" side_FR="front" sign_LR="-" sign_FR="+" wheel_angle="2.3562" />
-<xacro:wheel side_LR="right" side_FR="front" sign_LR="+" sign_FR="+" wheel_angle="0.7854" />
-<xacro:wheel side_LR="left" side_FR="rear" sign_LR="-" sign_FR="-" wheel_angle="-2.3562" />
-<xacro:wheel side_LR="right" side_FR="rear" sign_LR="+" sign_FR="-" wheel_angle="-0.7854" />
 <!--========BUILD ARMS======-->
 <include filename="$(find amigo_robot_model)/arms_DH/armDH.urdf.xacro" />
-<xacro:arm whichside="left" sidesign="-" orientationsign="1.5708" rolloffset="3.1416" />
-<xacro:arm whichside="right" sidesign="+" orientationsign="-1.5708" rolloffset="0.0"/>
-<!--====BUILD TRANSMISSION ELEMENTS====-->
-<include filename="$(find amigo_robot_model)/body/body.transmission.xacro" />
-<include filename="$(find amigo_robot_model)/arms_DH/armDH.transmission.xacro" />
-<include filename="$(find amigo_robot_model)/wheels/wheels.transmission.xacro" />
-<include filename="$(find amigo_robot_model)/head/head.transmission.xacro" />
+<xacro:arm whichside="right" sidesign="+1.0" rollsign="+"/>
+<xacro:arm whichside="left"  sidesign="-1.0" rollsign="-"/>
+<!--extra arm visuals-->
+<include filename="$(find amigo_robot_model)/arm_extra_visuals/arm_extra.urdf.xacro" />
+<xacro:arm_extra whichside="right" sidesign="+1.0" rollsign="+"/>
+<xacro:arm_extra whichside="left"  sidesign="-1.0" rollsign="-"/>
+<!--====BUILD STUFF THAT NEEDS TO RUN IN EITHER SIMULATION OR ON THE REAL ROBOT ====-->
+<include filename="$(find amigo_robot_model)/sim_or_robot_xacro/robot_real_$(optenv ROBOT_REAL false).urdf.xacro" />
 </robot>

File: wheels/wheels.urdf.xacro (robot description, xacro)
@@ -1,2 +1,3 @@
+<?xml version="1.0"?>
 <robot xmlns:xacro="http://ros.org/wiki/xacro">
 <!--wheels-->
@@ -6,32 +7,30 @@
     <child link="wheel_${side_LR}_${side_FR}"/>
     <axis xyz="1 0 0"/>
-    <origin xyz="${sign_LR}0.25 ${sign_FR}0.25 -0.3275" rpy="0 0 ${wheel_angle}"/>
+    <origin xyz="${sign_LR}0.2 ${sign_FR}0.2 0.08" rpy="0 0 ${wheel_angle}"/>
     <dynamics damping="1" friction="0.0"/>
     <limit effort="5.0" velocity="5.0"/>
   </joint>
-  <xacro:my_link name="wheel_${side_LR}_${side_FR}" mass="0.5" color="Blue">
+  <xacro:my_link name="wheel_${side_LR}_${side_FR}" mass="0.5" color="Grey">
     <cylinder radius="0.05" length="0.05"/>
     <origin xyz="0.0 0.0 0.0" rpy="0 0 0"/>
     <origin xyz="0.0 0.0 0.0" rpy="0 1.5708 0" />
     <inertia ixx="0.0006"  ixy="0"  ixz="0" iyy="0.0006" iyz="0" izz="0.0006" />
-    <color rgba="0.33 0.33 0.33 1.0"/>
    </xacro:my_link>
 </xacro:macro>
 <xacro:macro name="z_sphere" params="side_LR side_FR number y_ z_ roll_">
-   <joint name="omni_sphere${number}_joint_${side_LR}_${side_FR}" type="continuous">
-   <parent link="wheel_${side_LR}_${side_FR}"/>
-   <child link="omni_sphere${number}_${side_LR}_${side_FR}"/>
-   <axis xyz="0 1 0"/>
-   <origin xyz="0.0 ${y_} ${z_}" rpy="${roll_} 0 0"/>
-   <dynamics damping="0.01" friction="0.0"/>
-   <limit effort="0.5" velocity="0.05"/>
-   </joint>
-   <xacro:my_link name="omni_sphere${number}_${side_LR}_${side_FR}" mass="0.05" color="Blue">
-   <sphere radius="0.03" />
-   <origin xyz="0.0 0.0 0.0" rpy="0 0 0"/>
-   <origin xyz="0.0 0.0 0.0" rpy="0 0 0" />
-   <inertia ixx="0.000018"  ixy="0"  ixz="0" iyy="0.000018" iyz="0" izz="0.000018" />
-   <color rgba="0.33 0.33 0.33 1.0"/>
-   </xacro:my_link>
+	<joint name="omni_sphere${number}_joint_${side_LR}_${side_FR}" type="continuous">
+		<parent link="wheel_${side_LR}_${side_FR}"/>
+		<child link="omni_sphere${number}_${side_LR}_${side_FR}"/>
+		<axis xyz="0 1 0"/>
+		<origin xyz="0.0 ${y_} ${z_}" rpy="${roll_} 0 0"/>
+		<dynamics damping="0.01" friction="0.0"/>
+		<limit effort="0.5" velocity="0.05"/>
+	</joint>
+	<xacro:my_link name="omni_sphere${number}_${side_LR}_${side_FR}" mass="0.05" color="Grey">
+		<sphere radius="0.03" />
+		<origin xyz="0.0 0.0 0.0" rpy="0 0 0"/>
+		<origin xyz="0.0 0.0 0.0" rpy="0 0 0" />
+		<inertia ixx="0.000018"  ixy="0"  ixz="0" iyy="0.000018" iyz="0" izz="0.000018" />
+	</xacro:my_link>
 </xacro:macro>
 <xacro:macro name="spheres" params="nr y z roll">

Commit message: problem with self_filter solved
git-svn-id: https://roboticssrv.wtb.tue.nl/svn/ros/code/tue-ros-pkg/trunk/tue_robot_models/amigo_robot_model@6881 3a3c2cfb-d3b9-409e-9e75-db8fcdbcaac6

File: arms_DH/armDH.urdf.xacro (robot description, xacro)
@@ -28,5 +28,5 @@
    <origin xyz="0.0 -0.2 0.0" rpy="0 0 3.1415" />
    <inertia ixx="0.027"  ixy="0"  ixz="0" iyy="0.027" iyz="0" izz="0.004" />
-   <mesh filename="package://amigo_robot_model/arms_DH/upperarmtextured.dae" scale="0.001 0.001 0.001"/>
+   <mesh filename="package://amigo_robot_model/arms_DH/upperarmtextured2.dae" scale="0.001 0.001 0.001"/>
 </xacro:my_link_texturedmesh>
 <xacro:my_link name="elbow_link4_${whichside}" mass="0.1" color="Grey">
@@ -40,5 +40,5 @@
    <origin xyz="0.0 -0.14 0.0" rpy="0 -1.5708 0" />
    <inertia ixx="0.0054"  ixy="0"  ixz="0" iyy="0.0054" iyz="0" izz="0.0004" />
-   <mesh filename="package://amigo_robot_model/arms_DH/forearmtextured.dae" scale="0.001 0.001 0.001"/>
+   <mesh filename="package://amigo_robot_model/arms_DH/forearmtextured2.dae" scale="0.001 0.001 0.001"/>
 </xacro:my_link_texturedmesh>
 <xacro:my_link name="wrist_link6_${whichside}" mass="0.01" color="Black">

File: laser/laser.urdf.xacro (robot description, xacro)
@@ -2,9 +2,8 @@
 <robot xmlns:xacro="http://ros.org/wiki/xacro">
 <xacro:my_link name="base_laser" mass="0.5" color="Black">
-   <box size="0.05 0.05 0.05" /> <!--*-->
+   <box size="0.05 0.06 0.12" /> <!--*-->
    <origin xyz="0.0 0.0 0.0" rpy="0 0 0"/>
-   <origin xyz="0.0 0.0 0.0" rpy="0 0 0" />
+   <origin xyz="-0.005 0.0 0.0525" rpy="0 0 0" />
    <inertia ixx="0.0001"  ixy="0"  ixz="0" iyy="0.0001" iyz="0" izz="0.0001" /> <!--*-->
-   <color rgba="0.15 0.15 0.15 1.0"/>
 </xacro:my_link>
 <xacro:my_joint name="base_laser_joint" type="fixed" parent="base" child="base_laser">

Commit message: did some renaming of meshes and textures
git-svn-id: https://roboticssrv.wtb.tue.nl/svn/ros/code/tue-ros-pkg/trunk/tue_robot_models/amigo_robot_model@6884 3a3c2cfb-d3b9-409e-9e75-db8fcdbcaac6

File: arms_DH/armDH.urdf.xacro (robot description, xacro)
@@ -24,9 +24,9 @@
    <inertia ixx="0.001"  ixy="0"  ixz="0" iyy="0.001" iyz="0" izz="0.001" />
 </xacro:my_link>
-<xacro:my_link_texturedmesh name="upper_arm_${whichside}" mass="2.9" texture="torsocovers">
+<xacro:my_link_texturedmesh name="upper_arm_${whichside}" mass="2.9" texture="white">
    <origin xyz="0.0 -0.2 0.0" rpy="0 0 0"/>
    <origin xyz="-0.00959 -0.19131 -0.00001" rpy="0 0 3.1415" />
    <inertia ixx="0.027"  ixy="0"  ixz="0" iyy="0.027" iyz="0" izz="0.004" />
-   <mesh filename="package://amigo_robot_model/arms_DH/upperarmtextured2.dae" scale="0.001 0.001 0.001"/>
+   <mesh filename="package://amigo_robot_model/arms_DH/upperarmtextured.dae" scale="0.001 0.001 0.001"/>
 </xacro:my_link_texturedmesh>
 <xacro:my_link name="elbow_link4_${whichside}" mass="0.1" color="Grey">
@@ -36,9 +36,9 @@
    <inertia ixx="0.001"  ixy="0"  ixz="0" iyy="0.001" iyz="0" izz="0.001" />
 </xacro:my_link>
-<xacro:my_link_texturedmesh name="fore_arm_${whichside}" mass="0.1" texture="torsocovers">
+<xacro:my_link_texturedmesh name="fore_arm_${whichside}" mass="0.1" texture="white">
    <origin xyz="0.0 -0.14 0.0" rpy="0.0 0 0"/>
    <origin xyz="0.00425 -0.14868 0.00547" rpy="0 -1.5708 0" />
    <inertia ixx="0.0054"  ixy="0"  ixz="0" iyy="0.0054" iyz="0" izz="0.0004" />
-   <mesh filename="package://amigo_robot_model/arms_DH/forearmtextured2.dae" scale="0.001 0.001 0.001"/>
+   <mesh filename="package://amigo_robot_model/arms_DH/forearmtextured.dae" scale="0.001 0.001 0.001"/>
 </xacro:my_link_texturedmesh>
 <xacro:my_link name="wrist_link6_${whichside}" mass="0.01" color="Black">

File: body/body.urdf.xacro (robot description, xacro)
@@ -6,5 +6,5 @@
    <origin xyz="0.0 0.0 0.3275" rpy="0 0 -1.5708" />
    <inertia ixx="2.63"  ixy="0"  ixz="0" iyy="2.63" iyz="0" izz="2.4" /> <!--*-->
-   <mesh filename="package://amigo_robot_model/body/onderkantversiekrisreducedtextured.dae" scale="0.001 0.001 0.001"/>
+   <mesh filename="package://amigo_robot_model/body/bottomcovers.dae" scale="0.001 0.001 0.001"/>
    <box size="0.25 0.25 0.5"/>
 </xacro:my_link_texturedmesh_diff_coll>
@@ -21,5 +21,5 @@
    <inertia ixx="0"  ixy="0"  ixz="0" iyy="0" iyz="0" izz="0" />
 </xacro:my_link>
-<xacro:my_link_texturedmesh name="torso" mass="16" texture="torsocovers">
+<xacro:my_link_texturedmesh name="torso" mass="16" texture="white">
    <origin xyz="0.0 0.0 0.0" rpy="0 0 0"/>
    <origin xyz="0.045 0.0 0.06" rpy="-1.5708 0 -1.5708" />

File: head/head.urdf.xacro (robot description, xacro)
@@ -21,5 +21,5 @@
    <inertia ixx="0.001"  ixy="0"  ixz="0" iyy="0.001" iyz="0" izz="0.001" /> <!--*-->
 </xacro:my_link>
- <my_link_texturedmesh name="head" mass="0" texture="torsocovers">
+ <my_link_texturedmesh name="head" mass="0" texture="white">
    <origin xyz="0 0 0" rpy="0 0 0"/>
    <origin xyz="0.0 0.0 0.1" rpy="0 0 -1.5708"/>

File: materials.urdf.xacro (robot description, xacro)
@@ -28,6 +28,6 @@
     <texture filename="package://amigo_robot_model/Media/materials/textures/bottomcovers/finalreduced.jpg" />
   </material>
-  <material name="torsocovers">
-    <texture filename="package://amigo_robot_model/Media/materials/textures/torsocovers/white.jpg" />
+    <material name="white">
+    <texture filename="package://amigo_robot_model/Media/materials/textures/white/white.jpg" />
   </material>
 </robot>

Commit message: Joint bounds in URDF
git-svn-id: https://roboticssrv.wtb.tue.nl/svn/ros/code/tue-ros-pkg/trunk/tue_robot_models/amigo_robot_model@7042 3a3c2cfb-d3b9-409e-9e75-db8fcdbcaac6

File: arms_DH/armDH.urdf.xacro (robot description, xacro)
@@ -82,5 +82,5 @@
    <dynamics damping="6.0" friction="4.87"/>
    <axis xyz="${rollsign}1 0 0"/>
-   <limit effort="13.4" velocity="1.0" lower="-1.5708" upper="1e-3" />
+   <limit effort="13.4" velocity="1.0" lower="-1.58" upper="0.01" />
 </xacro:my_joint>
 <xacro:my_joint name="shoulder_pitch_joint_${whichside}" type="revolute" parent="shoulder_link1_${whichside}" child="shoulder_link2_${whichside}">
@@ -88,5 +88,5 @@
    <dynamics damping="6.0" friction="6.06"/>
    <axis xyz="0 -1 0"/>
-   <limit effort="13.4" velocity="1.0" lower="-1.5708" upper="1.5708" />
+   <limit effort="13.4" velocity="1.0" lower="-1.58" upper="1.58" />
 </xacro:my_joint>
 <xacro:my_joint name="shoulder_roll_joint_${whichside}" type="revolute" parent="shoulder_link2_${whichside}" child="upper_arm_${whichside}">
@@ -94,5 +94,5 @@
    <dynamics damping="6.0" friction="2.16"/>
    <axis xyz="0 ${sidesign} 0"/>
-   <limit effort="9.8" velocity="1.0" lower="-1.5708" upper="1.5708"/>
+   <limit effort="9.8" velocity="1.0" lower="-1.58" upper="1.58"/>
 </xacro:my_joint>
 <xacro:my_joint name="elbow_pitch_joint_${whichside}" type="revolute" parent="upper_arm_${whichside}" child="elbow_link4_${whichside}">
@@ -100,5 +100,5 @@
    <dynamics damping="2.5" friction="1.18"/>
    <axis xyz="0 -1 0"/>
-   <limit effort="4.5" velocity="1.0" lower="0.0" upper="2.5307" />
+   <limit effort="4.5" velocity="1.0" lower="-0.01" upper="2.24" />
 </xacro:my_joint>
 <xacro:my_joint name="elbow_roll_joint_${whichside}" type="revolute" parent="elbow_link4_${whichside}" child="fore_arm_${whichside}">
@@ -106,5 +106,5 @@
    <dynamics damping="2.5" friction="1.35"/>
    <axis xyz="0 ${sidesign} 0"/>
-   <limit effort="4.5" velocity="1.0" lower="-1.8326" upper="1.8326"/>
+   <limit effort="4.5" velocity="1.0" lower="-1.84" upper="1.84"/>
 </xacro:my_joint>
 <xacro:my_joint name="wrist_pitch_joint_${whichside}" type="revolute" parent="fore_arm_${whichside}" child="wrist_link6_${whichside}">
@@ -112,5 +112,5 @@
    <dynamics damping="0.5" friction="0.63"/>
    <axis xyz="0 -1 0"/>
-   <limit effort="1" velocity="1.0" lower="-0.9940" upper="0.9940"/>
+   <limit effort="1" velocity="1.0" lower="-0.96" upper="0.96"/>
 </xacro:my_joint>
 <xacro:my_joint name="wrist_yaw_joint_${whichside}" type="revolute" parent="wrist_link6_${whichside}" child="hand_${whichside}">
@@ -118,5 +118,5 @@
    <dynamics damping="0.5" friction="0.68"/>
    <axis xyz="0 0 ${sidesign}1"/>
-   <limit effort="1" velocity="1.0" lower="-0.7854" upper="0.7854"/>
+   <limit effort="1" velocity="1.0" lower="-0.8" upper="0.8"/>
 </xacro:my_joint>
 <xacro:my_joint name="finger1_joint_${whichside}" type="revolute" parent="hand_${whichside}" child="finger1_${whichside}">

Commit message: Increased joint constraints for move arm in URDF
git-svn-id: https://roboticssrv.wtb.tue.nl/svn/ros/code/tue-ros-pkg/trunk/tue_robot_models/amigo_robot_model@7145 3a3c2cfb-d3b9-409e-9e75-db8fcdbcaac6

File: arms_DH/armDH.urdf.xacro (robot description, xacro)
@@ -82,5 +82,5 @@
    <dynamics damping="6.0" friction="4.87"/>
    <axis xyz="${rollsign}1 0 0"/>
-   <limit effort="13.4" velocity="1.0" lower="-1.58" upper="0.01" />
+   <limit effort="13.4" velocity="1.0" lower="-1.67" upper="0.1" />
 </xacro:my_joint>
 <xacro:my_joint name="shoulder_pitch_joint_${whichside}" type="revolute" parent="shoulder_link1_${whichside}" child="shoulder_link2_${whichside}">
@@ -88,5 +88,5 @@
    <dynamics damping="6.0" friction="6.06"/>
    <axis xyz="0 -1 0"/>
-   <limit effort="13.4" velocity="1.0" lower="-1.58" upper="1.58" />
+   <limit effort="13.4" velocity="1.0" lower="-1.67" upper="1.67" />
 </xacro:my_joint>
 <xacro:my_joint name="shoulder_roll_joint_${whichside}" type="revolute" parent="shoulder_link2_${whichside}" child="upper_arm_${whichside}">
@@ -94,5 +94,5 @@
    <dynamics damping="6.0" friction="2.16"/>
    <axis xyz="0 ${sidesign} 0"/>
-   <limit effort="9.8" velocity="1.0" lower="-1.58" upper="1.58"/>
+   <limit effort="9.8" velocity="1.0" lower="-1.67" upper="1.67"/>
 </xacro:my_joint>
 <xacro:my_joint name="elbow_pitch_joint_${whichside}" type="revolute" parent="upper_arm_${whichside}" child="elbow_link4_${whichside}">
@@ -100,5 +100,5 @@
    <dynamics damping="2.5" friction="1.18"/>
    <axis xyz="0 -1 0"/>
-   <limit effort="4.5" velocity="1.0" lower="-0.01" upper="2.24" />
+   <limit effort="4.5" velocity="1.0" lower="-0.1" upper="2.33" />
 </xacro:my_joint>
 <xacro:my_joint name="elbow_roll_joint_${whichside}" type="revolute" parent="elbow_link4_${whichside}" child="fore_arm_${whichside}">
@@ -106,5 +106,5 @@
    <dynamics damping="2.5" friction="1.35"/>
    <axis xyz="0 ${sidesign} 0"/>
-   <limit effort="4.5" velocity="1.0" lower="-1.84" upper="1.84"/>
+   <limit effort="4.5" velocity="1.0" lower="-1.93" upper="1.93"/>
 </xacro:my_joint>
 <xacro:my_joint name="wrist_pitch_joint_${whichside}" type="revolute" parent="fore_arm_${whichside}" child="wrist_link6_${whichside}">
@@ -112,5 +112,5 @@
    <dynamics damping="0.5" friction="0.63"/>
    <axis xyz="0 -1 0"/>
-   <limit effort="1" velocity="1.0" lower="-0.96" upper="0.96"/>
+   <limit effort="1" velocity="1.0" lower="-1.05" upper="1.05"/>
 </xacro:my_joint>
 <xacro:my_joint name="wrist_yaw_joint_${whichside}" type="revolute" parent="wrist_link6_${whichside}" child="hand_${whichside}">
@@ -118,5 +118,5 @@
    <dynamics damping="0.5" friction="0.68"/>
    <axis xyz="0 0 ${sidesign}1"/>
-   <limit effort="1" velocity="1.0" lower="-0.8" upper="0.8"/>
+   <limit effort="1" velocity="1.0" lower="-0.89" upper="0.89"/>
 </xacro:my_joint>
 <xacro:my_joint name="finger1_joint_${whichside}" type="revolute" parent="hand_${whichside}" child="finger1_${whichside}">

Commit message: New joint limits in planner
git-svn-id: https://roboticssrv.wtb.tue.nl/svn/ros/code/tue-ros-pkg/trunk/tue_robot_models/amigo_robot_model@7159 3a3c2cfb-d3b9-409e-9e75-db8fcdbcaac6

File: arms_DH/armDH.urdf.xacro (robot description, xacro)
@@ -118,5 +118,5 @@
    <dynamics damping="0.5" friction="0.68"/>
    <axis xyz="0 0 ${sidesign}1"/>
-   <limit effort="1" velocity="1.0" lower="-0.89" upper="0.89"/>
+   <limit effort="1" velocity="1.0" lower="-0.71" upper="0.71"/>
 </xacro:my_joint>
 <xacro:my_joint name="finger1_joint_${whichside}" type="revolute" parent="hand_${whichside}" child="finger1_${whichside}">

Commit message: different topic for arm navigation
git-svn-id: https://roboticssrv.wtb.tue.nl/svn/ros/code/tue-ros-pkg/trunk/tue_robot_models/amigo_robot_model@7178 3a3c2cfb-d3b9-409e-9e75-db8fcdbcaac6

File: arms_DH/armDH.urdf.xacro (robot description, xacro)
@@ -82,5 +82,5 @@
    <dynamics damping="6.0" friction="4.87"/>
    <axis xyz="${rollsign}1 0 0"/>
-   <limit effort="13.4" velocity="1.0" lower="-1.67" upper="0.1" />
+   <limit effort="13.4" velocity="1.0" lower="-1.57" upper="0.0" />
 </xacro:my_joint>
 <xacro:my_joint name="shoulder_pitch_joint_${whichside}" type="revolute" parent="shoulder_link1_${whichside}" child="shoulder_link2_${whichside}">
@@ -88,5 +88,5 @@
    <dynamics damping="6.0" friction="6.06"/>
    <axis xyz="0 -1 0"/>
-   <limit effort="13.4" velocity="1.0" lower="-1.67" upper="1.67" />
+   <limit effort="13.4" velocity="1.0" lower="-1.57" upper="1.57" />
 </xacro:my_joint>
 <xacro:my_joint name="shoulder_roll_joint_${whichside}" type="revolute" parent="shoulder_link2_${whichside}" child="upper_arm_${whichside}">
@@ -94,5 +94,5 @@
    <dynamics damping="6.0" friction="2.16"/>
    <axis xyz="0 ${sidesign} 0"/>
-   <limit effort="9.8" velocity="1.0" lower="-1.67" upper="1.67"/>
+   <limit effort="9.8" velocity="1.0" lower="-1.57" upper="1.57"/>
 </xacro:my_joint>
 <xacro:my_joint name="elbow_pitch_joint_${whichside}" type="revolute" parent="upper_arm_${whichside}" child="elbow_link4_${whichside}">
@@ -100,5 +100,5 @@
    <dynamics damping="2.5" friction="1.18"/>
    <axis xyz="0 -1 0"/>
-   <limit effort="4.5" velocity="1.0" lower="-0.1" upper="2.33" />
+   <limit effort="4.5" velocity="1.0" lower="0.0" upper="2.23" />
 </xacro:my_joint>
 <xacro:my_joint name="elbow_roll_joint_${whichside}" type="revolute" parent="elbow_link4_${whichside}" child="fore_arm_${whichside}">
@@ -106,5 +106,5 @@
    <dynamics damping="2.5" friction="1.35"/>
    <axis xyz="0 ${sidesign} 0"/>
-   <limit effort="4.5" velocity="1.0" lower="-1.93" upper="1.93"/>
+   <limit effort="4.5" velocity="1.0" lower="-1.83" upper="1.83"/>
 </xacro:my_joint>
 <xacro:my_joint name="wrist_pitch_joint_${whichside}" type="revolute" parent="fore_arm_${whichside}" child="wrist_link6_${whichside}">
@@ -112,5 +112,5 @@
    <dynamics damping="0.5" friction="0.63"/>
    <axis xyz="0 -1 0"/>
-   <limit effort="1" velocity="1.0" lower="-1.05" upper="1.05"/>
+   <limit effort="1" velocity="1.0" lower="-0.95" upper="0.95"/>
 </xacro:my_joint>
 <xacro:my_joint name="wrist_yaw_joint_${whichside}" type="revolute" parent="wrist_link6_${whichside}" child="hand_${whichside}">
@@ -118,5 +118,5 @@
    <dynamics damping="0.5" friction="0.68"/>
    <axis xyz="0 0 ${sidesign}1"/>
-   <limit effort="1" velocity="1.0" lower="-0.71" upper="0.71"/>
+   <limit effort="1" velocity="1.0" lower="-0.61" upper="0.61"/>
 </xacro:my_joint>
 <xacro:my_joint name="finger1_joint_${whichside}" type="revolute" parent="hand_${whichside}" child="finger1_${whichside}">
