Commit message: some visual changes in arms
git-svn-id: https://roboticssrv.wtb.tue.nl/svn/ros/code/tue-ros-pkg/trunk/tue_robot_models/amigo_robot_model@6883 3a3c2cfb-d3b9-409e-9e75-db8fcdbcaac6

File: arm_extra_visuals/arm_extra.urdf.xacro (robot description, xacro)
@@ -3,23 +3,35 @@
 <xacro:macro name="arm_extra" params="whichside sidesign rollsign">
 <xacro:my_link name="upper_arm_top_${whichside}" mass="0.01" color="Black">
-   <cylinder radius="0.058" length="0.02"/>
+   <cylinder radius="0.0561" length="0.02"/>
    <origin xyz="0.0 0.0 0.0" rpy="0 0 0"/>
    <origin xyz="0.0 0.0 0.0" rpy="0 0 0" />
    <inertia ixx="0.027"  ixy="0"  ixz="0" iyy="0.027" iyz="0" izz="0.004" />
 </xacro:my_link>
-<xacro:my_link name="elbow_extra_block_${whichside}" mass="0.01" color="Red">
-   <box size="0.0 0.0 0.0"/>
+<xacro:my_link name="elbow_extra_block_${whichside}" mass="0.01" color="Black">
+   <box size="0.015 0.08 0.06"/>
+   <origin xyz="0.0 0.0 0.0" rpy="0 0 0"/>
+   <origin xyz="-0.036 0.0 0.02" rpy="0 0 0" />
+   <inertia ixx="0.001"  ixy="0"  ixz="0" iyy="0.001" iyz="0" izz="0.001" />
+</xacro:my_link>
+<xacro:my_link name="elbow_extra_block2_${whichside}" mass="0.01" color="Grey">
+   <cylinder radius="0.03" length="0.08"/>
+   <origin xyz="0.0 0.0 0.0" rpy="0 0 0"/>
+   <origin xyz="0.0 0.0 0.0" rpy="1.5708 0 0" />
+   <inertia ixx="0.001"  ixy="0"  ixz="0" iyy="0.001" iyz="0" izz="0.001" />
+</xacro:my_link>
+<xacro:my_link name="fore_arm_top_${whichside}" mass="0.01" color="Black">
+   <cylinder radius="0.037" length="0.01"/>
+   <origin xyz="0.0 0.0 0.0" rpy="0 0 0"/>
+   <origin xyz="0.0 0.0 0.01" rpy="0 0 0" />
+   <inertia ixx="0.0054"  ixy="0"  ixz="0" iyy="0.0054" iyz="0" izz="0.0004" />
+</xacro:my_link>
+<xacro:my_link name="wrist_visual_${whichside}" mass="0.01" color="Grey">
+   <cylinder radius="0.018" length="0.06"/>
    <origin xyz="0.0 0.0 0.0" rpy="0 0 0"/>
    <origin xyz="0.0 0.0 0.0" rpy="0 0 0" />
    <inertia ixx="0.001"  ixy="0"  ixz="0" iyy="0.001" iyz="0" izz="0.001" />
 </xacro:my_link>
-<xacro:my_link name="fore_arm_top_${whichside}" mass="0.01" color="Black">
-   <cylinder radius="0.04" length="0.01"/>
-   <origin xyz="0.0 0.0 0.0" rpy="0 0 0"/>
-   <origin xyz="0.0 0.0 0.01" rpy="0 0 0" />
-   <inertia ixx="0.0054"  ixy="0"  ixz="0" iyy="0.0054" iyz="0" izz="0.0004" />
-</xacro:my_link>
-<xacro:my_link name="wrist_to_hand_block_${whichside}" mass="0.01" color="Red">
-   <box size="0.0 0.0 0.0"/>
+<xacro:my_link name="wrist_to_hand_block_${whichside}" mass="0.01" color="Grey">
+   <box size="0.03 0.02 0.038"/>
    <origin xyz="0.0 0.0 0.0" rpy="0 0 0"/>
    <origin xyz="0.0 0.0 0.0" rpy="0 0 0" />
@@ -33,12 +45,22 @@
 </joint>
 <joint name="elbow_extra_block_joint_${whichside}" type="fixed">
-  <parent link="elbow_link4_${whichside}"/>
+  <parent link="upper_arm_${whichside}"/>
   <child link="elbow_extra_block_${whichside}"/>
-   <origin xyz="0.0 0.0 0.0" rpy="0 0 0"/>
+  <origin xyz="0.0 -0.31 0.0" rpy="-1.5708 0 0"/>
+</joint>
+<joint name="elbow_extra_block2_joint_${whichside}" type="fixed">
+  <parent link="upper_arm_${whichside}"/>
+  <child link="elbow_extra_block2_${whichside}"/>
+  <origin xyz="0.0 -0.31 0.0" rpy="-1.5708 0 0"/>
 </joint>
 <joint name="fore_arm_top_joint_${whichside}" type="fixed" >
   <parent link="fore_arm_${whichside}"/>
   <child link="fore_arm_top_${whichside}"/>
-   <origin xyz="0.0 0.0 0.0" rpy="1.5708 0 0"/>
+   <origin xyz="0.002 -0.011 0.0" rpy="1.5708 0 0"/>
+</joint>
+<joint name="wrist_visual_joint_${whichside}" type="fixed">
+  <parent link="wrist_link6_${whichside}"/>
+  <child link="wrist_visual_${whichside}"/>
+  <origin xyz="-0.02 0.0 0.0" rpy="1.5708 0 0"/>
 </joint>
 <joint name="wrist_to_hand_block_joint_${whichside}" type="fixed">

File: arms_DH/armDH.urdf.xacro (robot description, xacro)
@@ -26,24 +26,24 @@
 <xacro:my_link_texturedmesh name="upper_arm_${whichside}" mass="2.9" texture="torsocovers">
    <origin xyz="0.0 -0.2 0.0" rpy="0 0 0"/>
-   <origin xyz="0.0 -0.2 0.0" rpy="0 0 3.1415" />
+   <origin xyz="-0.00959 -0.19131 -0.00001" rpy="0 0 3.1415" />
    <inertia ixx="0.027"  ixy="0"  ixz="0" iyy="0.027" iyz="0" izz="0.004" />
    <mesh filename="package://amigo_robot_model/arms_DH/upperarmtextured2.dae" scale="0.001 0.001 0.001"/>
 </xacro:my_link_texturedmesh>
 <xacro:my_link name="elbow_link4_${whichside}" mass="0.1" color="Grey">
-   <cylinder radius="0.025" length="0.08"/>
+   <cylinder radius="0.0" length="0.0"/>
    <origin xyz="0.0 0.0 0.0" rpy="0 0 0"/>
-   <origin xyz="-0.017 0.0 0.015" rpy="1.5708 0 0" />
+   <origin xyz="0.0 0.0 0.0" rpy="0 0 0" />
    <inertia ixx="0.001"  ixy="0"  ixz="0" iyy="0.001" iyz="0" izz="0.001" />
 </xacro:my_link>
 <xacro:my_link_texturedmesh name="fore_arm_${whichside}" mass="0.1" texture="torsocovers">
    <origin xyz="0.0 -0.14 0.0" rpy="0.0 0 0"/>
-   <origin xyz="0.0 -0.14 0.0" rpy="0 -1.5708 0" />
+   <origin xyz="0.00425 -0.14868 0.00547" rpy="0 -1.5708 0" />
    <inertia ixx="0.0054"  ixy="0"  ixz="0" iyy="0.0054" iyz="0" izz="0.0004" />
    <mesh filename="package://amigo_robot_model/arms_DH/forearmtextured2.dae" scale="0.001 0.001 0.001"/>
 </xacro:my_link_texturedmesh>
 <xacro:my_link name="wrist_link6_${whichside}" mass="0.01" color="Black">
-   <cylinder radius="0.018" length="0.06"/>
+   <cylinder radius="0.0" length="0.0"/>
    <origin xyz="0.0 0.0 0.0" rpy="0 0 0"/>
-   <origin xyz="0.0 0.0 -0.034" rpy="1.5708 0 0" />
+   <origin xyz="0.0 0.0 0.0" rpy="1.5708 0 0" />
    <inertia ixx="0.001"  ixy="0"  ixz="0" iyy="0.001" iyz="0" izz="0.001" />
 </xacro:my_link>
@@ -51,5 +51,5 @@
    <box size="0.080 0.085 0.038"/>
    <origin xyz="0.048 0.0 0.0" rpy="0 0 0"/>
-   <origin xyz="0.048 0.0 -0.034" rpy="0 0 0" />
+   <origin xyz="0.048 0.0 0.0" rpy="0 0 0" />
    <inertia ixx="0.01"  ixy="0"  ixz="0" iyy="0.01" iyz="0" izz="0.01" />
 </xacro:my_link>
@@ -57,5 +57,5 @@
    <box size="0.02 0.022 0.11"/>
    <origin xyz="0.0 0.0 -0.055" rpy="0 0 0"/>
-   <origin xyz="-0.034 0.0 -0.055" rpy="0 0 0" />
+   <origin xyz="0.0 0.0 -0.055" rpy="0 0 0" />
    <inertia ixx="0.00037"  ixy="0"  ixz="0" iyy="0.00052" iyz="0" izz="0.00052" />
 </xacro:my_link>
@@ -63,9 +63,9 @@
    <box size="0.02 0.022 0.11"/>
    <origin xyz="0.0 0.0 -0.055" rpy="0 0 0"/>
-   <origin xyz="-0.034 0.0 -0.055" rpy="0 0 0" />
+   <origin xyz="0.0 0.0 -0.055" rpy="0 0 0" />
    <inertia ixx="0.00037"  ixy="0"  ixz="0" iyy="0.00052" iyz="0" izz="0.00052" />
 </xacro:my_link>
 <xacro:my_link name="grippoint_${whichside}" mass="0.01" color="Blue">
-   <box size="0.01 0.01 0.01"/>
+   <box size="0.0 0.0 0.0"/>
    <origin xyz="-0.1 0.0 0.0" rpy="0 0 0"/>
    <origin xyz="-0.1 0.0 0.0" rpy="0 0 0 " />
