Commit message: addes some documentation in the xacro files
git-svn-id: https://roboticssrv.wtb.tue.nl/svn/ros/code/tue-ros-pkg/trunk/tue_robot_models/amigo_robot_model@7273 3a3c2cfb-d3b9-409e-9e75-db8fcdbcaac6

File: arm_extra_visuals/arm_extra.urdf.xacro (robot description, xacro)
@@ -1,5 +1,15 @@
 <robot xmlns:xacro="http://ros.org/wiki/xacro">
-<!--Fill out Link macros-->
+   <author>Kris van Tienhoven</author>
+   <license>BSD</license>
+   <review status="unreviewed" notes=""/>
+<!--Start of the macro
+@param whichside is "left"  or "right"
+@param sidesign is -1 or +1
+@param rollsign is - or +
+The reason sidesign is -1 or +1 and not just - or + aswell is because
+it has to be reversable and xml cannot multiply - or + but can multiply
+ -1 and +1-->
 <xacro:macro name="arm_extra" params="whichside sidesign rollsign">
+<!--the black cylinder sealing the upper arm-->
 <xacro:my_link name="upper_arm_top_${whichside}" mass="0.01" color="Black">
    <cylinder radius="0.0561" length="0.02"/>
@@ -8,4 +18,5 @@
    <inertia ixx="0.027"  ixy="0"  ixz="0" iyy="0.027" iyz="0" izz="0.004" />
 </xacro:my_link>
+<!-- the black box under the upper arm, elbow visual 1 -->
 <xacro:my_link name="elbow_extra_block_${whichside}" mass="0.01" color="Black">
    <box size="0.015 0.08 0.06"/>
@@ -14,4 +25,5 @@
    <inertia ixx="0.001"  ixy="0"  ixz="0" iyy="0.001" iyz="0" izz="0.001" />
 </xacro:my_link>
+<!--the grey cylinder that connects the black box to the forearm, elbow visual 2-->
 <xacro:my_link name="elbow_extra_block2_${whichside}" mass="0.01" color="Grey">
    <cylinder radius="0.03" length="0.08"/>
@@ -20,4 +32,5 @@
    <inertia ixx="0.001"  ixy="0"  ixz="0" iyy="0.001" iyz="0" izz="0.001" />
 </xacro:my_link>
+<!--the black cylinder sealing the forearm -->
 <xacro:my_link name="fore_arm_top_${whichside}" mass="0.01" color="Black">
    <cylinder radius="0.037" length="0.01"/>
@@ -26,4 +39,5 @@
    <inertia ixx="0.0054"  ixy="0"  ixz="0" iyy="0.0054" iyz="0" izz="0.0004" />
 </xacro:my_link>
+<!--the grey cylinder at the end of the forearm-->
 <xacro:my_link name="wrist_visual_${whichside}" mass="0.01" color="Grey">
    <cylinder radius="0.018" length="0.06"/>
@@ -32,4 +46,5 @@
    <inertia ixx="0.001"  ixy="0"  ixz="0" iyy="0.001" iyz="0" izz="0.001" />
 </xacro:my_link>
+<!--the little grey box that connects the above cylinder with the hand -->
 <xacro:my_link name="wrist_to_hand_block_${whichside}" mass="0.01" color="Grey">
    <box size="0.03 0.02 0.038"/>
@@ -38,5 +53,5 @@
    <inertia ixx="0.001"  ixy="0"  ixz="0" iyy="0.001" iyz="0" izz="0.001" />
 </xacro:my_link>
-<!--joints-->
+<!--the joints start here-->
 <joint name="upper_arm_top_joint_${whichside}" type="fixed">
   <parent link="upper_arm_${whichside}" />

File: arms_DH/armDH.urdf.xacro (robot description, xacro)
@@ -4,6 +4,16 @@
 	xmlns:controller="http://playerstage.sourceforge.net/gazebo/xmlschema/#controller"
 	xmlns:interface="http://playerstage.sourceforge.net/gazebo/xmlschema/#interface">
-<!--Fill out Link macros-->
-<xacro:macro name="arm" params="whichside sidesign rollsign">
+	<author>Rob Janssen, Kris van Tienhoven</author>
+   <license>BSD</license>
+   <review status="unreviewed" notes=""/>
+<!--Start of the macro
+@param whichside is "left"  or "right"
+@param sidesign is -1 or +1
+@param rollsign is - or +
+The reason sidesign is -1 or +1 and not just - or + aswell is because
+it has to be reversable and xml cannot multiply - or + but can multiply
+ -1 and +1-->
+ <xacro:macro name="arm" params="whichside sidesign rollsign">
+<!--the end of the clavicle, yaw rotation-->
 <xacro:my_link name="shoulder_mount_${whichside}" mass="0.1" color="Black">
    <cylinder radius="0.05" length="0.11" />
@@ -12,4 +22,5 @@
    <inertia ixx="0.01"  ixy="0"  ixz="0" iyy="0.01" iyz="0" izz="0.01" />
 </xacro:my_link>
+<!--the cylinder on the end of the clavicle, pitch rotation-->
 <xacro:my_link name="shoulder_link1_${whichside}" mass="0.1" color="Black">
    <cylinder radius="0.045" length="0.015" />
@@ -18,4 +29,5 @@
    <inertia ixx="0.01"  ixy="0"  ixz="0" iyy="0.01" iyz="0" izz="0.01" />
 </xacro:my_link>
+<!--the box that connects the clavicle to the upper arm, roll rotation-->
 <xacro:my_link name="shoulder_link2_${whichside}" mass="0.1" color="Black">
    <box size="0.035 0.01 0.1" />
@@ -24,4 +36,5 @@
    <inertia ixx="0.001"  ixy="0"  ixz="0" iyy="0.001" iyz="0" izz="0.001" />
 </xacro:my_link>
+<!--the upper arm-->
 <xacro:my_link_texturedmesh name="upper_arm_${whichside}" mass="2.9" texture="white">
    <origin xyz="0.0 -0.2 0.0" rpy="0 0 0"/>
@@ -30,4 +43,6 @@
    <mesh filename="package://amigo_robot_model/arms_DH/upperarmtextured.dae" scale="0.001 0.001 0.001"/>
 </xacro:my_link_texturedmesh>
+<!--the elbow
+note: not visible, see arm_extra_visuals for the elbow visuals -->
 <xacro:my_link name="elbow_link4_${whichside}" mass="0.1" color="Grey">
    <cylinder radius="0.0" length="0.0"/>
@@ -36,4 +51,5 @@
    <inertia ixx="0.001"  ixy="0"  ixz="0" iyy="0.001" iyz="0" izz="0.001" />
 </xacro:my_link>
+<!--the forearm-->
 <xacro:my_link_texturedmesh name="fore_arm_${whichside}" mass="0.1" texture="white">
    <origin xyz="0.0 -0.14 0.0" rpy="0.0 0 0"/>
@@ -42,4 +58,6 @@
    <mesh filename="package://amigo_robot_model/arms_DH/forearmtextured.dae" scale="0.001 0.001 0.001"/>
 </xacro:my_link_texturedmesh>
+<!--the wrist
+note: not visible, see arm_extra_visuals for the wrist visuals -->
 <xacro:my_link name="wrist_link6_${whichside}" mass="0.01" color="Black">
    <cylinder radius="0.0" length="0.0"/>
@@ -48,4 +66,5 @@
    <inertia ixx="0.001"  ixy="0"  ixz="0" iyy="0.001" iyz="0" izz="0.001" />
 </xacro:my_link>
+<!--the hand -->
 <xacro:my_link name="hand_${whichside}" mass="0.2" color="Grey">
    <box size="0.080 0.085 0.038"/>
@@ -54,4 +73,5 @@
    <inertia ixx="0.01"  ixy="0"  ixz="0" iyy="0.01" iyz="0" izz="0.01" />
 </xacro:my_link>
+<!--the right finger-->
 <xacro:my_link name="finger1_${whichside}" mass="0.05" color="Black">
    <box size="0.02 0.022 0.11"/>
@@ -60,4 +80,5 @@
    <inertia ixx="0.00037"  ixy="0"  ixz="0" iyy="0.00052" iyz="0" izz="0.00052" />
 </xacro:my_link>
+<!--the left finger-->
 <xacro:my_link name="finger2_${whichside}" mass="0.05" color="Black">
    <box size="0.02 0.022 0.11"/>
@@ -66,4 +87,6 @@
    <inertia ixx="0.00037"  ixy="0"  ixz="0" iyy="0.00052" iyz="0" izz="0.00052" />
 </xacro:my_link>
+<!--the grippoint
+note: not visible, purely kinematic-->
 <xacro:my_link name="grippoint_${whichside}" mass="0.01" color="Blue">
    <box size="0.0 0.0 0.0"/>
@@ -72,5 +95,5 @@
    <inertia ixx="0.0001"  ixy="0"  ixz="0" iyy="0.0001" iyz="0" izz="0.0001" />
 </xacro:my_link>
-<!--Fill out Joint macros-->
+<!--the joints start here-->
   <joint name="shoulder_mount_joint_${whichside}" type="fixed">
     <parent link="torso"/>

File: body/body.urdf.xacro (robot description, xacro)
@@ -1,13 +1,16 @@
 <?xml version="1.0"?>
 <robot xmlns:xacro="http://ros.org/wiki/xacro">
-<!--body-->
-<xacro:my_link_texturedmesh_diff_coll name="base" mass="20" texture="bottomcovers">
-   <origin xyz="0.0 0.0 0.3275" rpy="0 0 0"/>
-   <origin xyz="0.0 0.0 0.23" rpy="0 0 -1.5708" />
-   <origin xyz="0.0 0.0 0.33" rpy="0 0 -1.5708" />
-   <inertia ixx="2.63"  ixy="0"  ixz="0" iyy="2.63" iyz="0" izz="2.4" /> <!--*-->
-   <mesh filename="package://amigo_robot_model/body/bottomcovers.dae" scale="0.001 0.001 0.001"/>
-   <box size="0.275 0.275 0.6"/>
-</xacro:my_link_texturedmesh_diff_coll>
+   <author>Rob Janssen, Kris van Tienhoven</author>
+   <license>BSD</license>
+   <review status="unreviewed" notes=""/>
+<!--links start here-->
+<!--the torso-->
+<xacro:my_link_texturedmesh name="torso" mass="16" texture="white">
+   <origin xyz="0.0 0.0 0.0" rpy="0 0 0"/>
+   <origin xyz="0.045 0.0 0.06" rpy="-1.5708 0 -1.5708" />
+   <inertia ixx="0.01"  ixy="0"  ixz="0" iyy="0.01" iyz="0" izz="0.01" />
+   <mesh filename="package://amigo_robot_model/body/torsocovers.dae" scale="0.001 0.001 0.001"/>
+</xacro:my_link_texturedmesh>
+<!--the spindle-->
 <xacro:my_link_texturedmesh name="torso_slider" mass="0.1" texture="aluminum">
    <origin xyz="0 0 0" rpy="0 0 0"/>
@@ -16,4 +19,15 @@
    <mesh filename="package://amigo_robot_model/body/torsoslidertextured.dae" scale="0.01 0.01 0.01"/>
 </xacro:my_link_texturedmesh>
+<!--the bottomcovers
+note: uses a different bounding box, because a normal one would be too inaccurate-->
+<xacro:my_link_texturedmesh_diff_coll name="base" mass="20" texture="bottomcovers">
+   <origin xyz="0.0 0.0 0.3275" rpy="0 0 0"/>
+   <origin xyz="0.0 0.0 0.23" rpy="0 0 -1.5708" />
+   <origin xyz="0.0 0.0 0.33" rpy="0 0 -1.5708" />
+   <inertia ixx="2.63"  ixy="0"  ixz="0" iyy="2.63" iyz="0" izz="2.4" />
+   <mesh filename="package://amigo_robot_model/body/bottomcovers.dae" scale="0.001 0.001 0.001"/>
+   <box size="0.275 0.275 0.6"/>
+</xacro:my_link_texturedmesh_diff_coll>
+<!--the root of the tf-tree, because it serves only this function it has no visuals-->
 <xacro:my_link name="base_link" mass="0" color="Red">
    <cylinder radius="0.0" length="0.00" />
@@ -22,4 +36,26 @@
    <inertia ixx="0"  ixy="0"  ixz="0" iyy="0" iyz="0" izz="0" />
 </xacro:my_link>
+<!-- joints start here -->
+  <joint name="spindle_joint" type="prismatic">
+    <parent link="base"/>
+    <child link="torso_slider"/>
+    <axis xyz="1 0 0"/>
+    <origin xyz="0.0 0.0 0.58" rpy="3.14159265 -1.5708 0"/>
+    <dynamics damping="3" friction="0.0"/> <!--*-->
+    <limit effort="30" velocity="1.0" lower="0.0" upper="0.41" /> <!--*-->
+  </joint>
+  <joint name="base_link_joint" type="fixed">
+    <parent link="base_link"/>
+    <child link="base"/>
+    <axis xyz="1 0 0"/>
+    <origin xyz="0.0 0.0 0.055" rpy="0 0 0"/>
+  </joint>
+    <joint name="torso_slider_joint" type="fixed">
+    <parent link="torso_slider"/>
+    <child link="torso"/>
+    <axis xyz="1 0 0"/>
+    <origin xyz="0.135 0.0 0.0" rpy="0 0 0"/>
+  </joint>
+<!--extra boundingbox for the batteries on the left-->
 <link name="batterycovercollision_left">
    <inertial>
@@ -47,4 +83,5 @@
     <origin xyz="0.0 0.25 0.1" rpy="0 0 0"/>
 </joint>
+<!--extra boundingbox for the batteries on the right-->
 <link name="batterycovercollision_right">
    <inertial>
@@ -72,5 +109,6 @@
     <origin xyz="0.0 -0.25 0.1" rpy="0 0 0"/>
 </joint>
-<link name="batterycovercollision_back">
+<!--extra boundingbox for the computers at the back-->
+<link name="computercovercollision">
    <inertial>
      <origin xyz="0.0 0.0 0.0" />
@@ -91,35 +129,9 @@
     </collision>
 </link>
-<joint name="batterycovercollision_back_joint" type="fixed">
+<joint name="computercovercollision_joint" type="fixed">
     <parent link="base"/>
-    <child link="batterycovercollision_back"/>
+    <child link="computercovercollision"/>
     <axis xyz="1 0 0"/>
     <origin xyz="-0.25 0.0 0.125" rpy="0 0 1.5708"/>
 </joint>
-<xacro:my_link_texturedmesh name="torso" mass="16" texture="white">
-   <origin xyz="0.0 0.0 0.0" rpy="0 0 0"/>
-   <origin xyz="0.045 0.0 0.06" rpy="-1.5708 0 -1.5708" />
-   <inertia ixx="0.01"  ixy="0"  ixz="0" iyy="0.01" iyz="0" izz="0.01" /> <!--*-->
-   <mesh filename="package://amigo_robot_model/body/torsocovers.dae" scale="0.001 0.001 0.001"/>
-</xacro:my_link_texturedmesh>
-  <joint name="spindle_joint" type="prismatic">
-    <parent link="base"/>
-    <child link="torso_slider"/>
-    <axis xyz="1 0 0"/>
-    <origin xyz="0.0 0.0 0.58" rpy="3.14159265 -1.5708 0"/>
-    <dynamics damping="3" friction="0.0"/> <!--*-->
-    <limit effort="30" velocity="1.0" lower="0.0" upper="0.41" /> <!--*-->
-  </joint>
-  <joint name="base_link_joint" type="fixed">
-    <parent link="base_link"/>
-    <child link="base"/>
-    <axis xyz="1 0 0"/>
-    <origin xyz="0.0 0.0 0.055" rpy="0 0 0"/>
-  </joint>
-    <joint name="torso_slider_joint" type="fixed">
-    <parent link="torso_slider"/>
-    <child link="torso"/>
-    <axis xyz="1 0 0"/>
-    <origin xyz="0.135 0.0 0.0" rpy="0 0 0"/>
-  </joint>
 </robot>

File: body_extra_visuals/body_extra.urdf.xacro (robot description, xacro)
@@ -1,5 +1,8 @@
 <?xml version="1.0"?>
 <robot xmlns:xacro="http://ros.org/wiki/xacro">
-<!--base plate-->
+   <author>Kris van Tienhoven</author>
+   <license>BSD</license>
+   <review status="unreviewed" notes=""/>
+<!--base plate at the bottom of the bottomcovers-->
 <xacro:my_link_textured name="base_plate" mass="0.1" texture="aluminum">
    <cylinder radius="0.333" length="0.02" />
@@ -14,5 +17,6 @@
     <origin xyz="0.0 0.0 0.05" rpy="0 0 0"/>
   </joint>
-<!--torso sliders-->
+<!--the extra sliders next to and behind the spindle-->
+<!--right link-->
 <xacro:my_link_texturedmesh name="torso_assist_slider_right" mass="0.01" texture="aluminum">
    <origin xyz="0 0 0" rpy="0 0 0"/>
@@ -21,4 +25,5 @@
    <mesh filename="package://amigo_robot_model/body_extra_visuals/torsoassistslidertextured.dae" scale="0.01 0.01 0.0125"/>
 </xacro:my_link_texturedmesh>
+<!--left link-->
 <xacro:my_link_texturedmesh name="torso_assist_slider_left" mass="0.01" texture="aluminum">
    <origin xyz="0 0 0" rpy="0 0 0"/>
@@ -27,4 +32,5 @@
    <mesh filename="package://amigo_robot_model/body_extra_visuals/torsoassistslidertextured.dae" scale="0.01 0.01 0.0125"/>
 </xacro:my_link_texturedmesh>
+<!--back link-->
 <xacro:my_link_texturedmesh name="torso_assist_slider_back" mass="0.01" texture="aluminum">
    <origin xyz="0 0 0" rpy="0 0 0"/>
@@ -33,4 +39,5 @@
    <mesh filename="package://amigo_robot_model/body_extra_visuals/torsoassistslidertextured.dae" scale="0.01 0.01 0.0125"/>
 </xacro:my_link_texturedmesh>
+<!--left joint-->
 <joint name="torso_slider_assist_joint_right" type="fixed">
     <parent link="torso"/>
@@ -38,4 +45,5 @@
     <origin xyz="-0.3 0.1 0.0" rpy="0 0 0"/>
 </joint>
+<!--right joint-->
 <joint name="torso_slider_assist_joint_left" type="fixed">
     <parent link="torso"/>
@@ -43,4 +51,5 @@
     <origin xyz="-0.3 -0.1 0.0" rpy="0 0 0"/>
 </joint>
+<!--back joint-->
 <joint name="torso_slider_assist_joint_back" type="fixed">
     <parent link="torso"/>
@@ -60,5 +69,6 @@
     <origin xyz="0.05 0.0 0.0" rpy="0 0 0"/>
 </joint>
-<!--closing up the torso-->
+<!--the geometry that seals the torso-->
+<!--right-->
 <xacro:my_link name="closure_right" mass="0.01" color="White">
    <box size="0.12 0.004 0.155"/>
@@ -72,4 +82,5 @@
     <origin xyz="0.045 0.12 0.0" rpy="0 0 0"/>
 </joint>
+<!--left-->
 <xacro:my_link name="closure_left" mass="0.01" color="White">
    <box size="0.12 0.004 0.155"/>
@@ -83,4 +94,5 @@
     <origin xyz="0.045 -0.12 0.0" rpy="0 0 0"/>
 </joint>
+<!--bottom-->
 <xacro:my_link name="closure_bottom" mass="0.01" color="White">
    <cylinder radius="0.1" length="0.004"/>

File: definitions.xacro (robot description, xacro)
@@ -1,5 +1,9 @@
 <?xml version="1.0"?>
 <robot xmlns:xacro="http://ros.org/wiki/xacro">
-<!-- *************** LINK Definition *****************-->
+<!-- *************** LINK Definitions *****************-->
+   <author>Kris van Tienhoven</author>
+   <license>BSD</license>
+   <review status="unreviewed" notes=""/>
+<!--use this type of link for standard shapes (bos, cylinder, sphere) with standard color -->
 <xacro:macro name="my_link" params="name mass color *type *origin *visualorigin *inertia">
   <link name="${name}">
@@ -29,4 +33,5 @@
     </gazebo>
 </xacro:macro>
+<!-- use this type of link if you want the standard shapes with a texture -->
 <xacro:macro name="my_link_textured" params="name mass texture *type *origin *visualorigin *inertia">
   <link name="${name}">
@@ -56,4 +61,5 @@
     </gazebo>
 </xacro:macro>
+<!--use this type of link for shapes that need to be collision free and thereby also invisible -->
 <xacro:macro name="my_link_coll_free" params="name mass color *type *origin *visualorigin *inertia">
   <link name="${name}">
@@ -77,4 +83,5 @@
     </gazebo>
 </xacro:macro>
+<!--use this type of link if you want to load a mesh with a standard color -->
 <xacro:macro name="my_link_mesh" params="name mass color *origin *visualorigin *inertia *mesh">
   <link name="${name}">
@@ -104,4 +111,5 @@
     </gazebo>
 </xacro:macro>
+<!-- use this type of link if you want to load a mesh with a texture -->
 <xacro:macro name="my_link_texturedmesh" params="name mass texture *origin *visualorigin *inertia *mesh">
   <link name="${name}">
@@ -130,4 +138,5 @@
     </gazebo>
 </xacro:macro>
+<!-- use this type of link if you want a mesh with texture and a different bouding box (then the box around the mesh itself) -->
 <xacro:macro name="my_link_texturedmesh_diff_coll" params="name mass texture *origin *visualorigin *collorigin *inertia *mesh *type">
   <link name="${name}">

File: head/head.urdf.xacro (robot description, xacro)
@@ -1,5 +1,9 @@
 <?xml version="1.0"?>
 <robot xmlns:xacro="http://ros.org/wiki/xacro">
-<!--body-->
+   <author>Kris van Tienhoven</author>
+   <license>BSD</license>
+   <review status="unreviewed" notes=""/>
+<!--head-->
+<!-- !!!!!!!!!something without a visual not sure what this is!!!!!!!!!!!! -->
 <xacro:my_link name="head_mount" mass="0.05" color="Blue">
    <box size="0.01 0.01  0.01 " />
@@ -8,4 +12,11 @@
    <inertia ixx="0.0001"  ixy="0"  ixz="0" iyy="0.0001" iyz="0" izz="0.0001" /> <!--*-->
 </xacro:my_link>
+  <joint name="head_mount_joint" type="fixed">
+    <parent link="torso"/>
+    <child link="head_mount"/>
+    <axis xyz="0 0 1"/>
+    <origin xyz="0.097 0.0 0.0" rpy="  0.0 0.0 0.0"/>
+  </joint>
+<!-- the link that represents the panning part of the neck, is below neck_tilt -->
 <xacro:my_link name="neck_pan" mass="0.05" color="Black">
    <cylinder radius="0.015" length="0.0525" /> <!--*--> <!--checked-->
@@ -15,4 +26,5 @@
    <color rgba="0.25 0.25 0.25 1.0"/>
 </xacro:my_link>
+<!-- the link that represents the tilting part of the neck, is above neck_pan -->
 <xacro:my_link_texturedmesh name="neck_tilt" mass="0.05" texture="aluminum">
    <origin xyz="0.0 -0.0 0.0285" rpy="0 0 0"/>
@@ -21,4 +33,5 @@
    <mesh filename="package://amigo_robot_model/head/necktilttextured.dae" scale="0.01 0.01 0.01"/>
 </xacro:my_link_texturedmesh>
+<!--the head itself-->
  <my_link_texturedmesh name="head" mass="0" texture="white">
    <origin xyz="0 0 0" rpy="0 0 0"/>
@@ -27,14 +40,9 @@
    <mesh filename="package://amigo_robot_model/head/headtextured.dae" scale="0.001 0.001 0.001"/>
   </my_link_texturedmesh>
-  <joint name="head_mount_joint" type="fixed">
-    <parent link="torso"/>
-    <child link="head_mount"/>
-    <axis xyz="0 0 1"/>
-    <origin xyz="0.097 0.0 0.0" rpy="  0.0 0.0 0.0"/>
-  </joint>
   <joint name="head_joint" type="fixed">
     <parent link="neck_tilt"/>
     <child link="head"/>
   </joint>
+<!-- the tilt and pan joints-->
 <xacro:my_joint name="neck_pan_joint" type="revolute" parent="head_mount" child="neck_pan">
    <origin xyz="0.0 0.0 0.0" rpy="3.14 -1.5708 0.0"/> <!--checked-->

File: laser/laser.urdf.xacro (robot description, xacro)
@@ -1,4 +1,8 @@
 <?xml version="1.0"?>
 <robot xmlns:xacro="http://ros.org/wiki/xacro">
+   <author>Kris van Tienhoven</author>
+   <license>BSD</license>
+   <review status="unreviewed" notes=""/>
+<!--the laser at the base of the robot -->
 <xacro:my_link name="base_laser" mass="0.5" color="Black">
    <box size="0.05 0.065 0.12" /> <!--*-->
@@ -13,4 +17,5 @@
    <limit effort="13.4" velocity="1.0" lower="-0.7809" upper="1.5708" />
 </xacro:my_joint>
+<!--the orange top of the laser-->
 <xacro:my_link_textured name="lasertop" mass="0.01" texture="orange">
    <box size="0.05 0.065 0.01" /> <!--*-->
@@ -23,4 +28,5 @@
     <child link="lasertop"/>
 </joint>
+<!--the tue logo in front of the laser-->
 <xacro:my_link_texturedmesh name="logo" mass="0.01" texture="logo">
    <origin xyz="0.0 0.0 0.0" rpy="0 0 0"/>

File: materials.urdf.xacro (robot description, xacro)
@@ -1,4 +1,8 @@
 <?xml version="1.0"?>
 <robot>
+   <author>Kris van Tienhoven</author>
+   <license>BSD</license>
+   <review status="unreviewed" notes=""/>
+<!-- this files contains the definitions for all colors and textures for rviz -->
   <material name="Blue">
     <color rgba="0.0 0.0 0.8 1.0"/>

File: robot.urdf.xacro (robot description, xacro)
@@ -4,4 +4,7 @@
        xmlns:controller="http://playerstage.sourceforge.net/gazebo/xmlschema/#controller"
        xmlns:interface="http://playerstage.sourceforge.net/gazebo/xmlschema/#interface">
+   <author>Rob Janssen</author>
+   <license>BSD</license>
+   <review status="unreviewed" notes=""/>
 <!--get plugins -->
 <include filename="$(find amigo_robot_model)/gazebo/gazebo.urdf.xacro" />

File: wheels/wheels.urdf.xacro (robot description, xacro)
@@ -1,5 +1,13 @@
 <?xml version="1.0"?>
 <robot xmlns:xacro="http://ros.org/wiki/xacro">
-<!--wheels-->
+   <author>Kris van Tienhoven</author>
+   <license>BSD</license>
+   <review status="unreviewed" notes=""/>
+<!--Start of the macro for the four cylinders that are the wheels
+@param side_LR is "left"  or "right"
+@param side_FR is "front" or "rear"
+@param sign_LR is - or +
+@param sign_FR is - or +
+@param wheel_angle is the initial rotation of the wheel -->
 <xacro:macro name="wheel" params="side_LR side_FR sign_LR sign_FR wheel_angle">
   <joint name="wheel_inner_joint_${side_LR}_${side_FR}" type="continuous">
@@ -18,4 +26,11 @@
    </xacro:my_link>
 </xacro:macro>
+<!--Start of the macro for the 12 spheres on each wheel
+@param side_LR is "left"  or "right"
+@param side_FR is "front" or "rear"
+@param number is a integer out of the interval [1...12]
+@param y_ is the y position of the sphere
+@param z_ is the z position of the wheel
+@param roll_ is the initial rotation of the sphere -->
 <xacro:macro name="z_sphere" params="side_LR side_FR number y_ z_ roll_">
 	<joint name="omni_sphere${number}_joint_${side_LR}_${side_FR}" type="continuous">
@@ -34,4 +49,9 @@
 	</xacro:my_link>
 </xacro:macro>
+<!--the macro that calls the macro for a sphere for each wheel
+@param nr is a integer out of the interval [1...12]
+@param y is the y position of the sphere
+@param z is the z position of the wheel
+@param roll is the initial rotation of the sphere -->
 <xacro:macro name="spheres" params="nr y z roll">
   <xacro:z_sphere side_LR="left" side_FR="front" number="${nr}" y_="${y}" z_="${z}" roll_="${roll}"/>
@@ -40,4 +60,5 @@
   <xacro:z_sphere side_LR="right" side_FR="rear" number="${nr}" y_="${y}" z_="${z}" roll_="${roll}"/>
 </xacro:macro>
+<!--calling the macro to create a sphere for each wheel 12 times-->
 <xacro:spheres nr="1" y="0.03" z="0.0" roll="0.0"/>
 <xacro:spheres nr="2" y="0.026" z="0.015" roll="0.5236"/>
