Commit message: Kinect urdf update
git-svn-id: https://roboticssrv.wtb.tue.nl/svn/ros/code/tue-ros-pkg/trunk/tue_robot_models/amigo_robot_model@7894 3a3c2cfb-d3b9-409e-9e75-db8fcdbcaac6

File: head/head.urdf.xacro (robot description, xacro)
@@ -16,5 +16,5 @@
     <child link="head_mount"/>
     <axis xyz="0 0 1"/>
-    <origin xyz="0.097 0.0 0.0" rpy="  0.0 0.0 0.0"/>
+    <origin xyz="0.097 0.0 0.045" rpy="  0.0 0.0 0.0"/>
   </joint>
 <!-- the link that represents the panning part of the neck, is below neck_tilt -->

File: kinect/kinect.urdf.xacro (robot description, xacro)
@@ -6,5 +6,5 @@
   <property name="M_PI" value="3.14159"/>
   <joint name="base_kinect_joint" type="fixed">
-    <origin xyz="0.07 0 0.07" rpy="0 0 0" /> <!-- THESE VALUES ARE ROUGH ESTIMATES!! -->
+    <origin xyz="0.035 0 0.07" rpy="0 0 0" /> <!-- THESE VALUES ARE ROUGH ESTIMATES!! -->
     <parent link="head" />
     <child link="openni_camera" />

Commit message: Updated kinect urdf
git-svn-id: https://roboticssrv.wtb.tue.nl/svn/ros/code/tue-ros-pkg/trunk/tue_robot_models/amigo_robot_model@7896 3a3c2cfb-d3b9-409e-9e75-db8fcdbcaac6

File: head/head.urdf.xacro (robot description, xacro)
@@ -16,5 +16,5 @@
     <child link="head_mount"/>
     <axis xyz="0 0 1"/>
-    <origin xyz="0.097 0.0 0.045" rpy="  0.0 0.0 0.0"/>
+    <origin xyz="0.107 0.0 0.045" rpy="  0.0 0.0 0.0"/>
   </joint>
 <!-- the link that represents the panning part of the neck, is below neck_tilt -->

File: kinect/kinect.urdf.xacro (robot description, xacro)
@@ -6,5 +6,5 @@
   <property name="M_PI" value="3.14159"/>
   <joint name="base_kinect_joint" type="fixed">
-    <origin xyz="0.035 0 0.07" rpy="0 0 0" /> <!-- THESE VALUES ARE ROUGH ESTIMATES!! -->
+    <origin xyz="0.027 0 0.06" rpy="0 0 0" /> <!-- THESE VALUES ARE ROUGH ESTIMATES!! -->
     <parent link="head" />
     <child link="openni_camera" />

Commit message: Removed block in urdf
git-svn-id: https://roboticssrv.wtb.tue.nl/svn/ros/code/tue-ros-pkg/trunk/tue_robot_models/amigo_robot_model@7963 3a3c2cfb-d3b9-409e-9e75-db8fcdbcaac6

File: head/head.urdf.xacro (robot description, xacro)
@@ -6,10 +6,17 @@
 <!--head-->
 <!-- !!!!!!!!!something without a visual not sure what this is!!!!!!!!!!!! -->
-<xacro:my_link name="head_mount" mass="0.05" color="Blue">
+<!--<xacro:my_link name="head_mount" mass="0.05" color="Blue">
    <box size="0.01 0.01  0.01 " />
    <origin xyz="0.0 0.0 0.0" rpy="0 0 0"/>
    <origin xyz="0.0 0.0 0.0" rpy="0 0 0" />
-   <inertia ixx="0.0001"  ixy="0"  ixz="0" iyy="0.0001" iyz="0" izz="0.0001" /> <!--*-->
-</xacro:my_link>
+   <inertia ixx="0.0001"  ixy="0"  ixz="0" iyy="0.0001" iyz="0" izz="0.0001" />
+</xacro:my_link>-->
+<link name="head_mount">
+  <inertial>
+`   <origin xyz="0 0 0" rpy="0 0 0"/>
+    <mass value="0.001"/>
+    <inertia ixx="0.001"  ixy="0"  ixz="0" iyy="0.001" iyz="0" izz="0.001" />
+  </inertial>
+</link>
   <joint name="head_mount_joint" type="fixed">
     <parent link="torso"/>
