Commit message: simulated kinect
git-svn-id: https://roboticssrv.wtb.tue.nl/svn/ros/code/tue-ros-pkg/trunk/tue_robot_models/amigo_robot_model@8790 3a3c2cfb-d3b9-409e-9e75-db8fcdbcaac6

File: gazebo/gazebo.urdf.xacro (robot description, xacro)
@@ -141,6 +141,6 @@
     </sensor:camera>
   </gazebo>
-  <gazebo reference="base_kinect_openni_camera">
-    <sensor:camera name="base_kinect_openni_camera">
+  <gazebo reference="base_camera_openni_camera">
+    <sensor:camera name="base_camera_openni_camera">
       <imageFormat>R8G8B8</imageFormat>
       <imageSize>640 480</imageSize>
@@ -150,5 +150,5 @@
       <updateRate>20</updateRate>
       <baseline>0.1</baseline>
-      <controller:gazebo_ros_openni_kinect name="base_kinect_kinect_camera_controller" plugin="libgazebo_ros_openni_kinect.so">
+      <controller:gazebo_ros_openni_kinect name="base_camera_openni_camera_controller" plugin="libgazebo_ros_openni_kinect.so">
         <alwaysOn>true</alwaysOn>
         <updateRate>20</updateRate>
@@ -157,5 +157,5 @@
         <pointCloudTopicName>/base_camera/camera/rgb/points_throttled_and_voxelized</pointCloudTopicName>
         <cameraInfoTopicName>/base_camera/camera/rgb/camera_info</cameraInfoTopicName>
-        <frameName>/base_camera_depth_optical_frame</frameName>
+        <frameName>/base_camera_openni_depth_optical_frame</frameName>
         <!--<distortion_k1>0.00000001</distortion_k1>
         <distortion_k2>0.00000001</distortion_k2>

File: kinect/base_kinect.urdf.xacro (robot description, xacro)
@@ -5,10 +5,10 @@
       xmlns:xacro="http://ros.org/wiki/xacro">
   <property name="M_PI" value="3.14159"/>
-  <joint name="base_kinect_base_kinect_joint" type="fixed">
+  <joint name="base_camera_openni_joint" type="fixed">
     <origin xyz="0.29 0 0.31" rpy="0 -0.07 0" /> <!-- THESE VALUES ARE ROUGH ESTIMATES!! -->
     <parent link="base_link" />
-    <child link="base_kinect_openni_camera" />
+    <child link="base_camera_openni_camera" />
   </joint>
-  <link name="base_kinect_openni_camera">
+  <link name="base_camera_openni_camera">
     <inertial>
       <mass value="0.01" />
@@ -35,10 +35,10 @@
     </collision>
   </link>
-  <joint name="base_kinect_kinect_depth_joint" type="fixed">
+  <joint name="base_camera_openni_depth_joint" type="fixed">
     <origin xyz="0 0.018 0" rpy="0 0 0" />
-    <parent link="base_kinect_openni_camera" />
-    <child link="base_kinect_openni_depth_frame" />
+    <parent link="base_camera_openni_camera" />
+    <child link="base_camera_openni_depth_frame" />
   </joint>
-  <link name="base_kinect_openni_depth_frame">
+  <link name="base_camera_openni_depth_frame">
     <inertial>
       <mass value="0.01" />
@@ -49,10 +49,10 @@
     </inertial>
   </link>
-  <joint name="base_kinect_kinect_depth_optical_joint" type="fixed">
+  <joint name="base_camera_openni_depth_optical_joint" type="fixed">
     <origin xyz="0 0 0" rpy="${-M_PI/2} 0 ${-M_PI/2}" />
-    <parent link="base_kinect_openni_depth_frame" />
-    <child link="base_kinect_openni_depth_optical_frame" />
+    <parent link="base_camera_openni_depth_frame" />
+    <child link="base_camera_openni_depth_optical_frame" />
   </joint>
-  <link name="base_kinect_openni_depth_optical_frame">
+  <link name="base_camera_openni_depth_optical_frame">
     <inertial>
       <mass value="0.001" />
@@ -63,10 +63,10 @@
     </inertial>
   </link>
-  <joint name="base_kinect_kinect_rgb_joint" type="fixed">
+  <joint name="base_camera_openni_rgb_joint" type="fixed">
     <origin xyz="0 -0.005 0" rpy="0 0 0" />
-    <parent link="base_kinect_openni_camera" />
-    <child link="base_kinect_openni_rgb_frame" />
+    <parent link="base_camera_openni_camera" />
+    <child link="base_camera_openni_rgb_frame" />
   </joint>
-  <link name="base_kinect_openni_rgb_frame">
+  <link name="base_camera_openni_rgb_frame">
     <inertial>
       <mass value="0.001" />
@@ -77,10 +77,10 @@
     </inertial>
   </link>
-  <joint name="base_kinect_kinect_rgb_optical_joint" type="fixed">
+  <joint name="base_camera_openni_rgb_optical_joint" type="fixed">
     <origin xyz="0 0 0" rpy="${-M_PI/2} 0 ${-M_PI/2}" />
-    <parent link="base_kinect_openni_rgb_frame" />
-    <child link="base_kinect_openni_rgb_optical_frame" />
+    <parent link="base_camera_openni_rgb_frame" />
+    <child link="base_camera_openni_rgb_optical_frame" />
   </joint>
-  <link name="base_kinect_openni_rgb_optical_frame">
+  <link name="base_camera_openni_rgb_optical_frame">
     <inertial>
       <mass value="0.001" />

Commit message: sdfsdf
git-svn-id: https://roboticssrv.wtb.tue.nl/svn/ros/code/tue-ros-pkg/trunk/tue_robot_models/amigo_robot_model@8794 3a3c2cfb-d3b9-409e-9e75-db8fcdbcaac6

File: gazebo/gazebo.urdf.xacro (robot description, xacro)
@@ -141,6 +141,6 @@
     </sensor:camera>
   </gazebo>
-  <gazebo reference="base_camera_openni_camera">
-    <sensor:camera name="base_camera_openni_camera">
+  <gazebo reference="base_kinect_openni_camera">
+    <sensor:camera name="base_kinect_openni_camera">
       <imageFormat>R8G8B8</imageFormat>
       <imageSize>640 480</imageSize>
@@ -150,5 +150,5 @@
       <updateRate>20</updateRate>
       <baseline>0.1</baseline>
-      <controller:gazebo_ros_openni_kinect name="base_camera_openni_camera_controller" plugin="libgazebo_ros_openni_kinect.so">
+      <controller:gazebo_ros_openni_kinect name="base_kinect_kinect_camera_controller" plugin="libgazebo_ros_openni_kinect.so">
         <alwaysOn>true</alwaysOn>
         <updateRate>20</updateRate>
@@ -157,5 +157,5 @@
         <pointCloudTopicName>/base_camera/camera/rgb/points_throttled_and_voxelized</pointCloudTopicName>
         <cameraInfoTopicName>/base_camera/camera/rgb/camera_info</cameraInfoTopicName>
-        <frameName>/base_camera_openni_depth_optical_frame</frameName>
+        <frameName>/base_camera_depth_optical_frame</frameName>
         <!--<distortion_k1>0.00000001</distortion_k1>
         <distortion_k2>0.00000001</distortion_k2>

File: kinect/base_kinect.urdf.xacro (robot description, xacro)
@@ -5,10 +5,10 @@
       xmlns:xacro="http://ros.org/wiki/xacro">
   <property name="M_PI" value="3.14159"/>
-  <joint name="base_camera_openni_joint" type="fixed">
+  <joint name="base_kinect_base_kinect_joint" type="fixed">
     <origin xyz="0.29 0 0.31" rpy="0 -0.07 0" /> <!-- THESE VALUES ARE ROUGH ESTIMATES!! -->
     <parent link="base_link" />
-    <child link="base_camera_openni_camera" />
+    <child link="base_kinect_openni_camera" />
   </joint>
-  <link name="base_camera_openni_camera">
+  <link name="base_kinect_openni_camera">
     <inertial>
       <mass value="0.01" />
@@ -35,10 +35,10 @@
     </collision>
   </link>
-  <joint name="base_camera_openni_depth_joint" type="fixed">
+  <joint name="base_kinect_kinect_depth_joint" type="fixed">
     <origin xyz="0 0.018 0" rpy="0 0 0" />
-    <parent link="base_camera_openni_camera" />
-    <child link="base_camera_openni_depth_frame" />
+    <parent link="base_kinect_openni_camera" />
+    <child link="base_kinect_openni_depth_frame" />
   </joint>
-  <link name="base_camera_openni_depth_frame">
+  <link name="base_kinect_openni_depth_frame">
     <inertial>
       <mass value="0.01" />
@@ -49,10 +49,10 @@
     </inertial>
   </link>
-  <joint name="base_camera_openni_depth_optical_joint" type="fixed">
+  <joint name="base_kinect_kinect_depth_optical_joint" type="fixed">
     <origin xyz="0 0 0" rpy="${-M_PI/2} 0 ${-M_PI/2}" />
-    <parent link="base_camera_openni_depth_frame" />
-    <child link="base_camera_openni_depth_optical_frame" />
+    <parent link="base_kinect_openni_depth_frame" />
+    <child link="base_kinect_openni_depth_optical_frame" />
   </joint>
-  <link name="base_camera_openni_depth_optical_frame">
+  <link name="base_kinect_openni_depth_optical_frame">
     <inertial>
       <mass value="0.001" />
@@ -63,10 +63,10 @@
     </inertial>
   </link>
-  <joint name="base_camera_openni_rgb_joint" type="fixed">
+  <joint name="base_kinect_kinect_rgb_joint" type="fixed">
     <origin xyz="0 -0.005 0" rpy="0 0 0" />
-    <parent link="base_camera_openni_camera" />
-    <child link="base_camera_openni_rgb_frame" />
+    <parent link="base_kinect_openni_camera" />
+    <child link="base_kinect_openni_rgb_frame" />
   </joint>
-  <link name="base_camera_openni_rgb_frame">
+  <link name="base_kinect_openni_rgb_frame">
     <inertial>
       <mass value="0.001" />
@@ -77,10 +77,10 @@
     </inertial>
   </link>
-  <joint name="base_camera_openni_rgb_optical_joint" type="fixed">
+  <joint name="base_kinect_kinect_rgb_optical_joint" type="fixed">
     <origin xyz="0 0 0" rpy="${-M_PI/2} 0 ${-M_PI/2}" />
-    <parent link="base_camera_openni_rgb_frame" />
-    <child link="base_camera_openni_rgb_optical_frame" />
+    <parent link="base_kinect_openni_rgb_frame" />
+    <child link="base_kinect_openni_rgb_optical_frame" />
   </joint>
-  <link name="base_camera_openni_rgb_optical_frame">
+  <link name="base_kinect_openni_rgb_optical_frame">
     <inertial>
       <mass value="0.001" />
