Commit message: Update amigo_robot_model and arm controller in simulation_controllers
git-svn-id: https://roboticssrv.wtb.tue.nl/svn/ros/code/tue-ros-pkg/trunk/tue_robot_models/amigo_robot_model@10896 3a3c2cfb-d3b9-409e-9e75-db8fcdbcaac6

File: description/arms/arm.transmission.xacro (robot description, xacro)
@@ -56,4 +56,16 @@
                 <motorTorqueConstant>1</motorTorqueConstant>
         </transmission>
+        <transmission name="finger1_tip_trans_${side}" type="pr2_mechanism_model/SimpleTransmission">
+                <actuator name="finger1_tip_motor_${side}" />
+                <joint name="finger1_tip_joint_${side}" />
+                <mechanicalReduction>1</mechanicalReduction>
+                <motorTorqueConstant>1</motorTorqueConstant>
+        </transmission>
+        <transmission name="finger2_tip_trans_${side}" type="pr2_mechanism_model/SimpleTransmission">
+                <actuator name="finger2_tip_motor_${side}" />
+                <joint name="finger2_tip_joint_${side}" />
+                <mechanicalReduction>1</mechanicalReduction>
+                <motorTorqueConstant>1</motorTorqueConstant>
+        </transmission>
 </xacro:macro>
 <xacro:arm_trans side="left"/>

File: description/arms/arm.urdf.xacro (robot description, xacro)
@@ -75,14 +75,28 @@
 <!--the right finger-->
 <xacro:my_link name="finger1_${whichside}" mass="0.05" color="Black">
-   <box size="0.02 0.022 0.11"/>
-   <origin xyz="0.0 0.0 -0.055" rpy="0 0 0"/>
-   <origin xyz="0.0 0.0 -0.055" rpy="0 0 0" />
+   <box size="0.018 0.018 0.06"/>
+   <origin xyz="0.0 0.0 -0.03" rpy="0 0 0"/>
+   <origin xyz="0.0 0.0 -0.03" rpy="0 0 0" />
+   <inertia ixx="0.01"  ixy="0"  ixz="0" iyy="0.01" iyz="0" izz="0.01" />
+</xacro:my_link>
+<!--the right finger tip-->
+<xacro:my_link name="finger1_tip_${whichside}" mass="0.05" color="Black">
+   <box size="0.018 0.018 0.06"/>
+   <origin xyz="0.0 0.0 -0.03" rpy="0 0 0"/>
+   <origin xyz="0.0 0.0 -0.03" rpy="0 0 0" />
    <inertia ixx="0.00037"  ixy="0"  ixz="0" iyy="0.00052" iyz="0" izz="0.00052" />
 </xacro:my_link>
 <!--the left finger-->
 <xacro:my_link name="finger2_${whichside}" mass="0.05" color="Black">
-   <box size="0.02 0.022 0.11"/>
-   <origin xyz="0.0 0.0 -0.055" rpy="0 0 0"/>
-   <origin xyz="0.0 0.0 -0.055" rpy="0 0 0" />
+   <box size="0.018 0.018 0.06"/>
+   <origin xyz="0.0 0.0 -0.03" rpy="0 0 0"/>
+   <origin xyz="0.0 0.0 -0.03" rpy="0 0 0" />
+   <inertia ixx="0.01"  ixy="0"  ixz="0" iyy="0.01" iyz="0" izz="0.01" />
+</xacro:my_link>
+<!--the left finger tip -->
+<xacro:my_link name="finger2_tip_${whichside}" mass="0.05" color="Black">
+   <box size="0.018 0.018 0.06"/>
+   <origin xyz="0.0 0.0 -0.03" rpy="0 0 0"/>
+   <origin xyz="0.0 0.0 -0.03" rpy="0 0 0" />
    <inertia ixx="0.00037"  ixy="0"  ixz="0" iyy="0.00052" iyz="0" izz="0.00052" />
 </xacro:my_link>
@@ -144,14 +158,26 @@
 </xacro:my_joint>
 <xacro:my_joint name="finger1_joint_${whichside}" type="revolute" parent="hand_${whichside}" child="finger1_${whichside}">
-   <origin xyz=" 0.075 0.04 0" rpy="0 -1.57 0"/>
-   <dynamics damping="0.5" friction="1.0"/>
-   <axis xyz="1 0 0"/>
-   <limit effort="3" velocity="1.0" lower="-0.3" upper="0.3"/>
+   <origin xyz=" 0.075 0.02 0" rpy="0 -1.57 0"/>
+   <dynamics damping="0.5" friction="1.0"/>
+   <axis xyz="1 0 0"/>
+   <limit effort="3" velocity="1.0" lower="-1.57" upper="1.57"/>
+</xacro:my_joint>
+<xacro:my_joint name="finger1_tip_joint_${whichside}" type="revolute" parent="finger1_${whichside}" child="finger1_tip_${whichside}">
+   <origin xyz=" 0 0.0 -0.06" rpy="0 0 0"/>
+   <dynamics damping="0.5" friction="1.0"/>
+   <axis xyz="1 0 0"/>
+   <limit effort="3" velocity="1.0" lower="-1.57" upper="1.57"/>
 </xacro:my_joint>
 <xacro:my_joint name="finger2_joint_${whichside}" type="revolute" parent="hand_${whichside}" child="finger2_${whichside}">
-   <origin xyz="0.075 -0.04 0" rpy="0 -1.57 0"/>
-   <dynamics damping="0.5" friction="1.0"/>
-   <axis xyz="1 0 0"/>
-   <limit effort="3" velocity="1.0" lower="-0.3" upper="0.3"/>
+   <origin xyz="0.075 -0.02 0" rpy="0 -1.57 0"/>
+   <dynamics damping="0.5" friction="1.0"/>
+   <axis xyz="1 0 0"/>
+   <limit effort="3" velocity="1.0" lower="-1.57" upper="1.57"/>
+</xacro:my_joint>
+<xacro:my_joint name="finger2_tip_joint_${whichside}" type="revolute" parent="finger2_${whichside}" child="finger2_tip_${whichside}">
+   <origin xyz="0 0 -0.06" rpy="0 0 0"/>
+   <dynamics damping="0.5" friction="1.0"/>
+   <axis xyz="1 0 0"/>
+   <limit effort="3" velocity="1.0" lower="-1.57" upper="1.57"/>
 </xacro:my_joint>
   <joint name="grippoint_joint_${whichside}" type="fixed">
@@ -161,3 +187,20 @@
   </joint>
 </xacro:macro>
+<!-- Friction Gripper -->
+<gazebo reference="finger1_right">
+	<mu1 value="100.0" />
+	<mu2 value="100.0" />
+</gazebo>
+<gazebo reference="finger1_tip_right">
+	<mu1 value="100.0" />
+	<mu2 value="100.0" />
+</gazebo>
+<gazebo reference="finger2_right">
+	<mu1 value="100.0" />
+	<mu2 value="100.0" />
+</gazebo>
+<gazebo reference="finger2_tip_right">
+	<mu1 value="100.0" />
+	<mu2 value="100.0" />
+</gazebo>
 </robot>

File: description/body_extra_visuals/body_extra.urdf.xacro (robot description, xacro)
@@ -71,5 +71,5 @@
 <!--the geometry that seals the torso-->
 <!--right-->
-<xacro:my_link name="closure_right" mass="0.01" color="White">
+<!--<xacro:my_link name="closure_right" mass="0.01" color="White">
    <box size="0.12 0.004 0.155"/>
    <origin xyz="0 0 0" rpy="0 0 0"/>
@@ -81,7 +81,7 @@
     <child link="closure_right"/>
     <origin xyz="0.045 0.12 0.0" rpy="0 0 0"/>
-</joint>
+</joint>-->
 <!--left-->
-<xacro:my_link name="closure_left" mass="0.01" color="White">
+<!--<xacro:my_link name="closure_left" mass="0.01" color="White">
    <box size="0.12 0.004 0.155"/>
    <origin xyz="0 0 0" rpy="0 0 0"/>
@@ -93,7 +93,7 @@
     <child link="closure_left"/>
     <origin xyz="0.045 -0.12 0.0" rpy="0 0 0"/>
-</joint>
+</joint>-->
 <!--bottom-->
-<xacro:my_link name="closure_bottom" mass="0.01" color="White">
+<!--<xacro:my_link name="closure_bottom" mass="0.01" color="White">
    <cylinder radius="0.1" length="0.004"/>
    <origin xyz="0 0 0" rpy="0 0 0"/>
@@ -105,4 +105,4 @@
     <child link="closure_bottom"/>
     <origin xyz="-0.05 0.0 0.0" rpy="0 1.5708 0"/>
-</joint>
+</joint>-->
 </robot>
