Commit message: Merged with Kris' version; now works under Fuerte
git-svn-id: https://roboticssrv.wtb.tue.nl/svn/ros/code/tue-ros-pkg/trunk/tue_robot_models/amigo_robot_model@9917 3a3c2cfb-d3b9-409e-9e75-db8fcdbcaac6

File: description/arms/arm.urdf.xacro (robot description, xacro)
@@ -41,5 +41,5 @@
    <origin xyz="-0.00959 -0.19131 -0.00001" rpy="0 0 3.1415" />
    <inertia ixx="0.027"  ixy="0"  ixz="0" iyy="0.027" iyz="0" izz="0.004" />
-   <mesh filename="package://amigo_robot_model/arms_DH/upperarmtextured.dae" scale="0.001 0.001 0.001"/>
+   <mesh filename="package://amigo_robot_model/Media/meshes/upperarmtextured.dae" scale="0.0004 0.0004 0.0004"/>
 </xacro:my_link_texturedmesh>
 <!--the elbow
@@ -56,5 +56,5 @@
    <origin xyz="0.00425 -0.14868 0.00547" rpy="0 -1.5708 0" />
    <inertia ixx="0.0054"  ixy="0"  ixz="0" iyy="0.0054" iyz="0" izz="0.0004" />
-   <mesh filename="package://amigo_robot_model/arms_DH/forearmtextured.dae" scale="0.001 0.001 0.001"/>
+   <mesh filename="package://amigo_robot_model/Media/meshes/forearmtextured.dae" scale="0.0004 0.0004 0.0004"/>
 </xacro:my_link_texturedmesh>
 <!--the wrist

File: description/body/body.urdf.xacro (robot description, xacro)
@@ -10,12 +10,12 @@
    <origin xyz="0.045 0.0 0.06" rpy="-1.5708 0 -1.5708" />
    <inertia ixx="0.01"  ixy="0"  ixz="0" iyy="0.01" iyz="0" izz="0.01" />
-   <mesh filename="package://amigo_robot_model/body/torsocovers.dae" scale="0.001 0.001 0.001"/>
+   <mesh filename="package://amigo_robot_model/Media/meshes/torsocovers.dae" scale="0.0004 0.0004 0.0004"/>
 </xacro:my_link_texturedmesh>
 <!--the spindle-->
 <xacro:my_link_texturedmesh name="torso_slider" mass="0.1" texture="aluminum">
    <origin xyz="0 0 0" rpy="0 0 0"/>
-   <origin xyz="-0.35 0.0 0.0" rpy="0 1.5708 0"/>
+   <origin xyz="0.05 0 0.0" rpy="0 0 1.5708"/>
    <inertia ixx="0.01"  ixy="0"  ixz="0" iyy="0.01" iyz="0" izz="0.01" />
-   <mesh filename="package://amigo_robot_model/body/torsoslidertextured.dae" scale="0.01 0.01 0.01"/>
+   <mesh filename="package://amigo_robot_model/Media/meshes/torsoslidertextured.dae" scale="0.004 0.004 0.004"/>
 </xacro:my_link_texturedmesh>
 <!--the bottomcovers
@@ -26,5 +26,5 @@
    <origin xyz="0.0 0.0 0.33" rpy="0 0 -1.5708" />
    <inertia ixx="2.63"  ixy="0"  ixz="0" iyy="2.63" iyz="0" izz="2.4" />
-   <mesh filename="package://amigo_robot_model/body/bottomcovers.dae" scale="0.001 0.001 0.001"/>
+   <mesh filename="package://amigo_robot_model/Media/meshes/bottomcovers.dae" scale="0.0004 0.0004 0.0004"/>
    <box size="0.275 0.275 0.6"/>
 </xacro:my_link_texturedmesh_diff_coll>

File: description/body_extra_visuals/body_extra.urdf.xacro (robot description, xacro)
@@ -23,5 +23,5 @@
    <origin xyz="-0.4  0.0 0.0" rpy="0 1.5708 0"/>
    <inertia ixx="0.01"  ixy="0"  ixz="0" iyy="0.01" iyz="0" izz="0.01" />
-   <mesh filename="package://amigo_robot_model/body_extra_visuals/torsoassistslidertextured.dae" scale="0.01 0.01 0.0125"/>
+   <mesh filename="package://amigo_robot_model/Media/meshes/torsoassistslidertextured.dae" scale="0.004 0.004 0.005"/>
 </xacro:my_link_texturedmesh>
 <!--left link-->
@@ -30,5 +30,5 @@
    <origin xyz="-0.4  0.0 0.0" rpy="0 1.5708 0"/>
    <inertia ixx="0.01"  ixy="0"  ixz="0" iyy="0.01" iyz="0" izz="0.01" />
-   <mesh filename="package://amigo_robot_model/body_extra_visuals/torsoassistslidertextured.dae" scale="0.01 0.01 0.0125"/>
+   <mesh filename="package://amigo_robot_model/Media/meshes/torsoassistslidertextured.dae" scale="0.004 0.004 0.005"/>
 </xacro:my_link_texturedmesh>
 <!--back link-->
@@ -37,5 +37,5 @@
    <origin xyz="-0.4 0.0 0.0" rpy="0 1.5708 0"/>
    <inertia ixx="0.01"  ixy="0"  ixz="0" iyy="0.01" iyz="0" izz="0.01" />
-   <mesh filename="package://amigo_robot_model/body_extra_visuals/torsoassistslidertextured.dae" scale="0.01 0.01 0.0125"/>
+   <mesh filename="package://amigo_robot_model/Media/meshes/torsoassistslidertextured.dae" scale="0.004 0.004 0.005"/>
 </xacro:my_link_texturedmesh>
 <!--left joint-->

File: description/gazebo/gazebo.urdf.xacro (robot description, xacro)
@@ -129,6 +129,5 @@
         <updateRate>20</updateRate>
         <imageTopicName>/camera/rgb/image_raw</imageTopicName>
-        <!--<pointCloudTopicName>/camera/rgb/points</pointCloudTopicName> --> <!-- To match listening component topic names -->
-        <pointCloudTopicName>/camera/rgb/points_throttled_and_voxelized</pointCloudTopicName> -->
+        <pointCloudTopicName>/camera/rgb/points</pointCloudTopicName>
         <cameraInfoTopicName>/camera/rgb/camera_info</cameraInfoTopicName>
         <frameName>/openni_depth_optical_frame</frameName>
@@ -141,28 +140,3 @@
     </sensor:camera>
   </gazebo>
-  <gazebo reference="base_kinect_openni_camera">
-    <sensor:camera name="base_kinect_openni_camera">
-      <imageFormat>R8G8B8</imageFormat>
-      <imageSize>640 480</imageSize>
-      <hfov>60</hfov>
-      <nearClip>0.05</nearClip>
-      <farClip>3</farClip>
-      <updateRate>20</updateRate>
-      <baseline>0.1</baseline>
-      <controller:gazebo_ros_openni_kinect name="base_kinect_kinect_camera_controller" plugin="libgazebo_ros_openni_kinect.so">
-        <alwaysOn>true</alwaysOn>
-        <updateRate>20</updateRate>
-        <imageTopicName>/base_camera/camera/rgb/image_raw</imageTopicName>
-        <!--<pointCloudTopicName>/base_kinect/camera/rgb/points</pointCloudTopicName> --> <!-- To match listening component topic names -->
-        <pointCloudTopicName>/base_camera/camera/rgb/points_throttled_and_voxelized</pointCloudTopicName>
-        <cameraInfoTopicName>/base_camera/camera/rgb/camera_info</cameraInfoTopicName>
-        <frameName>/base_camera_depth_optical_frame</frameName>
-        <!--<distortion_k1>0.00000001</distortion_k1>
-        <distortion_k2>0.00000001</distortion_k2>
-        <distortion_k3>0.00000001</distortion_k3>
-        <distortion_t1>0.00000001</distortion_t1>
-        <distortion_t2>0.00000001</distortion_t2>-->
-      </controller:gazebo_ros_openni_kinect>
-    </sensor:camera>
-  </gazebo>
 </robot>

File: description/head/head.urdf.xacro (robot description, xacro)
@@ -6,29 +6,22 @@
 <!--head-->
 <!-- !!!!!!!!!something without a visual not sure what this is!!!!!!!!!!!! -->
-<!--<xacro:my_link name="head_mount" mass="0.05" color="Blue">
+<xacro:my_link name="head_mount" mass="0.05" color="Blue">
    <box size="0.01 0.01  0.01 " />
    <origin xyz="0.0 0.0 0.0" rpy="0 0 0"/>
    <origin xyz="0.0 0.0 0.0" rpy="0 0 0" />
-   <inertia ixx="0.0001"  ixy="0"  ixz="0" iyy="0.0001" iyz="0" izz="0.0001" />
-</xacro:my_link>-->
-<link name="head_mount">
-  <inertial>
-`   <origin xyz="0 0 0" rpy="0 0 0"/>
-    <mass value="0.001"/>
-    <inertia ixx="0.001"  ixy="0"  ixz="0" iyy="0.001" iyz="0" izz="0.001" />
-  </inertial>
-</link>
+   <inertia ixx="0.0001"  ixy="0"  ixz="0" iyy="0.0001" iyz="0" izz="0.0001" /> <!--*-->
+</xacro:my_link>
   <joint name="head_mount_joint" type="fixed">
     <parent link="torso"/>
     <child link="head_mount"/>
     <axis xyz="0 0 1"/>
-    <origin xyz="0.107 0.0 0.045" rpy="  0.0 0.0 0.0"/>
+    <origin xyz="0.097 0.0 0.0" rpy="  0.0 0.0 0.0"/>
   </joint>
 <!-- the link that represents the panning part of the neck, is below neck_tilt -->
 <xacro:my_link name="neck_pan" mass="0.05" color="Black">
-   <cylinder radius="0.015" length="0.0525" /> <!--*--> <!--checked-->
+   <cylinder radius="0.015" length="0.0525" />
    <origin xyz="0.0 0.0 0.0335" rpy="0 0 0"/>
    <origin xyz="0.0 0.0 0.0335" rpy="0 0 0" />
-   <inertia ixx="0.0001"  ixy="0"  ixz="0" iyy="0.0001" iyz="0" izz="0.0001" /> <!--*-->
+   <inertia ixx="0.0001"  ixy="0"  ixz="0" iyy="0.0001" iyz="0" izz="0.0001" />
    <color rgba="0.25 0.25 0.25 1.0"/>
 </xacro:my_link>
@@ -37,6 +30,6 @@
    <origin xyz="0.0 -0.0 0.0285" rpy="0 0 0"/>
    <origin xyz="0.0 -0.0 0.015" rpy="0 0 0" />
-   <inertia ixx="0.001"  ixy="0"  ixz="0" iyy="0.001" iyz="0" izz="0.001" /> <!--*-->
-   <mesh filename="package://amigo_robot_model/head/necktilttextured.dae" scale="0.01 0.01 0.01"/>
+   <inertia ixx="0.001"  ixy="0"  ixz="0" iyy="0.001" iyz="0" izz="0.001" />
+   <mesh filename="package://amigo_robot_model/Media/meshes/necktilttextured.dae" scale="0.004 0.004 0.004"/>
 </xacro:my_link_texturedmesh>
 <!--the head itself-->
@@ -45,5 +38,5 @@
    <origin xyz="0.0 0.0 0.1" rpy="0 0 -1.5708"/>
    <inertia ixx="0"  ixy="0"  ixz="0" iyy="0" iyz="0" izz="0" />
-   <mesh filename="package://amigo_robot_model/head/headtextured.dae" scale="0.001 0.001 0.001"/>
+   <mesh filename="package://amigo_robot_model/Media/meshes/headtextured.dae" scale="0.0004 0.0004 0.0004"/>
   </my_link_texturedmesh>
   <joint name="head_joint" type="fixed">
@@ -53,5 +46,5 @@
 <!-- the tilt and pan joints-->
 <xacro:my_joint name="neck_pan_joint" type="revolute" parent="head_mount" child="neck_pan">
-   <origin xyz="0.0 0.0 0.0" rpy="3.14 -1.5708 0.0"/> <!--checked-->
+   <origin xyz="0.0 0.0 0.0" rpy="3.14 -1.5708 0.0"/>
    <dynamics damping="0.1" friction="0"/>
    <axis xyz="0 0 1"/>
@@ -59,5 +52,5 @@
 </xacro:my_joint>
 <xacro:my_joint name="neck_tilt_joint" type="revolute" parent="neck_pan" child="neck_tilt">
-   <origin xyz="0.0 0.0 0.0445" rpy="0.0 0.0 0.0"/> <!--checked-->
+   <origin xyz="0.0 0.0 0.0445" rpy="0.0 0.0 0.0"/>
    <dynamics damping="0.1" friction="0.0"/>
    <axis xyz="0 1 0"/>

File: description/kinect/kinect.urdf.xacro (robot description, xacro)
@@ -6,5 +6,5 @@
   <property name="M_PI" value="3.14159"/>
   <joint name="base_kinect_joint" type="fixed">
-    <origin xyz="0.027 0 0.06" rpy="0 0 0" /> <!-- THESE VALUES ARE ROUGH ESTIMATES!! -->
+    <origin xyz="0.07 0 0.07" rpy="0 0 0" /> <!-- THESE VALUES ARE ROUGH ESTIMATES!! -->
     <parent link="head" />
     <child link="openni_camera" />

File: description/laser/laser.urdf.xacro (robot description, xacro)
@@ -6,8 +6,8 @@
 <!--the laser at the base of the robot -->
 <xacro:my_link name="base_laser" mass="0.5" color="Black">
-   <box size="0.05 0.065 0.12" /> <!--*-->
+   <box size="0.05 0.065 0.12" />
    <origin xyz="0.0 0.0 0.0" rpy="0 0 0"/>
    <origin xyz="-0.005 0.0 -0.065" rpy="0 0 0" />
-   <inertia ixx="0.0001"  ixy="0"  ixz="0" iyy="0.0001" iyz="0" izz="0.0001" /> <!--*-->
+   <inertia ixx="0.0001"  ixy="0"  ixz="0" iyy="0.0001" iyz="0" izz="0.0001" />
 </xacro:my_link>
 <xacro:my_joint name="base_laser_joint" type="fixed" parent="base" child="base_laser">
@@ -19,8 +19,8 @@
 <!--the orange top of the laser-->
 <xacro:my_link_textured name="lasertop" mass="0.01" texture="orange">
-   <box size="0.05 0.065 0.01" /> <!--*-->
+   <box size="0.05 0.065 0.01" />
    <origin xyz="0.0 0.0 0.0" rpy="0 0 0"/>
    <origin xyz="-0.005 0.0 0.0" rpy="0 0 0" />
-   <inertia ixx="0.0001"  ixy="0"  ixz="0" iyy="0.0001" iyz="0" izz="0.0001" /> <!--*-->
+   <inertia ixx="0.0001"  ixy="0"  ixz="0" iyy="0.0001" iyz="0" izz="0.0001" />
 </xacro:my_link_textured>
 <joint name="lasertop_joint" type="fixed">
@@ -32,6 +32,6 @@
    <origin xyz="0.0 0.0 0.0" rpy="0 0 0"/>
    <origin xyz="0.025 0.0 -0.165" rpy="0 0 3.1415" />
-   <inertia ixx="0.0001"  ixy="0"  ixz="0" iyy="0.0001" iyz="0" izz="0.0001" /> <!--*-->
-   <mesh filename="package://amigo_robot_model/laser/logo.dae" scale="0.004 0.004 0.004"/>
+   <inertia ixx="0.0001"  ixy="0"  ixz="0" iyy="0.0001" iyz="0" izz="0.0001" />
+   <mesh filename="package://amigo_robot_model/Media/meshes/logo.dae" scale="0.0016 0.0016 0.0016"/>
 </xacro:my_link_texturedmesh>
   <joint name="logo_joint" type="fixed">

File: description/robot.urdf.xacro (robot description, xacro)
@@ -8,30 +8,28 @@
    <review status="unreviewed" notes=""/>
 <!--get plugins -->
-<include filename="$(find amigo_robot_model)/gazebo/gazebo.urdf.xacro" />
+<include filename="$(find amigo_robot_model)/description/gazebo/gazebo.urdf.xacro" />
 <!--get link & joint definitions -->
-<include filename="$(find amigo_robot_model)/definitions.xacro" />
+<include filename="$(find amigo_robot_model)/description/definitions.xacro" />
 <!--get custom materials -->
-<include filename="$(find amigo_robot_model)/materials.urdf.xacro" />
+<include filename="$(find amigo_robot_model)/description/materials.urdf.xacro" />
 <!--========BUILD BODY======-->
-<include filename="$(find amigo_robot_model)/body/body.urdf.xacro" />
+<include filename="$(find amigo_robot_model)/description/body/body.urdf.xacro" />
 <!--extra body visuals-->
-<include filename="$(find amigo_robot_model)/body_extra_visuals/body_extra.urdf.xacro" />
+<include filename="$(find amigo_robot_model)/description/body_extra_visuals/body_extra.urdf.xacro" />
 <!--========BUILD LASER======-->
-<include filename="$(find amigo_robot_model)/laser/laser.urdf.xacro" />
+<include filename="$(find amigo_robot_model)/description/laser/laser.urdf.xacro" />
 <!--========BUILD HEAD======-->
-<include filename="$(find amigo_robot_model)/head/head.urdf.xacro" />
+<include filename="$(find amigo_robot_model)/description/head/head.urdf.xacro" />
 <!--========BUILD KINECT======-->
-<include filename="$(find amigo_robot_model)/kinect/kinect.urdf.xacro" />
-<!--========BUILD BASE_KINECT======-->
-<include filename="$(find amigo_robot_model)/kinect/base_kinect.urdf.xacro" />
+<include filename="$(find amigo_robot_model)/description/kinect/kinect.urdf.xacro" />
 <!--========BUILD ARMS======-->
-<include filename="$(find amigo_robot_model)/arms_DH/armDH.urdf.xacro" />
+<include filename="$(find amigo_robot_model)/description/arms/arm.urdf.xacro" />
 <xacro:arm whichside="right" sidesign="+1.0" rollsign="+"/>
 <xacro:arm whichside="left"  sidesign="-1.0" rollsign="-"/>
 <!--extra arm visuals-->
-<include filename="$(find amigo_robot_model)/arm_extra_visuals/arm_extra.urdf.xacro" />
+<include filename="$(find amigo_robot_model)/description/arm_extra_visuals/arm_extra.urdf.xacro" />
 <xacro:arm_extra whichside="right" sidesign="+1.0" rollsign="+"/>
 <xacro:arm_extra whichside="left"  sidesign="-1.0" rollsign="-"/>
 <!--====BUILD STUFF THAT NEEDS TO RUN IN EITHER SIMULATION OR ON THE REAL ROBOT ====-->
-<include filename="$(find amigo_robot_model)/sim_or_robot_xacro/robot_real_$(optenv ROBOT_REAL false).urdf.xacro" />
+<include filename="$(find amigo_robot_model)/description/sim_or_robot_xacro/robot_real_$(optenv ROBOT_REAL false).urdf.xacro" />
 </robot>

File: description/sim_or_robot_xacro/robot_real_false.urdf.xacro (robot description, xacro)
@@ -1,7 +1,7 @@
 <?xml version="1.0"?>
 <robot xmlns:xacro="http://ros.org/wiki/xacro">
-<!-- This stuff is run only on in simulation and NOT on the real robot -->
+<!-- This stuff runs only in simulation and NOT on the real robot -->
 <!--====BUILD SIMULATION WHEELS====-->
-<include filename="$(find amigo_robot_model)/wheels/wheels.urdf.xacro" />
+<include filename="$(find amigo_robot_model)/description/wheels/wheels.urdf.xacro" />
 <xacro:wheel side_LR="left" side_FR="front" sign_LR="-" sign_FR="+" wheel_angle="2.3562" />
 <xacro:wheel side_LR="right" side_FR="front" sign_LR="+" sign_FR="+" wheel_angle="0.7854" />
@@ -9,7 +9,7 @@
 <xacro:wheel side_LR="right" side_FR="rear" sign_LR="+" sign_FR="-" wheel_angle="-0.7854" />
 <!--====BUILD SIMULATION TRANSMISSION ELEMENTS====-->
-<include filename="$(find amigo_robot_model)/body/body.transmission.xacro" />
-<include filename="$(find amigo_robot_model)/arms_DH/armDH.transmission.xacro" />
-<include filename="$(find amigo_robot_model)/wheels/wheels.transmission.xacro" />
-<include filename="$(find amigo_robot_model)/head/head.transmission.xacro" />
+<include filename="$(find amigo_robot_model)/description/body/body.transmission.xacro" />
+<include filename="$(find amigo_robot_model)/description/arms/arm.transmission.xacro" />
+<include filename="$(find amigo_robot_model)/description/wheels/wheels.transmission.xacro" />
+<include filename="$(find amigo_robot_model)/description/head/head.transmission.xacro" />
 </robot>

Commit message: Better arm simulation controllers (now take max torque into account)
git-svn-id: https://roboticssrv.wtb.tue.nl/svn/ros/code/tue-ros-pkg/trunk/tue_robot_models/amigo_robot_model@10780 3a3c2cfb-d3b9-409e-9e75-db8fcdbcaac6

File: description/arms/arm.urdf.xacro (robot description, xacro)
@@ -147,11 +147,11 @@
    <dynamics damping="0.1" friction="0.63"/>
    <axis xyz="1 0 0"/>
-   <limit effort="3" velocity="1.0" lower="-0.7854" upper="0.7854"/>
+   <limit effort="3" velocity="1.0" lower="-0.3" upper="0.3"/>
 </xacro:my_joint>
 <xacro:my_joint name="finger2_joint_${whichside}" type="revolute" parent="hand_${whichside}" child="finger2_${whichside}">
    <origin xyz="0.075 -0.04 0" rpy="0 -1.57 0"/>
-   <dynamics damping="0.1" friction="0.0"/>
+   <dynamics damping="0.1" friction="0.63"/>
    <axis xyz="1 0 0"/>
-   <limit effort="3" velocity="1.0" lower="-0.7854" upper="0.7854"/>
+   <limit effort="3" velocity="1.0" lower="-0.3" upper="0.3"/>
 </xacro:my_joint>
   <joint name="grippoint_joint_${whichside}" type="fixed">

Commit message: Increased torque values to resemble real world torques
git-svn-id: https://roboticssrv.wtb.tue.nl/svn/ros/code/tue-ros-pkg/trunk/tue_robot_models/amigo_robot_model@10856 3a3c2cfb-d3b9-409e-9e75-db8fcdbcaac6

File: description/arms/arm.urdf.xacro (robot description, xacro)
@@ -145,5 +145,5 @@
 <xacro:my_joint name="finger1_joint_${whichside}" type="revolute" parent="hand_${whichside}" child="finger1_${whichside}">
    <origin xyz=" 0.075 0.04 0" rpy="0 -1.57 0"/>
-   <dynamics damping="0.1" friction="0.63"/>
+   <dynamics damping="0.5" friction="1.0"/>
    <axis xyz="1 0 0"/>
    <limit effort="3" velocity="1.0" lower="-0.3" upper="0.3"/>
@@ -151,5 +151,5 @@
 <xacro:my_joint name="finger2_joint_${whichside}" type="revolute" parent="hand_${whichside}" child="finger2_${whichside}">
    <origin xyz="0.075 -0.04 0" rpy="0 -1.57 0"/>
-   <dynamics damping="0.1" friction="0.63"/>
+   <dynamics damping="0.5" friction="1.0"/>
    <axis xyz="1 0 0"/>
    <limit effort="3" velocity="1.0" lower="-0.3" upper="0.3"/>

Commit message: Gripper simulation controllers finally working as they should. Perfectly grasping now in Gazebo!
git-svn-id: https://roboticssrv.wtb.tue.nl/svn/ros/code/tue-ros-pkg/trunk/tue_robot_models/amigo_robot_model@10991 3a3c2cfb-d3b9-409e-9e75-db8fcdbcaac6

File: description/arms/arm.urdf.xacro (robot description, xacro)
@@ -80,4 +80,11 @@
    <inertia ixx="0.01"  ixy="0"  ixz="0" iyy="0.01" iyz="0" izz="0.01" />
 </xacro:my_link>
+<!--the right finger phalanx-->
+<xacro:my_link name="finger1_phalanx_${whichside}" mass="0.01" color="White">
+   <cylinder length="0.02" radius="0.009"/>
+   <origin xyz="0.0 0.0 0" rpy="0 0 0"/>
+   <origin xyz="0.0 0.0 0" rpy="0 0 0" />
+   <inertia ixx="0.001"  ixy="0"  ixz="0" iyy="0.001" iyz="0" izz="0.001" />
+</xacro:my_link>
 <!--the right finger tip-->
 <xacro:my_link name="finger1_tip_${whichside}" mass="0.05" color="Black">
@@ -93,4 +100,11 @@
    <origin xyz="0.0 0.0 -0.03" rpy="0 0 0" />
    <inertia ixx="0.01"  ixy="0"  ixz="0" iyy="0.01" iyz="0" izz="0.01" />
+</xacro:my_link>
+<!--the left finger phalanx-->
+<xacro:my_link name="finger2_phalanx_${whichside}" mass="0.01" color="White">
+   <cylinder length="0.02" radius="0.009"/>
+   <origin xyz="0.0 0.0 0" rpy="0 0 0"/>
+   <origin xyz="0.0 0.0 0" rpy="0 0 0" />
+   <inertia ixx="0.001"  ixy="0"  ixz="0" iyy="0.001" iyz="0" izz="0.001" />
 </xacro:my_link>
 <!--the left finger tip -->
@@ -163,4 +177,9 @@
    <limit effort="3" velocity="1.0" lower="-1.57" upper="1.57"/>
 </xacro:my_joint>
+<joint name="finger1_phalanx_joint_${whichside}" type="fixed">
+    <parent link="finger1_${whichside}"/>
+    <child link="finger1_phalanx_${whichside}"/>
+    <origin xyz="0 0 -0.06" rpy="0 1.57 0"/>
+</joint>
 <xacro:my_joint name="finger1_tip_joint_${whichside}" type="revolute" parent="finger1_${whichside}" child="finger1_tip_${whichside}">
    <origin xyz=" 0 0.0 -0.06" rpy="0 0 0"/>
@@ -172,11 +191,16 @@
    <origin xyz="0.075 -0.02 0" rpy="0 -1.57 0"/>
    <dynamics damping="0.5" friction="1.0"/>
-   <axis xyz="1 0 0"/>
-   <limit effort="3" velocity="1.0" lower="-1.57" upper="1.57"/>
-</xacro:my_joint>
+   <axis xyz="-1 0 0"/>
+   <limit effort="3" velocity="1.0" lower="-1.57" upper="1.57"/>
+</xacro:my_joint>
+<joint name="finger2_phalanx_joint_${whichside}" type="fixed">
+    <parent link="finger2_${whichside}"/>
+    <child link="finger2_phalanx_${whichside}"/>
+    <origin xyz="0 0 -0.06" rpy="0 1.57 0"/>
+</joint>
 <xacro:my_joint name="finger2_tip_joint_${whichside}" type="revolute" parent="finger2_${whichside}" child="finger2_tip_${whichside}">
    <origin xyz="0 0 -0.06" rpy="0 0 0"/>
    <dynamics damping="0.5" friction="1.0"/>
-   <axis xyz="1 0 0"/>
+   <axis xyz="-1 0 0"/>
    <limit effort="3" velocity="1.0" lower="-1.57" upper="1.57"/>
 </xacro:my_joint>
