Commit message: Small update on finger Phalanxes
git-svn-id: https://roboticssrv.wtb.tue.nl/svn/ros/code/tue-ros-pkg/trunk/tue_robot_models/amigo_robot_model@10992 3a3c2cfb-d3b9-409e-9e75-db8fcdbcaac6

File: description/arms/arm.urdf.xacro (robot description, xacro)
@@ -82,5 +82,5 @@
 <!--the right finger phalanx-->
 <xacro:my_link name="finger1_phalanx_${whichside}" mass="0.01" color="White">
-   <cylinder length="0.02" radius="0.009"/>
+   <cylinder length="0.019" radius="0.009"/>
    <origin xyz="0.0 0.0 0" rpy="0 0 0"/>
    <origin xyz="0.0 0.0 0" rpy="0 0 0" />
@@ -94,4 +94,11 @@
    <inertia ixx="0.00037"  ixy="0"  ixz="0" iyy="0.00052" iyz="0" izz="0.00052" />
 </xacro:my_link>
+<!--the right finger tip phalanx-->
+<xacro:my_link name="finger1_tip_phalanx_${whichside}" mass="0.01" color="White">
+   <cylinder length="0.017" radius="0.009"/>
+   <origin xyz="0.0 0.0 0" rpy="0 0 0"/>
+   <origin xyz="0.0 0.0 0" rpy="0 0 0" />
+   <inertia ixx="0.001"  ixy="0"  ixz="0" iyy="0.001" iyz="0" izz="0.001" />
+</xacro:my_link>
 <!--the left finger-->
 <xacro:my_link name="finger2_${whichside}" mass="0.05" color="Black">
@@ -103,5 +110,5 @@
 <!--the left finger phalanx-->
 <xacro:my_link name="finger2_phalanx_${whichside}" mass="0.01" color="White">
-   <cylinder length="0.02" radius="0.009"/>
+   <cylinder length="0.019" radius="0.009"/>
    <origin xyz="0.0 0.0 0" rpy="0 0 0"/>
    <origin xyz="0.0 0.0 0" rpy="0 0 0" />
@@ -114,4 +121,11 @@
    <origin xyz="0.0 0.0 -0.03" rpy="0 0 0" />
    <inertia ixx="0.00037"  ixy="0"  ixz="0" iyy="0.00052" iyz="0" izz="0.00052" />
+</xacro:my_link>
+<!--the left finger tip phalanx-->
+<xacro:my_link name="finger2_tip_phalanx_${whichside}" mass="0.01" color="White">
+   <cylinder length="0.017" radius="0.009"/>
+   <origin xyz="0.0 0.0 0" rpy="0 0 0"/>
+   <origin xyz="0.0 0.0 0" rpy="0 0 0" />
+   <inertia ixx="0.001"  ixy="0"  ixz="0" iyy="0.001" iyz="0" izz="0.001" />
 </xacro:my_link>
 <!--the grippoint
@@ -188,4 +202,9 @@
    <limit effort="3" velocity="1.0" lower="-1.57" upper="1.57"/>
 </xacro:my_joint>
+<joint name="finger1_tip_phalanx_joint_${whichside}" type="fixed">
+    <parent link="finger1_tip_${whichside}"/>
+    <child link="finger1_tip_phalanx_${whichside}"/>
+    <origin xyz="0 0 -0.06" rpy="0 1.57 0"/>
+</joint>
 <xacro:my_joint name="finger2_joint_${whichside}" type="revolute" parent="hand_${whichside}" child="finger2_${whichside}">
    <origin xyz="0.075 -0.02 0" rpy="0 -1.57 0"/>
@@ -205,4 +224,9 @@
    <limit effort="3" velocity="1.0" lower="-1.57" upper="1.57"/>
 </xacro:my_joint>
+<joint name="finger2_tip_phalanx_joint_${whichside}" type="fixed">
+    <parent link="finger2_tip_${whichside}"/>
+    <child link="finger2_tip_phalanx_${whichside}"/>
+    <origin xyz="0 0 -0.06" rpy="0 1.57 0"/>
+</joint>
   <joint name="grippoint_joint_${whichside}" type="fixed">
     <parent link="hand_${whichside}"/>

Commit message: Fixed first bug of Rein (IK not solved yet)
git-svn-id: https://roboticssrv.wtb.tue.nl/svn/ros/code/tue-ros-pkg/trunk/tue_robot_models/amigo_robot_model@11014 3a3c2cfb-d3b9-409e-9e75-db8fcdbcaac6

File: description/arms/arm.urdf.xacro (robot description, xacro)
@@ -80,4 +80,8 @@
    <inertia ixx="0.01"  ixy="0"  ixz="0" iyy="0.01" iyz="0" izz="0.01" />
 </xacro:my_link>
+<gazebo reference="finger1_${whichside}">
+  <mu1 value="100.0" />
+  <mu2 value="100.0" />
+</gazebo>
 <!--the right finger phalanx-->
 <xacro:my_link name="finger1_phalanx_${whichside}" mass="0.01" color="White">
@@ -94,4 +98,8 @@
    <inertia ixx="0.00037"  ixy="0"  ixz="0" iyy="0.00052" iyz="0" izz="0.00052" />
 </xacro:my_link>
+<gazebo reference="finger1_tip_${whichside}">
+  <mu1 value="100.0" />
+  <mu2 value="100.0" />
+</gazebo>
 <!--the right finger tip phalanx-->
 <xacro:my_link name="finger1_tip_phalanx_${whichside}" mass="0.01" color="White">
@@ -108,4 +116,8 @@
    <inertia ixx="0.01"  ixy="0"  ixz="0" iyy="0.01" iyz="0" izz="0.01" />
 </xacro:my_link>
+<gazebo reference="finger2_${whichside}">
+  <mu1 value="100.0" />
+  <mu2 value="100.0" />
+</gazebo>
 <!--the left finger phalanx-->
 <xacro:my_link name="finger2_phalanx_${whichside}" mass="0.01" color="White">
@@ -122,4 +134,8 @@
    <inertia ixx="0.00037"  ixy="0"  ixz="0" iyy="0.00052" iyz="0" izz="0.00052" />
 </xacro:my_link>
+<gazebo reference="finger2_tip_${whichside}">
+  <mu1 value="100.0" />
+  <mu2 value="100.0" />
+</gazebo>
 <!--the left finger tip phalanx-->
 <xacro:my_link name="finger2_tip_phalanx_${whichside}" mass="0.01" color="White">
@@ -229,26 +245,9 @@
     <origin xyz="0 0 -0.06" rpy="0 1.57 0"/>
 </joint>
-  <joint name="grippoint_joint_${whichside}" type="fixed">
-    <parent link="hand_${whichside}"/>
-    <child link="grippoint_${whichside}"/>
-    <origin xyz="0.14 0.0 0.0" rpy="0 0 0"/>
-  </joint>
+<joint name="grippoint_joint_${whichside}" type="fixed">
+  <parent link="hand_${whichside}"/>
+  <child link="grippoint_${whichside}"/>
+  <origin xyz="0.14 0.0 0.0" rpy="0 0 0"/>
+</joint>
 </xacro:macro>
-<!-- Friction Gripper -->
-<gazebo reference="finger1_right">
-	<mu1 value="100.0" />
-	<mu2 value="100.0" />
-</gazebo>
-<gazebo reference="finger1_tip_right">
-	<mu1 value="100.0" />
-	<mu2 value="100.0" />
-</gazebo>
-<gazebo reference="finger2_right">
-	<mu1 value="100.0" />
-	<mu2 value="100.0" />
-</gazebo>
-<gazebo reference="finger2_tip_right">
-	<mu1 value="100.0" />
-	<mu2 value="100.0" />
-</gazebo>
 </robot>
