Commit message: Removed weird blue block for head_mount
git-svn-id: https://roboticssrv.wtb.tue.nl/svn/ros/code/tue-ros-pkg/trunk/tue_robot_models/amigo_robot_model@11562 3a3c2cfb-d3b9-409e-9e75-db8fcdbcaac6

File: description/head/head.urdf.xacro (robot description, xacro)
@@ -6,16 +6,17 @@
 <!--head-->
 <!-- !!!!!!!!!something without a visual not sure what this is!!!!!!!!!!!! -->
-<xacro:my_link name="head_mount" mass="0.05" color="Blue">
-   <box size="0.01 0.01  0.01 " />
-   <origin xyz="0.0 0.0 0.0" rpy="0 0 0"/>
-   <origin xyz="0.0 0.0 0.0" rpy="0 0 0" />
-   <inertia ixx="0.0001"  ixy="0"  ixz="0" iyy="0.0001" iyz="0" izz="0.0001" /> <!--*-->
-</xacro:my_link>
-  <joint name="head_mount_joint" type="fixed">
-    <parent link="torso"/>
-    <child link="head_mount"/>
-    <axis xyz="0 0 1"/>
-    <origin xyz="0.097 0.0 0.0" rpy="  0.0 0.0 0.0"/>
-  </joint>
+<link name="head_mount">
+  <inertial>
+    <origin xyz="0.0 0.0 0.0" rpy="0 0 0"/>
+    <mass value="0.001"/>
+    <inertia ixx="0.0001"  ixy="0"  ixz="0" iyy="0.0001" iyz="0" izz="0.0001" />
+  </inertial>
+</link>
+<joint name="head_mount_joint" type="fixed">
+  <parent link="torso"/>
+  <child link="head_mount"/>
+  <axis xyz="0 0 1"/>
+  <origin xyz="0.097 0.0 0.0" rpy="  0.0 0.0 0.0"/>
+</joint>
 <!-- the link that represents the panning part of the neck, is below neck_tilt -->
 <xacro:my_link name="neck_pan" mass="0.05" color="Black">

Commit message: Extended neck of URDF model
git-svn-id: https://roboticssrv.wtb.tue.nl/svn/ros/code/tue-ros-pkg/trunk/tue_robot_models/amigo_robot_model@12189 3a3c2cfb-d3b9-409e-9e75-db8fcdbcaac6

File: description/head/head.urdf.xacro (robot description, xacro)
@@ -36,6 +36,6 @@
 <!--the head itself-->
  <my_link_texturedmesh name="head" mass="0" texture="white">
-   <origin xyz="0 0 0" rpy="0 0 0"/>
-   <origin xyz="0.0 0.0 0.1" rpy="0 0 -1.5708"/>
+   <origin xyz="0 0 0.041" rpy="0 0 0"/>
+   <origin xyz="0.0 0.0 0.141" rpy="0 0 -1.5708"/>
    <inertia ixx="0"  ixy="0"  ixz="0" iyy="0" iyz="0" izz="0" />
    <mesh filename="package://amigo_robot_model/Media/meshes/headtextured.dae" scale="0.0004 0.0004 0.0004"/>
