Commit message: Base kinect update
git-svn-id: https://roboticssrv.wtb.tue.nl/svn/ros/code/tue-ros-pkg/trunk/tue_robot_models/amigo_robot_model@10907 3a3c2cfb-d3b9-409e-9e75-db8fcdbcaac6

File: description/kinect/base_kinect.urdf.xacro (robot description, xacro)
@@ -6,5 +6,5 @@
   <property name="M_PI" value="3.14159"/>
   <joint name="base_kinect_base_kinect_joint" type="fixed">
-    <origin xyz="0.29 0 0.31" rpy="0 -0.07 0" /> <!-- THESE VALUES ARE ROUGH ESTIMATES!! -->
+    <origin xyz="0.5 0 0.5" rpy="0 -0.07 0" /> <!-- THESE VALUES ARE ROUGH ESTIMATES!! -->
     <parent link="base_link" />
     <child link="base_kinect_openni_camera" />
@@ -26,12 +26,12 @@
       </geometry>
     </visual>
-    <collision>
-     <origin xyz=" 0 0 0 " rpy="0 0 0" />
-      <geometry>
-	<!--<box size="0 0 0"/>-->
-        <!--mesh filename="package://amigo_robot_model/description/kinect/meshes/kinect.dae" scale="0.001 0.001 0.001"/-->
-        <mesh filename="package://amigo_robot_model/description/kinect/meshes/kinect_without_base.dae"/>
-      </geometry>
-    </collision>
+    <!--<collision>-->
+     <!--<origin xyz=" 0 0 0 " rpy="0 0 0" />-->
+      <!--<geometry>-->
+	<!--<box size="0.01 0.01 0.01"/>-->
+        <!--<mesh filename="package://amigo_robot_model/description/kinect/meshes/kinect.dae" scale="0.001 0.001 0.001"/>-->
+        <!--<mesh filename="package://amigo_robot_model/description/kinect/meshes/kinect_without_base.dae"/>-->
+      <!--</geometry>-->
+    <!--</collision>-->
   </link>
   <joint name="base_kinect_kinect_depth_joint" type="fixed">

Commit message: Base kinect position change
git-svn-id: https://roboticssrv.wtb.tue.nl/svn/ros/code/tue-ros-pkg/trunk/tue_robot_models/amigo_robot_model@10913 3a3c2cfb-d3b9-409e-9e75-db8fcdbcaac6

File: description/kinect/base_kinect.urdf.xacro (robot description, xacro)
@@ -6,6 +6,6 @@
   <property name="M_PI" value="3.14159"/>
   <joint name="base_kinect_base_kinect_joint" type="fixed">
-    <origin xyz="0.5 0 0.5" rpy="0 -0.07 0" /> <!-- THESE VALUES ARE ROUGH ESTIMATES!! -->
-    <parent link="base_link" />
+    <origin xyz="0.3 0 0.26" rpy="0 -0.07 0" /> <!-- THESE VALUES STILL HAVE TO BE CALIBRATED!! -->
+    <parent link="base" />
     <child link="base_kinect_openni_camera" />
   </joint>

Commit message: Added base kinect mesh: seems to work now!
git-svn-id: https://roboticssrv.wtb.tue.nl/svn/ros/code/tue-ros-pkg/trunk/tue_robot_models/amigo_robot_model@11560 3a3c2cfb-d3b9-409e-9e75-db8fcdbcaac6

File: description/kinect/base_kinect.urdf.xacro (robot description, xacro)
@@ -26,12 +26,12 @@
       </geometry>
     </visual>
-    <!--<collision>-->
-     <!--<origin xyz=" 0 0 0 " rpy="0 0 0" />-->
-      <!--<geometry>-->
+    <collision>
+     <origin xyz=" 0 0 0 " rpy="0 0 0" />
+      <geometry>
 	<!--<box size="0.01 0.01 0.01"/>-->
         <!--<mesh filename="package://amigo_robot_model/description/kinect/meshes/kinect.dae" scale="0.001 0.001 0.001"/>-->
-        <!--<mesh filename="package://amigo_robot_model/description/kinect/meshes/kinect_without_base.dae"/>-->
-      <!--</geometry>-->
-    <!--</collision>-->
+        <mesh filename="package://amigo_robot_model/description/kinect/meshes/kinect_without_base.dae"/>
+      </geometry>
+    </collision>
   </link>
   <joint name="base_kinect_kinect_depth_joint" type="fixed">

Commit message: calibrated base kinect with new mount
git-svn-id: https://roboticssrv.wtb.tue.nl/svn/ros/code/tue-ros-pkg/trunk/tue_robot_models/amigo_robot_model@13155 3a3c2cfb-d3b9-409e-9e75-db8fcdbcaac6

File: description/kinect/base_kinect.urdf.xacro (robot description, xacro)
@@ -6,5 +6,5 @@
   <property name="M_PI" value="3.14159"/>
   <joint name="base_kinect_base_kinect_joint" type="fixed">
-    <origin xyz="0.3 0 0.26" rpy="0 -0.07 0" /> <!-- THESE VALUES STILL HAVE TO BE CALIBRATED!! -->
+    <origin xyz="0.3 0 0.3" rpy="0 0.0 0" />
     <parent link="base" />
     <child link="base_kinect_openni_camera" />
