Commit message: tuned pitch and yaw of head kinect
git-svn-id: https://roboticssrv.wtb.tue.nl/svn/ros/code/tue-ros-pkg/trunk/tue_robot_models/amigo_robot_model@15166 3a3c2cfb-d3b9-409e-9e75-db8fcdbcaac6

File: description/kinect/kinect.urdf.xacro (robot description, xacro)
@@ -6,5 +6,5 @@
   <property name="M_PI" value="3.14159"/>
   <joint name="base_kinect_joint" type="fixed">
-    <origin xyz="0.07 0 0.07" rpy="0 0 0" /> <!-- THESE VALUES ARE ROUGH ESTIMATES!! -->
+    <origin xyz="0.07 0 0.07" rpy="0 -0.01 0.05" /> <!-- THESE VALUES ARE ROUGH ESTIMATES!! -->
     <parent link="head" />
     <child link="openni_camera" />

Commit message: recalibrated base_kinect_joint
git-svn-id: https://roboticssrv.wtb.tue.nl/svn/ros/code/tue-ros-pkg/trunk/tue_robot_models/amigo_robot_model@15877 3a3c2cfb-d3b9-409e-9e75-db8fcdbcaac6

File: description/kinect/kinect.urdf.xacro (robot description, xacro)
@@ -6,5 +6,5 @@
   <property name="M_PI" value="3.14159"/>
   <joint name="base_kinect_joint" type="fixed">
-    <origin xyz="0.07 0 0.07" rpy="0 -0.01 0.05" /> <!-- THESE VALUES ARE ROUGH ESTIMATES!! -->
+    <origin xyz="0.07 0 0.07" rpy="0.0 0.01 0.075" /> <!-- THESE VALUES ARE ROUGH ESTIMATES!! -->
     <parent link="head" />
     <child link="openni_camera" />

Commit message: updated head kinect position in urdf model
git-svn-id: https://roboticssrv.wtb.tue.nl/svn/ros/code/tue-ros-pkg/trunk/tue_robot_models/amigo_robot_model@17969 3a3c2cfb-d3b9-409e-9e75-db8fcdbcaac6

File: description/kinect/kinect.urdf.xacro (robot description, xacro)
@@ -6,5 +6,5 @@
   <property name="M_PI" value="3.14159"/>
   <joint name="base_kinect_joint" type="fixed">
-    <origin xyz="0.07 0 0.07" rpy="0.0 0.01 0.075" /> <!-- THESE VALUES ARE ROUGH ESTIMATES!! -->
+    <origin xyz="0.07 0.05 0.10" rpy="0 0.01 0.015" /> <!-- THESE VALUES ARE ROUGH ESTIMATES!! -->
     <parent link="head" />
     <child link="openni_camera" />
