Commit message: joint limits
git-svn-id: https://roboticssrv.wtb.tue.nl/svn/ros/code/tue-ros-pkg/trunk/tue_robot_models/amigo_robot_model@10711 3a3c2cfb-d3b9-409e-9e75-db8fcdbcaac6

File: description/base/base.urdf.xacro (robot description, xacro)
@@ -9,4 +9,5 @@
         <child link="base_link"/>
         <dynamics damping="100" friction="20" />
+	<limit effort="1000" velocity="1000" lower="-1000" upper="1000" />
     </joint>
     <link name="base_y_link">
@@ -23,4 +24,5 @@
         <child link="base_y_link" />
         <dynamics damping="100" friction="20" />
+        <limit effort="1000" velocity="1000" lower="-1000" upper="1000" />
     </joint>
     <link name="base_x_link">
@@ -37,4 +39,5 @@
         <child link="base_x_link" />
         <dynamics damping="100" friction="20" />
+	<limit effort="1000" velocity="1000" lower="-1000" upper="1000" />
     </joint>
     <link name="base_fixed_link">

Commit message: Robot pose EKF now in the chain
git-svn-id: https://roboticssrv.wtb.tue.nl/svn/ros/code/tue-ros-pkg/trunk/tue_robot_models/amigo_robot_model@13850 3a3c2cfb-d3b9-409e-9e75-db8fcdbcaac6

File: description/base/base.urdf.xacro (robot description, xacro)
@@ -48,9 +48,9 @@
         </inertial>
     </link>
-    <joint name="base_fixed_joint" type="fixed">
+<!--    <joint name="base_fixed_joint" type="fixed">
         <parent link="world" />
         <origin rpy="0 0 0" xyz="0 0 0" />
         <child link="base_fixed_link" />
     </joint>
-    <link name="world" />
+    <link name="world" /> -->
 </robot>

Commit message: Fixed world bug
git-svn-id: https://roboticssrv.wtb.tue.nl/svn/ros/code/tue-ros-pkg/trunk/tue_robot_models/amigo_robot_model@13861 3a3c2cfb-d3b9-409e-9e75-db8fcdbcaac6

File: description/base/base.urdf.xacro (robot description, xacro)
@@ -48,9 +48,9 @@
         </inertial>
     </link>
-<!--    <joint name="base_fixed_joint" type="fixed">
+    <joint name="base_fixed_joint" type="fixed">
         <parent link="world" />
         <origin rpy="0 0 0" xyz="0 0 0" />
         <child link="base_fixed_link" />
     </joint>
-    <link name="world" /> -->
+    <link name="world" />
 </robot>
