Commit message: Added urdf values for laser on back (in comments)
git-svn-id: https://roboticssrv.wtb.tue.nl/svn/ros/code/tue-ros-pkg/trunk/tue_robot_models/amigo_robot_model@14078 3a3c2cfb-d3b9-409e-9e75-db8fcdbcaac6

File: description/laser/laser.urdf.xacro (robot description, xacro)
@@ -12,4 +12,5 @@
 </xacro:my_link>
 <xacro:my_joint name="base_laser_joint" type="fixed" parent="base" child="base_laser">
+   <!--VALUES FOR LASER ON BACK OF AMIGO <origin xyz="-0.235 0.0 0.185" rpy="0 0 3.14"/>-->
    <origin xyz="0.31 0.0 0.185" rpy="0 0 0"/>
    <dynamics damping="0.1" friction="0"/>
