Commit message: updated position of laser, orientation and cropping still needs to be calibrated
git-svn-id: https://roboticssrv.wtb.tue.nl/svn/ros/code/tue-ros-pkg/trunk/tue_robot_models/amigo_robot_model@14599 3a3c2cfb-d3b9-409e-9e75-db8fcdbcaac6

File: description/laser/back_laser.urdf.xacro (robot description, xacro)
@@ -12,5 +12,5 @@
 </xacro:my_link>
 <xacro:my_joint name="back_laser_joint" type="fixed" parent="base" child="back_laser">
-   <origin xyz="-0.235 0.0 0.245" rpy="0 0 3.14"/>
+   <origin xyz="-0.27 0.0 0.245" rpy="0 0 3.14"/>
    <dynamics damping="0.1" friction="0"/>
    <axis xyz="0 1 0"/>
