Commit message: Tuned position of torso laser
git-svn-id: https://roboticssrv.wtb.tue.nl/svn/ros/code/tue-ros-pkg/trunk/tue_robot_models/amigo_robot_model@15816 3a3c2cfb-d3b9-409e-9e75-db8fcdbcaac6

File: description/laser/torso_laser.urdf.xacro (robot description, xacro)
@@ -13,5 +13,5 @@
 <!-- ToDO: Measure exact offset -->
 <xacro:my_joint name="torso_laser_joint" type="fixed" parent="torso" child="torso_laser">
-   <origin xyz="-0.08 0.0 0.05" rpy="0 -1.57 0"/>
+   <origin xyz="-0.0994 0.0 0.075" rpy="0 -1.57 0"/>
    <dynamics damping="0.1" friction="0"/>
    <axis xyz="0 1 0"/>

Commit message: Tuned torso LRF position
git-svn-id: https://roboticssrv.wtb.tue.nl/svn/ros/code/tue-ros-pkg/trunk/tue_robot_models/amigo_robot_model@16961 3a3c2cfb-d3b9-409e-9e75-db8fcdbcaac6

File: description/laser/torso_laser.urdf.xacro (robot description, xacro)
@@ -4,4 +4,10 @@
    <license>BSD</license>
    <review status="unreviewed" notes=""/>
+<xacro:my_link name="torso_dummy" mass="0" color="Red">
+   <cylinder radius="0.0" length="0.00" />
+   <origin xyz="0.0 0.0 0.0" rpy="0 0 0"/>
+   <origin xyz="0.0 0.0 0.0" rpy="0 0 0" />
+   <inertia ixx="0"  ixy="0"  ixz="0" iyy="0" iyz="0" izz="0" />
+</xacro:my_link>
 <!--the laser at the torso of the robot -->
 <xacro:my_link name="torso_laser" mass="0.5" color="Black">
@@ -12,6 +18,14 @@
 </xacro:my_link>
 <!-- ToDO: Measure exact offset -->
-<xacro:my_joint name="torso_laser_joint" type="fixed" parent="torso" child="torso_laser">
-   <origin xyz="-0.0994 0.0 0.075" rpy="0 -1.57 0"/>
+<xacro:my_joint name="torso_dummy_joint" type="fixed" parent="torso" child="torso_dummy">
+   <origin xyz="-0.0994 0.0 0.075" rpy="0.0 -1.57 0.0"/>
+   <dynamics damping="0.1" friction="0"/>
+   <axis xyz="0 1 0"/>
+   <limit effort="13.4" velocity="1.0" lower="-0.7809" upper="1.5708" />
+</xacro:my_joint>
+<!-- ToDO: Measure exact offset -->
+<xacro:my_joint name="torso_laser_joint" type="fixed" parent="torso_dummy" child="torso_laser">
+   <!--<origin xyz="0.0 0.0 0.0" rpy="0.0 0.0 -0.05"/>-->
+   <origin xyz="0.0 0.0 0.0" rpy="0.0 0.0 -0.05"/>
    <dynamics damping="0.1" friction="0"/>
    <axis xyz="0 1 0"/>
