Commit message: Added base kinect for Bas C
git-svn-id: https://roboticssrv.wtb.tue.nl/svn/ros/code/tue-ros-pkg/trunk/tue_robot_models/amigo_robot_model@10898 3a3c2cfb-d3b9-409e-9e75-db8fcdbcaac6

File: description/gazebo/gazebo.urdf.xacro (robot description, xacro)
@@ -143,3 +143,30 @@
     </sensor:camera>
   </gazebo>
+  <gazebo reference="base_openni_camera">
+    <sensor:camera name="base_openni_camera">
+      <imageFormat>R8G8B8</imageFormat>
+      <imageSize>640 480</imageSize>
+      <hfov>60</hfov>
+      <nearClip>0.05</nearClip>
+      <farClip>3</farClip>
+      <updateRate>20</updateRate>
+      <baseline>0.1</baseline>
+      <controller:gazebo_ros_openni_kinect name="base_kinect_camera_controller" plugin="libkinect_controller.so"> <!-- THIS IS THE FORKED VERSION UNTIL NOW (OCT16 2012) THE VERSION IN GAZEBO_PLUGINS WAS NOT SHOWING DEPTH IMAGE PROPERLY!! -->
+        <alwaysOn>true</alwaysOn>
+        <updateRate>20</updateRate>
+	<cameraName>base_camera</cameraName>
+        <imageTopicName>/base_camera/rgb/image_color</imageTopicName>
+	<cameraInfoTopicName>/base_camera/rgb/camera_info</cameraInfoTopicName>
+	<depthImageTopicName>/base_camera/depth/image</depthImageTopicName>
+	<depthImageCameraInfoTopicName>/base_camera/depth/camera_info</depthImageCameraInfoTopicName>
+	<pointCloudTopicName>/base_camera/rgb/points</pointCloudTopicName>
+        <frameName>/base_kinect_openni_depth_optical_frame</frameName>
+        <!--<distortion_k1>0.00000001</distortion_k1>
+        <distortion_k2>0.00000001</distortion_k2>
+        <distortion_k3>0.00000001</distortion_k3>
+        <distortion_t1>0.00000001</distortion_t1>
+        <distortion_t2>0.00000001</distortion_t2>-->
+      </controller:gazebo_ros_openni_kinect>
+    </sensor:camera>
+  </gazebo>
 </robot>

File: description/kinect/base_kinect.urdf.xacro (robot description, xacro)
@@ -22,6 +22,6 @@
       <geometry>
 	<!--<box size="0 0 0"/>-->
-        <!--mesh filename="package://amigo_robot_model/kinect/meshes/kinect.dae" scale="0.001 0.001 0.001"/-->
-        <mesh filename="package://amigo_robot_model/kinect/meshes/kinect_without_base.dae"/>
+        <!--mesh filename="package://amigo_robot_model/description/kinect/meshes/kinect.dae" scale="0.001 0.001 0.001"/-->
+        <mesh filename="package://amigo_robot_model/description/kinect/meshes/kinect_without_base.dae"/>
       </geometry>
     </visual>
@@ -30,6 +30,6 @@
       <geometry>
 	<!--<box size="0 0 0"/>-->
-        <!--mesh filename="package://amigo_robot_model/kinect/meshes/kinect.dae" scale="0.001 0.001 0.001"/-->
-        <mesh filename="package://amigo_robot_model/kinect/meshes/kinect_without_base.dae"/>
+        <!--mesh filename="package://amigo_robot_model/description/kinect/meshes/kinect.dae" scale="0.001 0.001 0.001"/-->
+        <mesh filename="package://amigo_robot_model/description/kinect/meshes/kinect_without_base.dae"/>
       </geometry>
     </collision>

File: description/robot_complex.urdf.xacro (robot description, xacro)
@@ -21,4 +21,5 @@
 <!--========BUILD KINECT======-->
 <include filename="$(find amigo_robot_model)/description/kinect/kinect.urdf.xacro" />
+<include filename="$(find amigo_robot_model)/description/kinect/base_kinect.urdf.xacro" />
 <!--========BUILD ARMS======-->
 <include filename="$(find amigo_robot_model)/description/arms/arm.urdf.xacro" />

File: description/robot_simple.urdf.xacro (robot description, xacro)
@@ -21,4 +21,5 @@
 <!--========BUILD KINECT======-->
 <include filename="$(find amigo_robot_model)/description/kinect/kinect.urdf.xacro" />
+<include filename="$(find amigo_robot_model)/description/kinect/base_kinect.urdf.xacro" />
 <!--========BUILD ARMS======-->
 <include filename="$(find amigo_robot_model)/description/arms/arm.urdf.xacro" />

Commit message: Gazebo cleanup
git-svn-id: https://roboticssrv.wtb.tue.nl/svn/ros/code/tue-ros-pkg/trunk/tue_robot_models/amigo_robot_model@13864 3a3c2cfb-d3b9-409e-9e75-db8fcdbcaac6

File: description/gazebo/gazebo.urdf.xacro (robot description, xacro)
@@ -3,11 +3,6 @@
        xmlns:controller="http://playerstage.sourceforge.net/gazebo/xmlschema/#controller"
        xmlns:interface="http://playerstage.sourceforge.net/gazebo/xmlschema/#interface">
-<!--======== Plugins ========-->
-<gazebo>
-      <controller:gazebo_ros_time name="gazebo_ros_time" plugin="libgazebo_ros_time.so">
-        <alwaysOn>true</alwaysOn>
-        <updateRate>1000.0</updateRate>
-        <interface:audio name="dummy_gazebo_ros_time_iface_should_not_be_here"/>
-      </controller:gazebo_ros_time>
+  <!--======== Plugins ========-->
+  <gazebo>
       <controller:gazebo_ros_controller_manager name="gazebo_ros_controller_manager" plugin="libgazebo_ros_controller_manager.so">
         <alwaysOn>true</alwaysOn>
@@ -19,22 +14,13 @@
          <updateRate>1000.0</updateRate>
          <bodyName>base_link</bodyName>
-         <topicName>body_pose_ground_truth</topicName>
-         <xyzOffsets>0.0 0.0 0</xyzOffsets>
-         <rpyOffsets>0 0 0</rpyOffsets>
+         <topicName>imu_data</topicName>
+	 <serviceName>imu_service</serviceName>
+	 <gaussianNoise>2.89e-08</gaussianNoise>
+         <xyzOffset>0 0 0</xyzOffset>
+         <rpyOffset>0 0 0</rpyOffset>
          <interface:position name="imu_position_iface"/>
        </controller:gazebo_ros_imu>
-       <controller:gazebo_ros_p3d name="base_controller" plugin="libgazebo_ros_p3d.so">
-        <alwaysOn>true</alwaysOn>
-        <updateRate>100.0</updateRate>
-        <bodyName>base_link</bodyName>
-        <topicName>base_pose_ground_truth</topicName>
-        <gaussianNoise>0.01</gaussianNoise>
-        <frameName>map</frameName>
-        <xyzOffsets>25.7 25.7 0</xyzOffsets> <!-- initialize odometry for fake localization-->
-        <rpyOffsets>0 0 0</rpyOffsets>
-        <interface:position name="p3d_base_position"/>
-      </controller:gazebo_ros_p3d>
   </gazebo>
- <gazebo reference="base_laser">
+  <gazebo reference="base_laser">
     <sensor:ray name="base_ray_sensor">
       <origin>0.0 0.0 0.0</origin>
@@ -55,65 +41,9 @@
         <topicName>base_scan</topicName>
         <frameName>/base_laser</frameName>
+	<hokuyoMinIntensity>101</hokuyoMinIntensity>
         <interface:laser name="base_ros_ray_sensor_iface"/>
       </controller:gazebo_ros_laser>
     </sensor:ray>
-</gazebo>
- <gazebo reference="top_laser">
-    <sensor:ray name="top_ray_sensor">
-      <origin>0.0 0.0 0.0</origin>
-      <rayCount>683</rayCount>
-      <rangeCount>683</rangeCount>
-      <laserCount>1</laserCount>
-      <displayRays>false</displayRays>
-      <minAngle>-135</minAngle>
-      <maxAngle> 135</maxAngle>
-      <minRange>0.05</minRange>
-      <maxRange>10.0</maxRange>
-      <resRange>0.01</resRange>
-      <updateRate>100.0</updateRate>
-      <controller:gazebo_ros_laser name="top_ros_ray_sensor_controller" plugin="libgazebo_ros_laser.so">
-        <gaussianNoise>0.005</gaussianNoise>
-        <alwaysOn>true</alwaysOn>
-        <updateRate>15.0</updateRate>
-        <topicName>top_scan</topicName>
-        <frameName>/top_laser</frameName>
-        <interface:laser name="top_ros_ray_sensor_iface"/>
-      </controller:gazebo_ros_laser>
-    </sensor:ray>
-</gazebo>
-<!--
-  <gazebo reference="camera_left">
-    <sensor:camera name="camera_left_sensor">
-      <controller:gazebo_ros_camera name="controller_left-name" plugin="libgazebo_ros_camera.so">
-        <alwaysOn>true</alwaysOn>
-        <updateRate>15.0</updateRate>
-        <imageTopicName>/left/image_raw</imageTopicName>
-        <cameraInfoTopicName>/left/camera_info</cameraInfoTopicName>
-        <frameName>/camera_tf</frameName>
-      </controller:gazebo_ros_camera>
-    </sensor:camera>
   </gazebo>
-  <gazebo reference="camera_right">
-    <sensor:camera name="camera_right_sensor">
-      <controller:gazebo_ros_camera name="controller_right-name" plugin="libgazebo_ros_camera.so">
-        <alwaysOn>true</alwaysOn>
-        <updateRate>15.0</updateRate>
-        <imageTopicName>/right/image_raw</imageTopicName>
-        <cameraInfoTopicName>/right/camera_info</cameraInfoTopicName>
-        <frameName>/camera_tf</frameName>
-      </controller:gazebo_ros_camera>
-    </sensor:camera>
-  </gazebo>
-  <gazebo reference="camera_center">
-    <sensor:camera name="camera_center_sensor">
-      <controller:gazebo_ros_camera name="controller_center_name" plugin="libgazebo_ros_camera.so">
-        <alwaysOn>true</alwaysOn>
-        <updateRate>15.0</updateRate>
-        <imageTopicName>/center/image_raw</imageTopicName>
-        <cameraInfoTopicName>/center/camera_info</cameraInfoTopicName>
-        <frameName>/camera_tf</frameName>
-      </controller:gazebo_ros_camera>
-    </sensor:camera>
-  </gazebo>-->
   <gazebo reference="openni_camera">
     <sensor:camera name="openni_camera">
@@ -135,9 +65,14 @@
 	<pointCloudTopicName>/camera/rgb/points</pointCloudTopicName>
         <frameName>/openni_depth_optical_frame</frameName>
-        <!--<distortion_k1>0.00000001</distortion_k1>
-        <distortion_k2>0.00000001</distortion_k2>
-        <distortion_k3>0.00000001</distortion_k3>
-        <distortion_t1>0.00000001</distortion_t1>
-        <distortion_t2>0.00000001</distortion_t2>-->
+        <distortionK1>0.0</distortionK1>
+        <distortionK2>0.0</distortionK2>
+        <distortionK3>0.0</distortionK3>
+        <distortionT1>0.0</distortionT1>
+        <distortionT2>0.0</distortionT2>
+	<CxPrime>0.0</CxPrime>
+	<Cx>0.0</Cx>
+	<Cy>0.0</Cy>
+	<focalLength>0.0</focalLength>
+	<hackBaseline>0.0</hackBaseline>
       </controller:gazebo_ros_openni_kinect>
     </sensor:camera>
@@ -162,9 +97,14 @@
 	<pointCloudTopicName>/base_camera/rgb/points</pointCloudTopicName>
         <frameName>/base_kinect_openni_depth_optical_frame</frameName>
-        <!--<distortion_k1>0.00000001</distortion_k1>
-        <distortion_k2>0.00000001</distortion_k2>
-        <distortion_k3>0.00000001</distortion_k3>
-        <distortion_t1>0.00000001</distortion_t1>
-        <distortion_t2>0.00000001</distortion_t2>-->
+        <distortionK1>0.0</distortionK1>
+        <distortionK2>0.0</distortionK2>
+        <distortionK3>0.0</distortionK3>
+        <distortionT1>0.0</distortionT1>
+        <distortionT2>0.0</distortionT2>
+	<CxPrime>0.0</CxPrime>
+	<Cx>0.0</Cx>
+	<Cy>0.0</Cy>
+	<focalLength>0.0</focalLength>
+	<hackBaseline>0.0</hackBaseline>
       </controller:gazebo_ros_openni_kinect>
     </sensor:camera>

Commit message: Added back laser
git-svn-id: https://roboticssrv.wtb.tue.nl/svn/ros/code/tue-ros-pkg/trunk/tue_robot_models/amigo_robot_model@14202 3a3c2cfb-d3b9-409e-9e75-db8fcdbcaac6

File: description/gazebo/gazebo.urdf.xacro (robot description, xacro)
@@ -22,6 +22,6 @@
        </controller:gazebo_ros_imu>
   </gazebo>
-  <gazebo reference="base_laser">
-    <sensor:ray name="base_ray_sensor">
+  <gazebo reference="front_laser">
+    <sensor:ray name="front_laser_sensor">
       <origin>0.0 0.0 0.0</origin>
       <rayCount>683</rayCount>
@@ -35,12 +35,36 @@
       <resRange>0.01</resRange>
       <updateRate>100.0</updateRate>
-      <controller:gazebo_ros_laser name="base_ros_ray_sensor_controller" plugin="libgazebo_ros_laser.so">
+      <controller:gazebo_ros_laser name="front_laser_sensor_controller" plugin="libgazebo_ros_laser.so">
         <gaussianNoise>0.005</gaussianNoise>
         <alwaysOn>true</alwaysOn>
         <updateRate>15.0</updateRate>
-        <topicName>base_scan</topicName>
-        <frameName>/base_laser</frameName>
+        <topicName>scan</topicName>
+        <frameName>/front_laser</frameName>
 	<hokuyoMinIntensity>101</hokuyoMinIntensity>
-        <interface:laser name="base_ros_ray_sensor_iface"/>
+        <interface:laser name="front_laser_sensor_iface"/>
+      </controller:gazebo_ros_laser>
+    </sensor:ray>
+  </gazebo>
+  <gazebo reference="back_laser">
+    <sensor:ray name="back_laser_sensor">
+      <origin>0.0 0.0 0.0</origin>
+      <rayCount>683</rayCount>
+      <rangeCount>683</rangeCount>
+      <laserCount>1</laserCount>
+      <displayRays>false</displayRays>
+      <minAngle>-120</minAngle>
+      <maxAngle> 120</maxAngle>
+      <minRange>0.05</minRange>
+      <maxRange>10.0</maxRange>
+      <resRange>0.01</resRange>
+      <updateRate>100.0</updateRate>
+      <controller:gazebo_ros_laser name="back_laser_sensor_controller" plugin="libgazebo_ros_laser.so">
+        <gaussianNoise>0.005</gaussianNoise>
+        <alwaysOn>true</alwaysOn>
+        <updateRate>15.0</updateRate>
+        <topicName>scan</topicName>
+        <frameName>/back_laser</frameName>
+	<hokuyoMinIntensity>101</hokuyoMinIntensity>
+        <interface:laser name="back_laser_sensor_iface"/>
       </controller:gazebo_ros_laser>
     </sensor:ray>

File: description/laser/front_laser.urdf.xacro (robot description, xacro)
@@ -4,6 +4,6 @@
    <license>BSD</license>
    <review status="unreviewed" notes=""/>
-<!--the laser at the base of the robot -->
-<xacro:my_link name="base_laser" mass="0.5" color="Black">
+<!--the laser at the front of the robot -->
+<xacro:my_link name="front_laser" mass="0.5" color="Black">
    <box size="0.05 0.065 0.12" />
    <origin xyz="0.0 0.0 0.0" rpy="0 0 0"/>
@@ -11,7 +11,6 @@
    <inertia ixx="0.0001"  ixy="0"  ixz="0" iyy="0.0001" iyz="0" izz="0.0001" />
 </xacro:my_link>
-<xacro:my_joint name="base_laser_joint" type="fixed" parent="base" child="base_laser">
-   <!--VALUES FOR LASER ON BACK OF AMIGO <origin xyz="-0.235 0.0 0.185" rpy="0 0 3.14"/>-->
-   <origin xyz="0.31 0.0 0.185" rpy="0 0 0"/>
+<xacro:my_joint name="front_laser_joint" type="fixed" parent="base" child="front_laser">
+   <origin xyz="0.31 0.0 0.245" rpy="0 0 0"/>
    <dynamics damping="0.1" friction="0"/>
    <axis xyz="0 1 0"/>
@@ -19,5 +18,5 @@
 </xacro:my_joint>
 <!--the orange top of the laser-->
-<xacro:my_link_textured name="lasertop" mass="0.01" texture="orange">
+<xacro:my_link_textured name="front_lasertop" mass="0.01" texture="orange">
    <box size="0.05 0.065 0.01" />
    <origin xyz="0.0 0.0 0.0" rpy="0 0 0"/>
@@ -25,7 +24,7 @@
    <inertia ixx="0.0001"  ixy="0"  ixz="0" iyy="0.0001" iyz="0" izz="0.0001" />
 </xacro:my_link_textured>
-<joint name="lasertop_joint" type="fixed">
-    <parent link="base_laser"/>
-    <child link="lasertop"/>
+<joint name="front_lasertop_joint" type="fixed">
+    <parent link="front_laser"/>
+    <child link="front_lasertop"/>
 </joint>
 <!--the tue logo in front of the laser-->
@@ -37,5 +36,5 @@
 </xacro:my_link_texturedmesh>
   <joint name="logo_joint" type="fixed">
-    <parent link="base_laser"/>
+    <parent link="front_laser"/>
     <child link="logo"/>
   </joint>

File: description/robot_complex.urdf.xacro (robot description, xacro)
@@ -15,6 +15,7 @@
 <!--extra body visuals-->
 <include filename="$(find amigo_robot_model)/description/body_extra_visuals/body_extra.urdf.xacro" />
-<!--========BUILD LASER======-->
-<include filename="$(find amigo_robot_model)/description/laser/laser.urdf.xacro" />
+<!--========BUILD LASERS======-->
+<include filename="$(find amigo_robot_model)/description/laser/front_laser.urdf.xacro" />
+<include filename="$(find amigo_robot_model)/description/laser/back_laser.urdf.xacro" />
 <!--========BUILD HEAD======-->
 <include filename="$(find amigo_robot_model)/description/head/head.urdf.xacro" />

File: description/robot_simple.urdf.xacro (robot description, xacro)
@@ -15,6 +15,7 @@
 <!--extra body visuals-->
 <include filename="$(find amigo_robot_model)/description/body_extra_visuals/body_extra.urdf.xacro" />
-<!--========BUILD LASER======-->
-<include filename="$(find amigo_robot_model)/description/laser/laser.urdf.xacro" />
+<!--========BUILD LASERS======-->
+<include filename="$(find amigo_robot_model)/description/laser/front_laser.urdf.xacro" />
+<include filename="$(find amigo_robot_model)/description/laser/back_laser.urdf.xacro" />
 <!--========BUILD HEAD======-->
 <include filename="$(find amigo_robot_model)/description/head/head.urdf.xacro" />
