Commit message: Renamed spindle joint
git-svn-id: https://roboticssrv.wtb.tue.nl/svn/ros/code/tue-ros-pkg/trunk/tue_robot_models/amigo_robot_model@18359 3a3c2cfb-d3b9-409e-9e75-db8fcdbcaac6

File: description/body/body.transmission.xacro (robot description, xacro)
@@ -4,5 +4,5 @@
         <transmission name="spindle_trans" type="pr2_mechanism_model/SimpleTransmission">
                 <actuator name="spindle_motor" />
-                <joint name="spindle_joint" />
+                <joint name="torso_joint" />
                 <mechanicalReduction>1</mechanicalReduction>
                 <motorTorqueConstant>1</motorTorqueConstant>

File: description/body/body.urdf.xacro (robot description, xacro)
@@ -34,5 +34,5 @@
 </xacro:my_link>
 <!-- joints start here -->
-<joint name="spindle_joint" type="prismatic">
+<joint name="torso_joint" type="prismatic">
   <parent link="base"/>
   <child link="torso_slider"/>
